Commit message: global search and replace create -> turtlebot

File: turtlebot_urdf/urdf/create.urdf.xacro (robot description, xacro)
@@ -1,9 +1,9 @@
 <?xml version="1.0"?>
-<robot name="create"
+<robot name="turtlebot"
     xmlns:sensor="http://playerstage.sourceforge.net/gazebo/xmlschema/#sensor"
     xmlns:controller="http://playerstage.sourceforge.net/gazebo/xmlschema/#controller"
     xmlns:interface="http://playerstage.sourceforge.net/gazebo/xmlschema/#interface">
     <!-- Included URDF Files -->
-    <include filename="$(find create_urdf)/urdf/create_base.xacro" />
-    <create />
+    <include filename="$(find turtlebot_urdf)/urdf/turtlebot_base.xacro" />
+    <turtlebot />
 </robot>

File: turtlebot_urdf/urdf/create_base.xacro (robot description, xacro)
@@ -5,7 +5,7 @@
     xmlns:interface="http://playerstage.sourceforge.net/gazebo/xmlschema/#interface">
     <!-- Included URDF Files -->
-    <include filename="$(find create_urdf)/urdf/materials.urdf.xacro" />
+    <include filename="$(find turtlebot_urdf)/urdf/materials.urdf.xacro" />
     <!--
-    <include filename="$(find create_urdf)/urdf/create_wheel.xacro" />
+    <include filename="$(find turtlebot_urdf)/urdf/turtlebot_wheel.xacro" />
     -->
     <!-- Properties (Constants) -->
@@ -14,5 +14,5 @@
     <property name="base_size_y" value="0.33" />
     <property name="base_calibration_factor" value="0.5" />
-    <macro name="create">
+    <macro name="turtlebot">
         <!-- base_footprint is a fictitious link(frame) that is on the ground right below base_link origin,
              navigation stack depends on this frame -->
@@ -58,5 +58,5 @@
                 <origin xyz="0.0 0.0 0.02" rpy="0 0 0" />
                 <geometry>
-                    <mesh filename="package://create_urdf/meshes/create_body.dae"/>
+                    <mesh filename="package://turtlebot_urdf/meshes/turtlebot_body.dae"/>
                 </geometry>
                 <material name="Blue" />
@@ -65,5 +65,5 @@
                 <origin xyz="0.0 0.0 0.0" rpy="0 0 0" />
                 <geometry>
-                    <mesh filename="package://create_urdf/meshes/create_body.stl"/>
+                    <mesh filename="package://turtlebot_urdf/meshes/turtlebot_body.stl"/>
                 </geometry>
             </collision>

File: turtlebot_urdf/urdf/create_wheel.xacro (robot description, xacro)
@@ -7,5 +7,5 @@
     <property name="M_PI" value="3.14159"/>
     <property name="wheel_offset_z" value="-0.0128" />
-    <macro name="create_wheel" params="suffix parent reflect">
+    <macro name="turtlebot_wheel" params="suffix parent reflect">
         <joint name="${parent}_${suffix}_motor_joint" type="fixed">
             <origin xyz="0 ${reflect*base_calibration_factor*base_size_y/2} ${wheel_offset_z}" rpy="0 0 0" />
@@ -70,8 +70,8 @@
             <elem key="kp"  value="100000000.0" />
             <elem key="kd"  value="1.0" />
-            <material>Create/Grey</material>
+            <material>Turtlebot/Grey</material>
         </gazebo>
         <gazebo reference="${parent}_${suffix}_motor_link" >
-            <material>Create/White</material>
+            <material>Turtlebot/White</material>
         </gazebo>
         <transmission type="pr2_mechanism_model/SimpleTransmission" name="${parent}_${suffix}_wheel_trans">
