Commit message: fixing filenames
--HG--
rename : turtlebot_bringup/create.launch => turtlebot_bringup/turtlebot.launch
rename : turtlebot_bringup/create_solo.launch => turtlebot_bringup/turtlebot_solo.launch
rename : turtlebot_driver/src/create_driver.py => turtlebot_driver/src/turtlebot_driver.py
rename : turtlebot_node/nodes/create_node.py => turtlebot_node/nodes/turtlebot_node.py
rename : turtlebot_node/src/create_node/__init__.py => turtlebot_node/src/turtlebot_node/__init__.py
rename : turtlebot_node/src/create_node/diagnostics.py => turtlebot_node/src/turtlebot_node/diagnostics.py
rename : turtlebot_node/src/create_node/gyro.py => turtlebot_node/src/turtlebot_node/gyro.py
rename : turtlebot_urdf/urdf/create.urdf.xacro => turtlebot_urdf/urdf/turtlebot.urdf.xacro
rename : turtlebot_urdf/urdf/create_base.xacro => turtlebot_urdf/urdf/turtlebot_base.xacro
rename : turtlebot_urdf/urdf/create_wheel.xacro => turtlebot_urdf/urdf/turtlebot_wheel.xacro

File: turtlebot_urdf/urdf/turtlebot_base.xacro (robot description, xacro)
@@ -58,5 +58,5 @@
                 <origin xyz="0.0 0.0 0.02" rpy="0 0 0" />
                 <geometry>
-                    <mesh filename="package://turtlebot_urdf/meshes/turtlebot_body.dae"/>
+                    <mesh filename="package://turtlebot_urdf/meshes/create_body.dae"/>
                 </geometry>
                 <material name="Blue" />
@@ -65,5 +65,5 @@
                 <origin xyz="0.0 0.0 0.0" rpy="0 0 0" />
                 <geometry>
-                    <mesh filename="package://turtlebot_urdf/meshes/turtlebot_body.stl"/>
+                    <mesh filename="package://turtlebot_urdf/meshes/create_body.stl"/>
                 </geometry>
             </collision>
