Commit message: adding new cool models

File: turtlebot_urdf/urdf/turtlebot.xacro (robot description, xacro)
@@ -1,4 +1,5 @@
 <?xml version="1.0"?>
 <robot>
+  <include filename="$(find turtlebot_urdf)/urdf/turtlebot_hardware.xacro" />
   <material name="Blue">
     <color rgba="0.0 0.0 0.8 1.0"/>
@@ -9,5 +10,5 @@
   <property name="base_x" value="0.33" />
   <property name="base_y" value="0.33" />
-  <macro name ="turtlebot">
+  <macro name="turtlebot">
     <link name="base_link">
       <inertial>
@@ -31,27 +32,10 @@
       </collision>
     </link>
-    <joint name="gyro_joint" type="fixed">
-      <origin xyz="0 0 0.03" rpy="0 0 0" />
-      <parent link="base_link"/>
-      <child link="gyro_link" />
-    </joint>
-    <link name="gyro_link">
-      <inertial>
-        <mass value="0.01" />
-        <origin xyz="0 0 0.03" />
-        <inertia ixx="1.0" ixy="0.0" ixz="0.0"
-                 iyy="1.0" iyz="0.0"
-                 izz="1.0" />
-      </inertial>
-      <visual>
-        <origin xyz="0.0 0.0 0.02" rpy="0 0 0" />
-        <geometry>
-          <cylinder radius="0.002" length="0.006" />
-        </geometry>
-        <material name="Blue" />
-      </visual>
-    </link>
+    <turtlebot_spacer number="0" x_loc="-0.00254" y_loc="0.1114679" z_loc="0.062992"/>
+    <turtlebot_spacer number="1" x_loc="-0.00254" y_loc="-0.1114679" z_loc="0.062992"/>
+    <turtlebot_spacer number="2" x_loc="-0.07239" y_loc="-0.1114679" z_loc="0.062992"/>
+    <turtlebot_spacer number="3" x_loc="-0.07239" y_loc="0.1114679" z_loc="0.062992"/>
     <joint name="plate_0_joint" type="fixed">
-      <origin xyz="-0.17 0 0.1" rpy="0 0 0" />
+      <origin xyz="-0.04334 0 0.066167" rpy="0 0 0" />
       <parent link="base_link"/>
       <child link="plate_0_link" />
@@ -68,5 +52,5 @@
         <origin xyz=" 0 0 0 " rpy="0 0 0" />
         <geometry>
-          <mesh filename="package://turtlebot_urdf/meshes/Turtlebot_Plate_0_Logo.3ds" scale="${M_SCALE} ${M_SCALE} ${M_SCALE}"/>
+          <mesh filename="package://turtlebot_urdf/meshes/Turtlebot_Plate_0_Logo.dae" scale="${M_SCALE} ${M_SCALE} ${M_SCALE}"/>
         </geometry>
       </visual>

Commit message: adding the next models in the chain

File: turtlebot_urdf/urdf/turtlebot.xacro (robot description, xacro)
@@ -37,5 +37,5 @@
     <turtlebot_spacer number="3" x_loc="-0.07239" y_loc="0.1114679" z_loc="0.062992"/>
     <joint name="plate_0_joint" type="fixed">
-      <origin xyz="-0.04334 0 0.066167" rpy="0 0 0" />
+      <origin xyz="-0.04334 0  0.0645795" rpy="0 0 0" />
       <parent link="base_link"/>
       <child link="plate_0_link" />
@@ -62,4 +62,8 @@
       </collision>
     </link>
+    <turtlebot_standoff_1in number="0" x_loc="0.0676402" y_loc="0.1314196" z_loc="0.0709803"/>
+    <turtlebot_standoff_1in number="1" x_loc="0.0676402" y_loc="-0.1314196" z_loc="0.0709803"/>
+    <turtlebot_standoff_1in number="2" x_loc="-0.052832" y_loc="-0.1314196" z_loc="0.0709803"/>
+    <turtlebot_standoff_1in number="3" x_loc="-0.052832" y_loc="0.1314196" z_loc="0.0709803"/>
   </macro>
 </robot>

File: turtlebot_urdf/urdf/turtlebot_hardware.xacro (robot description, xacro)
@@ -31,3 +31,31 @@
     </link>
   </macro>
+  <macro name="turtlebot_standoff_1in" params="number x_loc y_loc z_loc">
+    <joint name="standoff_1in_${number}_joint" type="fixed">
+      <origin xyz="${x_loc} ${y_loc} ${z_loc}" rpy="0 0 0" />
+      <parent link="base_link"/>
+      <child link="standoff_1in_${number}_link" />
+    </joint>
+    <link name="standoff_1in_${number}_link">
+      <inertial>
+	<mass value="1" />
+	<origin xyz="0 0 0" />
+	<inertia ixx="1.0" ixy="0.0" ixz="0.0"
+		 iyy="1.0" iyz="0.0"
+		 izz="1.0" />
+      </inertial>
+      <visual>
+	<origin xyz=" 0 0 0 " rpy="0 0 0" />
+	<geometry>
+	  <mesh filename="package://turtlebot_urdf/meshes/68-04552-1000-RA_Turtlebot_M-F_Standoff.dae" scale="${M_SCALE} ${M_SCALE} ${M_SCALE}"/>
+	</geometry>
+      </visual>
+      <collision>
+	<origin xyz="0.0 0.0 0.0" rpy="0 0 0" />
+	<geometry>
+	  <mesh filename="package://turtlebot_urdf/meshes/68-04552-1000-RA_Turtlebot_M-F_Standoff.dae"/>
+	</geometry>
+      </collision>
+    </link>
+  </macro>
 </robot>

Commit message: added two more layers to the model almost done

File: turtlebot_urdf/urdf/turtlebot.xacro (robot description, xacro)
@@ -32,8 +32,8 @@
       </collision>
     </link>
-    <turtlebot_spacer number="0" x_loc="-0.00254" y_loc="0.1114679" z_loc="0.062992"/>
-    <turtlebot_spacer number="1" x_loc="-0.00254" y_loc="-0.1114679" z_loc="0.062992"/>
-    <turtlebot_spacer number="2" x_loc="-0.07239" y_loc="-0.1114679" z_loc="0.062992"/>
-    <turtlebot_spacer number="3" x_loc="-0.07239" y_loc="0.1114679" z_loc="0.062992"/>
+    <turtlebot_spacer parent="base_link" number="0" x_loc="-0.00254" y_loc="0.1114679" z_loc="0.062992"/>
+    <turtlebot_spacer parent="base_link" number="1" x_loc="-0.00254" y_loc="-0.1114679" z_loc="0.062992"/>
+    <turtlebot_spacer parent="base_link" number="2" x_loc="-0.07239" y_loc="-0.1114679" z_loc="0.062992"/>
+    <turtlebot_spacer parent="base_link" number="3" x_loc="-0.07239" y_loc="0.1114679" z_loc="0.062992"/>
     <joint name="plate_0_joint" type="fixed">
       <origin xyz="-0.04334 0  0.0645795" rpy="0 0 0" />
@@ -62,8 +62,64 @@
       </collision>
     </link>
-    <turtlebot_standoff_1in number="0" x_loc="0.0676402" y_loc="0.1314196" z_loc="0.0709803"/>
-    <turtlebot_standoff_1in number="1" x_loc="0.0676402" y_loc="-0.1314196" z_loc="0.0709803"/>
-    <turtlebot_standoff_1in number="2" x_loc="-0.052832" y_loc="-0.1314196" z_loc="0.0709803"/>
-    <turtlebot_standoff_1in number="3" x_loc="-0.052832" y_loc="0.1314196" z_loc="0.0709803"/>
+    <turtlebot_standoff_1in parent="base_link" number="0" x_loc="0.0676402" y_loc="0.1314196" z_loc="0.0709803"/>
+    <turtlebot_standoff_1in parent="base_link" number="1" x_loc="0.0676402" y_loc="-0.1314196" z_loc="0.0709803"/>
+    <turtlebot_standoff_1in parent="base_link" number="2" x_loc="-0.052832" y_loc="-0.1314196" z_loc="0.0709803"/>
+    <turtlebot_standoff_1in parent="base_link" number="3" x_loc="-0.052832" y_loc="0.1314196" z_loc="0.0709803"/>
+    <joint name="plate_1_joint" type="fixed">
+      <origin xyz="0.04068 0 0.0318008" rpy="0 0 0" />
+      <parent link="plate_0_link"/>
+      <child link="plate_1_link" />
+    </joint>
+    <link name="plate_1_link">
+      <inertial>
+        <mass value="12" />
+        <origin xyz="0 0 0" />
+        <inertia ixx="1.0" ixy="0.0" ixz="0.0"
+                 iyy="1.0" iyz="0.0"
+                 izz="1.0" />
+      </inertial>
+      <visual>
+        <origin xyz=" 0 0 0 " rpy="0 0 0" />
+        <geometry>
+          <mesh filename="package://turtlebot_urdf/meshes/Turtlebot_Plate_1_Logo.dae" scale="${M_SCALE} ${M_SCALE} ${M_SCALE}"/>
+        </geometry>
+      </visual>
+      <collision>
+        <origin xyz="0.0 0.0 0.0" rpy="0 0 0" />
+        <geometry>
+          <mesh filename="package://turtlebot_urdf/meshes/Turtlebot_Plate_1_Logo.dae"/>
+        </geometry>
+      </collision>
+    </link>
+    <turtlebot_standoff_2in parent="standoff_1in_0_link" number="0" x_loc="0" y_loc="0" z_loc="0.0318008"/>
+    <turtlebot_standoff_2in parent="standoff_1in_1_link" number="1" x_loc="0" y_loc="0" z_loc="0.0318008"/>
+    <turtlebot_standoff_2in parent="standoff_1in_2_link" number="2" x_loc="0" y_loc="0" z_loc="0.0318008"/>
+    <turtlebot_standoff_2in parent="standoff_1in_3_link" number="3" x_loc="0" y_loc="0" z_loc="0.0318008"/>
+    <joint name="plate_2_joint" type="fixed">
+      <origin xyz="0 0 0.0572008" rpy="0 0 0" />
+      <parent link="plate_1_link"/>
+      <child link="plate_2_link" />
+    </joint>
+    <link name="plate_2_link">
+      <inertial>
+        <mass value="12" />
+        <origin xyz="0 0 0" />
+        <inertia ixx="1.0" ixy="0.0" ixz="0.0"
+                 iyy="1.0" iyz="0.0"
+                 izz="1.0" />
+      </inertial>
+      <visual>
+        <origin xyz=" 0 0 0 " rpy="0 0 0" />
+        <geometry>
+          <mesh filename="package://turtlebot_urdf/meshes/Turtlebot_Plate_1_Logo.dae" scale="${M_SCALE} ${M_SCALE} ${M_SCALE}"/>
+        </geometry>
+      </visual>
+      <collision>
+        <origin xyz="0.0 0.0 0.0" rpy="0 0 0" />
+        <geometry>
+          <mesh filename="package://turtlebot_urdf/meshes/Turtlebot_Plate_1_Logo.dae"/>
+        </geometry>
+      </collision>
+    </link>
   </macro>
 </robot>

File: turtlebot_urdf/urdf/turtlebot_hardware.xacro (robot description, xacro)
@@ -3,8 +3,8 @@
   <property name="M_PI" value="3.14159"/>
   <property name="M_SCALE" value="0.001"/>
-  <macro name="turtlebot_spacer" params="number x_loc y_loc z_loc">
+  <macro name="turtlebot_spacer" params="parent number x_loc y_loc z_loc">
     <joint name="spacer_${number}_joint" type="fixed">
       <origin xyz="${x_loc} ${y_loc} ${z_loc}" rpy="0 0 0" />
-      <parent link="base_link"/>
+      <parent link="${parent}"/>
       <child link="spacer_${number}_link" />
     </joint>
@@ -31,8 +31,8 @@
     </link>
   </macro>
-  <macro name="turtlebot_standoff_1in" params="number x_loc y_loc z_loc">
+  <macro name="turtlebot_standoff_1in" params="parent number x_loc y_loc z_loc">
     <joint name="standoff_1in_${number}_joint" type="fixed">
       <origin xyz="${x_loc} ${y_loc} ${z_loc}" rpy="0 0 0" />
-      <parent link="base_link"/>
+      <parent link="${parent}"/>
       <child link="standoff_1in_${number}_link" />
     </joint>
@@ -59,3 +59,31 @@
     </link>
   </macro>
+  <macro name="turtlebot_standoff_2in" params="parent number x_loc y_loc z_loc">
+    <joint name="standoff_2in_${number}_joint" type="fixed">
+      <origin xyz="${x_loc} ${y_loc} ${z_loc}" rpy="0 0 0" />
+      <parent link="${parent}"/>
+      <child link="standoff_2in_${number}_link" />
+    </joint>
+    <link name="standoff_2in_${number}_link">
+      <inertial>
+	<mass value="1" />
+	<origin xyz="0 0 0" />
+	<inertia ixx="1.0" ixy="0.0" ixz="0.0"
+		 iyy="1.0" iyz="0.0"
+		 izz="1.0" />
+      </inertial>
+      <visual>
+	<origin xyz=" 0 0 0 " rpy="0 0 0" />
+	<geometry>
+	  <mesh filename="package://turtlebot_urdf/meshes/68-04552-2000-RA_Turtlebot_M-F_Standoff.dae" scale="${M_SCALE} ${M_SCALE} ${M_SCALE}"/>
+	</geometry>
+      </visual>
+      <collision>
+	<origin xyz="0.0 0.0 0.0" rpy="0 0 0" />
+	<geometry>
+	  <mesh filename="package://turtlebot_urdf/meshes/68-04552-2000-RA_Turtlebot_M-F_Standoff.dae"/>
+	</geometry>
+      </collision>
+    </link>
+  </macro>
 </robot>

Commit message: first pass.. ned to fix the top plate and add the kinect but looks good

File: turtlebot_urdf/urdf/turtlebot.xacro (robot description, xacro)
@@ -122,4 +122,34 @@
       </collision>
     </link>
+    <turtlebot_standoff_8in parent="standoff_2in_0_link" number="0" x_loc="0" y_loc="0" z_loc="0.05715"/>
+    <turtlebot_standoff_8in parent="standoff_2in_1_link" number="1" x_loc="0" y_loc="0" z_loc="0.05715"/>
+    <turtlebot_standoff_8in parent="standoff_2in_2_link" number="2" x_loc="0" y_loc="0" z_loc="0.05715"/>
+    <turtlebot_standoff_8in parent="standoff_2in_3_link" number="3" x_loc="0" y_loc="0" z_loc="0.05715"/>
+    <joint name="plate_3_joint" type="fixed">
+      <origin xyz="-0.01316 0 0.20955" rpy="0 0 0" />
+      <parent link="plate_2_link"/>
+      <child link="plate_3_link" />
+    </joint>
+    <link name="plate_3_link">
+      <inertial>
+        <mass value="12" />
+        <origin xyz="0 0 0" />
+        <inertia ixx="1.0" ixy="0.0" ixz="0.0"
+                 iyy="1.0" iyz="0.0"
+                 izz="1.0" />
+      </inertial>
+      <visual>
+        <origin xyz=" 0 0 0 " rpy="0 0 0" />
+        <geometry>
+          <mesh filename="package://turtlebot_urdf/meshes/Turtlebot_Plate_2_Logo.dae" scale="${M_SCALE} ${M_SCALE} ${M_SCALE}"/>
+        </geometry>
+      </visual>
+      <collision>
+        <origin xyz="0.0 0.0 0.0" rpy="0 0 0" />
+        <geometry>
+          <mesh filename="package://turtlebot_urdf/meshes/Turtlebot_Plate_2_Logo.dae"/>
+        </geometry>
+      </collision>
+    </link>
   </macro>
 </robot>

File: turtlebot_urdf/urdf/turtlebot_hardware.xacro (robot description, xacro)
@@ -87,3 +87,31 @@
     </link>
   </macro>
+  <macro name="turtlebot_standoff_8in" params="parent number x_loc y_loc z_loc">
+    <joint name="standoff_8in_${number}_joint" type="fixed">
+      <origin xyz="${x_loc} ${y_loc} ${z_loc}" rpy="0 0 0" />
+      <parent link="${parent}"/>
+      <child link="standoff_8in_${number}_link" />
+    </joint>
+    <link name="standoff_8in_${number}_link">
+      <inertial>
+	<mass value="1" />
+	<origin xyz="0 0 0" />
+	<inertia ixx="1.0" ixy="0.0" ixz="0.0"
+		 iyy="1.0" iyz="0.0"
+		 izz="1.0" />
+      </inertial>
+      <visual>
+	<origin xyz=" 0 0 0 " rpy="0 0 0" />
+	<geometry>
+	  <mesh filename="package://turtlebot_urdf/meshes/68-02421-8000-RA_Turtlebot_F-F_Standoff.dae" scale="${M_SCALE} ${M_SCALE} ${M_SCALE}"/>
+	</geometry>
+      </visual>
+      <collision>
+	<origin xyz="0.0 0.0 0.0" rpy="0 0 0" />
+	<geometry>
+	  <mesh filename="package://turtlebot_urdf/meshes/68-02421-8000-RA_Turtlebot_F-F_Standoff.dae"/>
+	</geometry>
+      </collision>
+    </link>
+  </macro>
 </robot>

Commit message: adding new mesh

File: turtlebot_urdf/urdf/turtlebot.xacro (robot description, xacro)
@@ -37,5 +37,5 @@
     <turtlebot_spacer parent="base_link" number="3" x_loc="-0.07239" y_loc="0.1114679" z_loc="0.062992"/>
     <joint name="plate_0_joint" type="fixed">
-      <origin xyz="-0.04334 0  0.0645795" rpy="0 0 0" />
+      <origin xyz="-0.04334 0  0.06775704" rpy="0 0 0" />
       <parent link="base_link"/>
       <child link="plate_0_link" />
@@ -52,5 +52,5 @@
         <origin xyz=" 0 0 0 " rpy="0 0 0" />
         <geometry>
-          <mesh filename="package://turtlebot_urdf/meshes/Turtlebot_Plate_0_Logo.dae" scale="${M_SCALE} ${M_SCALE} ${M_SCALE}"/>
+          <mesh filename="package://turtlebot_urdf/meshes/plate_0_logo.dae" scale="${M_SCALE} ${M_SCALE} ${M_SCALE}"/>
         </geometry>
       </visual>
@@ -58,5 +58,5 @@
         <origin xyz="0.0 0.0 0.0" rpy="0 0 0" />
         <geometry>
-          <mesh filename="package://turtlebot_urdf/meshes/Turtlebot_Plate_0_Logo.dae"/>
+          <mesh filename="package://turtlebot_urdf/meshes/plate_0_logo.dae"/>
         </geometry>
       </collision>
@@ -82,5 +82,5 @@
         <origin xyz=" 0 0 0 " rpy="0 0 0" />
         <geometry>
-          <mesh filename="package://turtlebot_urdf/meshes/Turtlebot_Plate_1_Logo.dae" scale="${M_SCALE} ${M_SCALE} ${M_SCALE}"/>
+          <mesh filename="package://turtlebot_urdf/meshes/plate_1_logo.dae" scale="${M_SCALE} ${M_SCALE} ${M_SCALE}"/>
         </geometry>
       </visual>
@@ -88,5 +88,5 @@
         <origin xyz="0.0 0.0 0.0" rpy="0 0 0" />
         <geometry>
-          <mesh filename="package://turtlebot_urdf/meshes/Turtlebot_Plate_1_Logo.dae"/>
+          <mesh filename="package://turtlebot_urdf/meshes/plate_1_logo.dae"/>
         </geometry>
       </collision>
@@ -112,5 +112,5 @@
         <origin xyz=" 0 0 0 " rpy="0 0 0" />
         <geometry>
-          <mesh filename="package://turtlebot_urdf/meshes/Turtlebot_Plate_1_Logo.dae" scale="${M_SCALE} ${M_SCALE} ${M_SCALE}"/>
+          <mesh filename="package://turtlebot_urdf/meshes/plate_1_logo.dae" scale="${M_SCALE} ${M_SCALE} ${M_SCALE}"/>
         </geometry>
       </visual>
@@ -118,5 +118,5 @@
         <origin xyz="0.0 0.0 0.0" rpy="0 0 0" />
         <geometry>
-          <mesh filename="package://turtlebot_urdf/meshes/Turtlebot_Plate_1_Logo.dae"/>
+          <mesh filename="package://turtlebot_urdf/meshes/plate_1_logo.dae"/>
         </geometry>
       </collision>
@@ -142,5 +142,5 @@
         <origin xyz=" 0 0 0 " rpy="0 0 0" />
         <geometry>
-          <mesh filename="package://turtlebot_urdf/meshes/Turtlebot_Plate_2_Logo.dae" scale="${M_SCALE} ${M_SCALE} ${M_SCALE}"/>
+          <mesh filename="package://turtlebot_urdf/meshes/plate_2_logo.dae" scale="${M_SCALE} ${M_SCALE} ${M_SCALE}"/>
         </geometry>
       </visual>
@@ -148,5 +148,5 @@
         <origin xyz="0.0 0.0 0.0" rpy="0 0 0" />
         <geometry>
-          <mesh filename="package://turtlebot_urdf/meshes/Turtlebot_Plate_2_Logo.dae"/>
+          <mesh filename="package://turtlebot_urdf/meshes/plate_2_logo.dae"/>
         </geometry>
       </collision>

Commit message: adding final touches

File: turtlebot_urdf/urdf/turtlebot.xacro (robot description, xacro)
@@ -2,6 +2,6 @@
 <robot>
   <include filename="$(find turtlebot_urdf)/urdf/turtlebot_hardware.xacro" />
-  <material name="Blue">
-    <color rgba="0.0 0.0 0.8 1.0"/>
+  <material name="Green">
+    <color rgba="0.0 0.8 0.0 1.0"/>
   </material>
   <property name="M_PI" value="3.14159"/>
@@ -36,4 +36,24 @@
     <turtlebot_spacer parent="base_link" number="2" x_loc="-0.07239" y_loc="-0.1114679" z_loc="0.062992"/>
     <turtlebot_spacer parent="base_link" number="3" x_loc="-0.07239" y_loc="0.1114679" z_loc="0.062992"/>
+    <joint name="gyro_joint" type="fixed">
+      <origin xyz="0 0 0.04" rpy="0 0 0" />
+      <parent link="base_link" />
+      <child link="gyro_link" />
+    </joint>
+    <link name="gyro_link">
+      <visual>
+        <geometry>
+          <box size="0.02 0.035 0.002" />
+        </geometry>
+        <material name="Green" />
+      </visual>
+      <inertial>
+        <mass value="0.0001" />
+        <origin xyz="0 0 0" />
+        <inertia ixx="0.0001" ixy="0.0" ixz="0.0"
+                 iyy="0.0001" iyz="0.0"
+                 izz="0.0001" />
+      </inertial>
+    </link>
     <joint name="plate_0_joint" type="fixed">
       <origin xyz="-0.04334 0  0.06775704" rpy="0 0 0" />
@@ -122,4 +142,88 @@
       </collision>
     </link>
+    <joint name="base_kinect_joint" type="fixed">
+      <origin xyz="-0.0844382 0 0.1047496" rpy="0 0 0" />
+      <parent link="plate_2_link" />
+      <child link="kinect_link" />
+    </joint>
+    <link name="kinect_link">
+      <inertial>
+        <mass value="12" />
+        <origin xyz="0 0 0" />
+        <inertia ixx="1.0" ixy="0.0" ixz="0.0"
+                 iyy="1.0" iyz="0.0"
+                 izz="1.0" />
+      </inertial>
+      <visual>
+        <origin xyz=" 0 0 0 " rpy="0 0 0" />
+        <geometry>
+          <mesh filename="package://turtlebot_urdf/meshes/68-04546_Kinect_Sensor.3ds" scale="${M_SCALE} ${M_SCALE} ${M_SCALE}"/>
+        </geometry>
+      </visual>
+      <collision>
+        <origin xyz="0.0 0.0 0.0" rpy="0 0 0" />
+        <geometry>
+          <mesh filename="package://turtlebot_urdf/meshes/68-04546_Kinect_Sensor.3ds"/>
+          </geometry>
+      </collision>
+    </link>
+    <joint name="kinect_depth_joint" type="fixed">
+      <origin xyz="0 0.018 0" rpy="0 0 0" />
+      <parent link="kinect_link" />
+      <child link="kinect_depth_frame" />
+    </joint>
+    <link name="kinect_depth_frame">
+      <inertial>
+        <mass value="0.0001" />
+        <origin xyz="0 0 0" />
+        <inertia ixx="0.0001" ixy="0.0" ixz="0.0"
+                 iyy="0.0001" iyz="0.0"
+                 izz="0.0001" />
+      </inertial>
+    </link>
+    <joint name="kinect_depth_optical_joint" type="fixed">
+      <origin xyz="0 0 0" rpy="${-M_PI/2} 0 ${-M_PI/2}" />
+      <parent link="kinect_depth_frame" />
+      <child link="kinect_depth_optical_frame" />
+    </joint>
+    <link name="kinect_depth_optical_frame">
+      <inertial>
+        <mass value="0.0001" />
+        <origin xyz="0 0 0" />
+        <inertia ixx="0.0001" ixy="0.0" ixz="0.0"
+                 iyy="0.0001" iyz="0.0"
+                 izz="0.0001" />
+      </inertial>
+    </link>
+    <joint name="kinect_rgb_joint" type="fixed">
+      <origin xyz="0 -0.005 0" rpy="0 0 0" />
+      <parent link="kinect_link" />
+      <child link="kinect_rgb_frame" />
+    </joint>
+    <link name="kinect_rgb_frame">
+      <inertial>
+        <mass value="0.0001" />
+        <origin xyz="0 0 0" />
+        <inertia ixx="0.0001" ixy="0.0" ixz="0.0"
+                 iyy="0.0001" iyz="0.0"
+                 izz="0.0001" />
+      </inertial>
+    </link>
+    <joint name="kinect_rgb_optical_joint" type="fixed">
+      <origin xyz="0 0 0" rpy="${-M_PI/2} 0 ${-M_PI/2}" />
+      <parent link="kinect_rgb_frame" />
+      <child link="kinect_rgb_optical_frame" />
+    </joint>
+    <link name="kinect_rgb_optical_frame">
+      <inertial>
+        <mass value="0.0001" />
+        <origin xyz="0 0 0" />
+        <inertia ixx="0.0001" ixy="0.0" ixz="0.0"
+                 iyy="0.0001" iyz="0.0"
+                 izz="0.0001" />
+      </inertial>
+    </link>
+    <turtlebot_standoff_kinect parent="plate_2_link" number="0" x_loc="-0.1024382" y_loc="0.098" z_loc="0.0032004"/>
+    <turtlebot_standoff_kinect parent="plate_2_link" number="1" x_loc="-0.1024382" y_loc="-0.098" z_loc="0.0032004"/>
     <turtlebot_standoff_8in parent="standoff_2in_0_link" number="0" x_loc="0" y_loc="0" z_loc="0.05715"/>
     <turtlebot_standoff_8in parent="standoff_2in_1_link" number="1" x_loc="0" y_loc="0" z_loc="0.05715"/>
@@ -127,5 +231,5 @@
     <turtlebot_standoff_8in parent="standoff_2in_3_link" number="3" x_loc="0" y_loc="0" z_loc="0.05715"/>
     <joint name="plate_3_joint" type="fixed">
-      <origin xyz="-0.01316 0 0.20955" rpy="0 0 0" />
+      <origin xyz="-0.01316 0 0.2063496" rpy="0 0 0" />
       <parent link="plate_2_link"/>
       <child link="plate_3_link" />

File: turtlebot_urdf/urdf/turtlebot_hardware.xacro (robot description, xacro)
@@ -115,3 +115,31 @@
     </link>
   </macro>
+  <macro name="turtlebot_standoff_kinect" params="parent number x_loc y_loc z_loc">
+    <joint name="standoff_kinect_${number}_joint" type="fixed">
+      <origin xyz="${x_loc} ${y_loc} ${z_loc}" rpy="0 0 0" />
+      <parent link="${parent}"/>
+      <child link="standoff_kinect_${number}_link" />
+    </joint>
+    <link name="standoff_kinect_${number}_link">
+      <inertial>
+	<mass value="1" />
+	<origin xyz="0 0 0" />
+	<inertia ixx="1.0" ixy="0.0" ixz="0.0"
+		 iyy="1.0" iyz="0.0"
+		 izz="1.0" />
+      </inertial>
+      <visual>
+	<origin xyz=" 0 0 0 " rpy="0 0 0" />
+	<geometry>
+	  <mesh filename="package://turtlebot_urdf/meshes/68-04556-RA_Kinect_Standoff_Assy.3ds" scale="${M_SCALE} ${M_SCALE} ${M_SCALE}"/>
+	</geometry>
+      </visual>
+      <collision>
+	<origin xyz="0.0 0.0 0.0" rpy="0 0 0" />
+	<geometry>
+	  <mesh filename="package://turtlebot_urdf/meshes/68-04556-RA_Kinect_Standoff_Assy.3ds"/>
+	</geometry>
+      </collision>
+    </link>
+  </macro>
 </robot>
