Commit message: search and replace on urdf

File: turtlebot_description/urdf/turtlebot.urdf.xacro (robot description, xacro)
@@ -5,5 +5,5 @@
     xmlns:interface="http://playerstage.sourceforge.net/gazebo/xmlschema/#interface">
     <!-- Included URDF Files -->
-    <include filename="$(find turtlebot_urdf)/urdf/turtlebot.xacro" />
+    <include filename="$(find turtlebot_description)/urdf/turtlebot.xacro" />
     <turtlebot />
 </robot>

File: turtlebot_description/urdf/turtlebot.xacro (robot description, xacro)
@@ -1,5 +1,5 @@
 <?xml version="1.0"?>
 <robot>
-  <include filename="$(find turtlebot_urdf)/urdf/turtlebot_hardware.xacro" />
+  <include filename="$(find turtlebot_description)/urdf/turtlebot_hardware.xacro" />
   <material name="Green">
     <color rgba="0.0 0.8 0.0 1.0"/>
@@ -53,11 +53,11 @@
         <origin xyz=" 0 0 0 " rpy="0 0 0" />
         <geometry>
-          <mesh filename="package://turtlebot_urdf/meshes/68-04545_iRobot_Create.dae" scale="${SCALE} ${SCALE} ${SCALE}"/>
-        </geometry>
-      </visual>
-      <collision>
-        <origin xyz="0.0 0.0 0.0" rpy="0 0 0" />
-        <geometry>
-          <mesh filename="package://turtlebot_urdf/meshes/68-04545_iRobot_Create.STL"/>
+          <mesh filename="package://turtlebot_description/meshes/68-04545_iRobot_Create.dae" scale="${SCALE} ${SCALE} ${SCALE}"/>
+        </geometry>
+      </visual>
+      <collision>
+        <origin xyz="0.0 0.0 0.0" rpy="0 0 0" />
+        <geometry>
+          <mesh filename="package://turtlebot_description/meshes/68-04545_iRobot_Create.STL"/>
         </geometry>
       </collision>
@@ -103,11 +103,11 @@
         <origin xyz=" 0 0 0 " rpy="0 0 0" />
         <geometry>
-          <mesh filename="package://turtlebot_urdf/meshes/plate_0_logo.dae" scale="${M_SCALE} ${M_SCALE} ${M_SCALE}"/>
-        </geometry>
-      </visual>
-      <collision>
-        <origin xyz="0.0 0.0 0.0" rpy="0 0 0" />
-        <geometry>
-          <mesh filename="package://turtlebot_urdf/meshes/plate_0_logo.dae"/>
+          <mesh filename="package://turtlebot_description/meshes/plate_0_logo.dae" scale="${M_SCALE} ${M_SCALE} ${M_SCALE}"/>
+        </geometry>
+      </visual>
+      <collision>
+        <origin xyz="0.0 0.0 0.0" rpy="0 0 0" />
+        <geometry>
+          <mesh filename="package://turtlebot_description/meshes/plate_0_logo.dae"/>
         </geometry>
       </collision>
@@ -133,11 +133,11 @@
         <origin xyz=" 0 0 0 " rpy="0 0 0" />
         <geometry>
-          <mesh filename="package://turtlebot_urdf/meshes/plate_1_logo.dae" scale="${M_SCALE} ${M_SCALE} ${M_SCALE}"/>
-        </geometry>
-      </visual>
-      <collision>
-        <origin xyz="0.0 0.0 0.0" rpy="0 0 0" />
-        <geometry>
-          <mesh filename="package://turtlebot_urdf/meshes/plate_1_logo.dae"/>
+          <mesh filename="package://turtlebot_description/meshes/plate_1_logo.dae" scale="${M_SCALE} ${M_SCALE} ${M_SCALE}"/>
+        </geometry>
+      </visual>
+      <collision>
+        <origin xyz="0.0 0.0 0.0" rpy="0 0 0" />
+        <geometry>
+          <mesh filename="package://turtlebot_description/meshes/plate_1_logo.dae"/>
         </geometry>
       </collision>
@@ -163,11 +163,11 @@
         <origin xyz=" 0 0 0 " rpy="0 0 0" />
         <geometry>
-          <mesh filename="package://turtlebot_urdf/meshes/plate_1_logo.dae" scale="${M_SCALE} ${M_SCALE} ${M_SCALE}"/>
-        </geometry>
-      </visual>
-      <collision>
-        <origin xyz="0.0 0.0 0.0" rpy="0 0 0" />
-        <geometry>
-          <mesh filename="package://turtlebot_urdf/meshes/plate_1_logo.dae"/>
+          <mesh filename="package://turtlebot_description/meshes/plate_1_logo.dae" scale="${M_SCALE} ${M_SCALE} ${M_SCALE}"/>
+        </geometry>
+      </visual>
+      <collision>
+        <origin xyz="0.0 0.0 0.0" rpy="0 0 0" />
+        <geometry>
+          <mesh filename="package://turtlebot_description/meshes/plate_1_logo.dae"/>
         </geometry>
       </collision>
@@ -189,11 +189,11 @@
         <origin xyz=" 0 0 0 " rpy="0 0 0" />
         <geometry>
-          <mesh filename="package://turtlebot_urdf/meshes/68-04546_Kinect_Sensor.3ds" scale="${M_SCALE} ${M_SCALE} ${M_SCALE}"/>
-        </geometry>
-      </visual>
-      <collision>
-        <origin xyz="0.0 0.0 0.0" rpy="0 0 0" />
-        <geometry>
-          <mesh filename="package://turtlebot_urdf/meshes/68-04546_Kinect_Sensor.3ds"/>
+          <mesh filename="package://turtlebot_description/meshes/68-04546_Kinect_Sensor.3ds" scale="${M_SCALE} ${M_SCALE} ${M_SCALE}"/>
+        </geometry>
+      </visual>
+      <collision>
+        <origin xyz="0.0 0.0 0.0" rpy="0 0 0" />
+        <geometry>
+          <mesh filename="package://turtlebot_description/meshes/68-04546_Kinect_Sensor.3ds"/>
           </geometry>
       </collision>
@@ -277,11 +277,11 @@
         <origin xyz=" 0 0 0 " rpy="0 0 0" />
         <geometry>
-          <mesh filename="package://turtlebot_urdf/meshes/plate_2_logo.dae" scale="${M_SCALE} ${M_SCALE} ${M_SCALE}"/>
-        </geometry>
-      </visual>
-      <collision>
-        <origin xyz="0.0 0.0 0.0" rpy="0 0 0" />
-        <geometry>
-          <mesh filename="package://turtlebot_urdf/meshes/plate_2_logo.dae"/>
+          <mesh filename="package://turtlebot_description/meshes/plate_2_logo.dae" scale="${M_SCALE} ${M_SCALE} ${M_SCALE}"/>
+        </geometry>
+      </visual>
+      <collision>
+        <origin xyz="0.0 0.0 0.0" rpy="0 0 0" />
+        <geometry>
+          <mesh filename="package://turtlebot_description/meshes/plate_2_logo.dae"/>
         </geometry>
       </collision>

File: turtlebot_description/urdf/turtlebot_hardware.xacro (robot description, xacro)
@@ -20,5 +20,5 @@
 	<origin xyz=" 0 0 0 " rpy="0 0 0" />
 	<geometry>
-	  <mesh filename="package://turtlebot_urdf/meshes/68-02403-125_Spacer.dae" scale="${M_SCALE} ${M_SCALE} ${M_SCALE}"/>
+	  <mesh filename="package://turtlebot_description/meshes/68-02403-125_Spacer.dae" scale="${M_SCALE} ${M_SCALE} ${M_SCALE}"/>
 	</geometry>
       </visual>
@@ -26,5 +26,5 @@
 	<origin xyz="0.0 0.0 0.0" rpy="0 0 0" />
 	<geometry>
-	  <mesh filename="package://turtlebot_urdf/meshes/68-02403-125_Spacer.dae"/>
+	  <mesh filename="package://turtlebot_description/meshes/68-02403-125_Spacer.dae"/>
 	</geometry>
       </collision>
@@ -48,5 +48,5 @@
 	<origin xyz=" 0 0 0 " rpy="0 0 0" />
 	<geometry>
-	  <mesh filename="package://turtlebot_urdf/meshes/68-04552-1000-RA_Turtlebot_M-F_Standoff.dae" scale="${M_SCALE} ${M_SCALE} ${M_SCALE}"/>
+	  <mesh filename="package://turtlebot_description/meshes/68-04552-1000-RA_Turtlebot_M-F_Standoff.dae" scale="${M_SCALE} ${M_SCALE} ${M_SCALE}"/>
 	</geometry>
       </visual>
@@ -54,5 +54,5 @@
 	<origin xyz="0.0 0.0 0.0" rpy="0 0 0" />
 	<geometry>
-	  <mesh filename="package://turtlebot_urdf/meshes/68-04552-1000-RA_Turtlebot_M-F_Standoff.dae"/>
+	  <mesh filename="package://turtlebot_description/meshes/68-04552-1000-RA_Turtlebot_M-F_Standoff.dae"/>
 	</geometry>
       </collision>
@@ -76,5 +76,5 @@
 	<origin xyz=" 0 0 0 " rpy="0 0 0" />
 	<geometry>
-	  <mesh filename="package://turtlebot_urdf/meshes/68-04552-2000-RA_Turtlebot_M-F_Standoff.dae" scale="${M_SCALE} ${M_SCALE} ${M_SCALE}"/>
+	  <mesh filename="package://turtlebot_description/meshes/68-04552-2000-RA_Turtlebot_M-F_Standoff.dae" scale="${M_SCALE} ${M_SCALE} ${M_SCALE}"/>
 	</geometry>
       </visual>
@@ -82,5 +82,5 @@
 	<origin xyz="0.0 0.0 0.0" rpy="0 0 0" />
 	<geometry>
-	  <mesh filename="package://turtlebot_urdf/meshes/68-04552-2000-RA_Turtlebot_M-F_Standoff.dae"/>
+	  <mesh filename="package://turtlebot_description/meshes/68-04552-2000-RA_Turtlebot_M-F_Standoff.dae"/>
 	</geometry>
       </collision>
@@ -104,5 +104,5 @@
 	<origin xyz=" 0 0 0 " rpy="0 0 0" />
 	<geometry>
-	  <mesh filename="package://turtlebot_urdf/meshes/68-02421-8000-RA_Turtlebot_F-F_Standoff.dae" scale="${M_SCALE} ${M_SCALE} ${M_SCALE}"/>
+	  <mesh filename="package://turtlebot_description/meshes/68-02421-8000-RA_Turtlebot_F-F_Standoff.dae" scale="${M_SCALE} ${M_SCALE} ${M_SCALE}"/>
 	</geometry>
       </visual>
@@ -110,5 +110,5 @@
 	<origin xyz="0.0 0.0 0.0" rpy="0 0 0" />
 	<geometry>
-	  <mesh filename="package://turtlebot_urdf/meshes/68-02421-8000-RA_Turtlebot_F-F_Standoff.dae"/>
+	  <mesh filename="package://turtlebot_description/meshes/68-02421-8000-RA_Turtlebot_F-F_Standoff.dae"/>
 	</geometry>
       </collision>
@@ -132,5 +132,5 @@
 	<origin xyz=" 0 0 0 " rpy="0 0 0" />
 	<geometry>
-	  <mesh filename="package://turtlebot_urdf/meshes/68-04556-RA_Kinect_Standoff_Assy.3ds" scale="${M_SCALE} ${M_SCALE} ${M_SCALE}"/>
+	  <mesh filename="package://turtlebot_description/meshes/68-04556-RA_Kinect_Standoff_Assy.3ds" scale="${M_SCALE} ${M_SCALE} ${M_SCALE}"/>
 	</geometry>
       </visual>
@@ -138,5 +138,5 @@
 	<origin xyz="0.0 0.0 0.0" rpy="0 0 0" />
 	<geometry>
-	  <mesh filename="package://turtlebot_urdf/meshes/68-04556-RA_Kinect_Standoff_Assy.3ds"/>
+	  <mesh filename="package://turtlebot_description/meshes/68-04556-RA_Kinect_Standoff_Assy.3ds"/>
 	</geometry>
       </collision>
