Commit message: Fixed up the robot urdf and meshes

File: turtlebot_description/urdf/turtlebot.xacro (robot description, xacro)
@@ -2,4 +2,5 @@
 <robot>
   <include filename="$(find turtlebot_description)/urdf/turtlebot_hardware.xacro" />
+  <include filename="$(find turtlebot_description)/urdf/gazebo.urdf.xacro"/>
   <material name="Green">
     <color rgba="0.0 0.8 0.0 1.0"/>
@@ -7,284 +8,384 @@
   <property name="M_PI" value="3.14159"/>
   <property name="SCALE" value="0.0254"/>
-  <property name="M_SCALE" value="0.001"/>
   <property name="base_x" value="0.33" />
   <property name="base_y" value="0.33" />
   <macro name="turtlebot">
-        <!-- base_footprint is a fictitious link(frame) that is on the ground right below base_link origin,
-             navigation stack depends on this frame -->
-        <link name="base_footprint">
-            <inertial>
-                <mass value="0.0001" />
-                <origin xyz="0 0 0" />
-                <inertia ixx="0.0001" ixy="0.0" ixz="0.0"
-                         iyy="0.0001" iyz="0.0"
-                         izz="0.0001" />
-            </inertial>
-            <visual>
-                <origin xyz="0 0 0" rpy="0 0 0" />
-                <geometry>
-                    <box size="0.001 0.001 0.001" />
-                </geometry>
-                <material name="Green" />
-            </visual>
-            <collision>
-                <origin xyz="0 0 0.017" rpy="0 0 0" />
-                <geometry>
-                  <box size="0.001 0.001 0.001" />
-                </geometry>
-            </collision>
-        </link>
-        <joint name="base_footprint_joint" type="fixed">
-            <!-- NB: While you would think this would make it go up, it is oddly reversed.
-                 This moves the joint to 0,0,0 where we want it for rviz, etc. -->
-            <origin xyz="0 0 0.017" rpy="0 0 0" />
-            <parent link="base_footprint"/>
-            <child link="base_link" />
-        </joint>
-    <link name="base_link">
-      <inertial>
-        <mass value="12" />
-        <origin xyz="0 0 0.017" />
-        <inertia ixx="1.0" ixy="0.0" ixz="0.0"
-                 iyy="1.0" iyz="0.0"
-                 izz="1.0" />
-      </inertial>
-      <visual>
-        <origin xyz=" 0 0 0 " rpy="0 0 0" />
-        <geometry>
-          <mesh filename="package://turtlebot_description/meshes/68-04545_iRobot_Create.dae" scale="${SCALE} ${SCALE} ${SCALE}"/>
-        </geometry>
-      </visual>
-      <collision>
-        <origin xyz="0.0 0.0 0.0" rpy="0 0 0" />
-        <geometry>
-          <mesh filename="package://turtlebot_description/meshes/68-04545_iRobot_Create.STL"/>
-        </geometry>
-      </collision>
-    </link>
-    <turtlebot_spacer parent="base_link" number="0" x_loc="-0.00254" y_loc="0.1114679" z_loc="0.062992"/>
-    <turtlebot_spacer parent="base_link" number="1" x_loc="-0.00254" y_loc="-0.1114679" z_loc="0.062992"/>
-    <turtlebot_spacer parent="base_link" number="2" x_loc="-0.07239" y_loc="-0.1114679" z_loc="0.062992"/>
-    <turtlebot_spacer parent="base_link" number="3" x_loc="-0.07239" y_loc="0.1114679" z_loc="0.062992"/>
-    <joint name="gyro_joint" type="fixed">
-      <origin xyz="0 0 0.04" rpy="0 0 0" />
-      <parent link="base_link" />
-      <child link="gyro_link" />
-    </joint>
-    <link name="gyro_link">
-      <visual>
-        <geometry>
-          <box size="0.02 0.035 0.002" />
-        </geometry>
-        <material name="Green" />
-      </visual>
-      <inertial>
-        <mass value="0.0001" />
-        <origin xyz="0 0 0" />
-        <inertia ixx="0.0001" ixy="0.0" ixz="0.0"
-                 iyy="0.0001" iyz="0.0"
-                 izz="0.0001" />
-      </inertial>
-    </link>
-    <joint name="plate_0_joint" type="fixed">
-      <origin xyz="-0.04334 0  0.06775704" rpy="0 0 0" />
-      <parent link="base_link"/>
-      <child link="plate_0_link" />
-    </joint>
-    <link name="plate_0_link">
-      <inertial>
-        <mass value="12" />
-        <origin xyz="0 0 0" />
-        <inertia ixx="1.0" ixy="0.0" ixz="0.0"
-                 iyy="1.0" iyz="0.0"
-                 izz="1.0" />
-      </inertial>
-      <visual>
-        <origin xyz=" 0 0 0 " rpy="0 0 0" />
-        <geometry>
-          <mesh filename="package://turtlebot_description/meshes/plate_0_logo.dae" scale="${M_SCALE} ${M_SCALE} ${M_SCALE}"/>
-        </geometry>
-      </visual>
-      <collision>
-        <origin xyz="0.0 0.0 0.0" rpy="0 0 0" />
-        <geometry>
-          <mesh filename="package://turtlebot_description/meshes/plate_0_logo.dae"/>
-        </geometry>
-      </collision>
-    </link>
-    <turtlebot_standoff_1in parent="base_link" number="0" x_loc="0.0676402" y_loc="0.1314196" z_loc="0.0709803"/>
-    <turtlebot_standoff_1in parent="base_link" number="1" x_loc="0.0676402" y_loc="-0.1314196" z_loc="0.0709803"/>
-    <turtlebot_standoff_1in parent="base_link" number="2" x_loc="-0.052832" y_loc="-0.1314196" z_loc="0.0709803"/>
-    <turtlebot_standoff_1in parent="base_link" number="3" x_loc="-0.052832" y_loc="0.1314196" z_loc="0.0709803"/>
-    <joint name="plate_1_joint" type="fixed">
-      <origin xyz="0.04068 0 0.0318008" rpy="0 0 0" />
-      <parent link="plate_0_link"/>
-      <child link="plate_1_link" />
-    </joint>
-    <link name="plate_1_link">
-      <inertial>
-        <mass value="12" />
-        <origin xyz="0 0 0" />
-        <inertia ixx="1.0" ixy="0.0" ixz="0.0"
-                 iyy="1.0" iyz="0.0"
-                 izz="1.0" />
-      </inertial>
-      <visual>
-        <origin xyz=" 0 0 0 " rpy="0 0 0" />
-        <geometry>
-          <mesh filename="package://turtlebot_description/meshes/plate_1_logo.dae" scale="${M_SCALE} ${M_SCALE} ${M_SCALE}"/>
-        </geometry>
-      </visual>
-      <collision>
-        <origin xyz="0.0 0.0 0.0" rpy="0 0 0" />
-        <geometry>
-          <mesh filename="package://turtlebot_description/meshes/plate_1_logo.dae"/>
-        </geometry>
-      </collision>
-    </link>
-    <turtlebot_standoff_2in parent="standoff_1in_0_link" number="0" x_loc="0" y_loc="0" z_loc="0.0318008"/>
-    <turtlebot_standoff_2in parent="standoff_1in_1_link" number="1" x_loc="0" y_loc="0" z_loc="0.0318008"/>
-    <turtlebot_standoff_2in parent="standoff_1in_2_link" number="2" x_loc="0" y_loc="0" z_loc="0.0318008"/>
-    <turtlebot_standoff_2in parent="standoff_1in_3_link" number="3" x_loc="0" y_loc="0" z_loc="0.0318008"/>
-    <joint name="plate_2_joint" type="fixed">
-      <origin xyz="0 0 0.0572008" rpy="0 0 0" />
-      <parent link="plate_1_link"/>
-      <child link="plate_2_link" />
-    </joint>
-    <link name="plate_2_link">
-      <inertial>
-        <mass value="12" />
-        <origin xyz="0 0 0" />
-        <inertia ixx="1.0" ixy="0.0" ixz="0.0"
-                 iyy="1.0" iyz="0.0"
-                 izz="1.0" />
-      </inertial>
-      <visual>
-        <origin xyz=" 0 0 0 " rpy="0 0 0" />
-        <geometry>
-          <mesh filename="package://turtlebot_description/meshes/plate_1_logo.dae" scale="${M_SCALE} ${M_SCALE} ${M_SCALE}"/>
-        </geometry>
-      </visual>
-      <collision>
-        <origin xyz="0.0 0.0 0.0" rpy="0 0 0" />
-        <geometry>
-          <mesh filename="package://turtlebot_description/meshes/plate_1_logo.dae"/>
-        </geometry>
-      </collision>
-    </link>
-    <joint name="base_kinect_joint" type="fixed">
-      <origin xyz="-0.0844382 0 0.1047496" rpy="0 0 0" />
-      <parent link="plate_2_link" />
-      <child link="kinect_link" />
-    </joint>
-    <link name="kinect_link">
-      <inertial>
-        <mass value="12" />
-        <origin xyz="0 0 0" />
-        <inertia ixx="1.0" ixy="0.0" ixz="0.0"
-                 iyy="1.0" iyz="0.0"
-                 izz="1.0" />
-      </inertial>
-      <visual>
-        <origin xyz=" 0 0 0 " rpy="0 0 0" />
-        <geometry>
-          <mesh filename="package://turtlebot_description/meshes/68-04546_Kinect_Sensor.3ds" scale="${M_SCALE} ${M_SCALE} ${M_SCALE}"/>
-        </geometry>
-      </visual>
-      <collision>
-        <origin xyz="0.0 0.0 0.0" rpy="0 0 0" />
-        <geometry>
-          <mesh filename="package://turtlebot_description/meshes/68-04546_Kinect_Sensor.3ds"/>
-          </geometry>
-      </collision>
-    </link>
-    <joint name="kinect_depth_joint" type="fixed">
-      <origin xyz="0 0.018 0" rpy="0 0 0" />
-      <parent link="kinect_link" />
-      <child link="kinect_depth_frame" />
-    </joint>
-    <link name="kinect_depth_frame">
-      <inertial>
-        <mass value="0.0001" />
-        <origin xyz="0 0 0" />
-        <inertia ixx="0.0001" ixy="0.0" ixz="0.0"
-                 iyy="0.0001" iyz="0.0"
-                 izz="0.0001" />
-      </inertial>
-    </link>
-    <joint name="kinect_depth_optical_joint" type="fixed">
-      <origin xyz="0 0 0" rpy="${-M_PI/2} 0 ${-M_PI/2}" />
-      <parent link="kinect_depth_frame" />
-      <child link="kinect_depth_optical_frame" />
-    </joint>
-    <link name="kinect_depth_optical_frame">
-      <inertial>
-        <mass value="0.0001" />
-        <origin xyz="0 0 0" />
-        <inertia ixx="0.0001" ixy="0.0" ixz="0.0"
-                 iyy="0.0001" iyz="0.0"
-                 izz="0.0001" />
-      </inertial>
-    </link>
-    <joint name="kinect_rgb_joint" type="fixed">
-      <origin xyz="0 -0.005 0" rpy="0 0 0" />
-      <parent link="kinect_link" />
-      <child link="kinect_rgb_frame" />
-    </joint>
-    <link name="kinect_rgb_frame">
-      <inertial>
-        <mass value="0.0001" />
-        <origin xyz="0 0 0" />
-        <inertia ixx="0.0001" ixy="0.0" ixz="0.0"
-                 iyy="0.0001" iyz="0.0"
-                 izz="0.0001" />
-      </inertial>
-    </link>
-    <joint name="kinect_rgb_optical_joint" type="fixed">
-      <origin xyz="0 0 0" rpy="${-M_PI/2} 0 ${-M_PI/2}" />
-      <parent link="kinect_rgb_frame" />
-      <child link="kinect_rgb_optical_frame" />
-    </joint>
-    <link name="kinect_rgb_optical_frame">
-      <inertial>
-        <mass value="0.0001" />
-        <origin xyz="0 0 0" />
-        <inertia ixx="0.0001" ixy="0.0" ixz="0.0"
-                 iyy="0.0001" iyz="0.0"
-                 izz="0.0001" />
-      </inertial>
-    </link>
-    <turtlebot_standoff_kinect parent="plate_2_link" number="0" x_loc="-0.1024382" y_loc="0.098" z_loc="0.0032004"/>
-    <turtlebot_standoff_kinect parent="plate_2_link" number="1" x_loc="-0.1024382" y_loc="-0.098" z_loc="0.0032004"/>
-    <turtlebot_standoff_8in parent="standoff_2in_0_link" number="0" x_loc="0" y_loc="0" z_loc="0.05715"/>
-    <turtlebot_standoff_8in parent="standoff_2in_1_link" number="1" x_loc="0" y_loc="0" z_loc="0.05715"/>
-    <turtlebot_standoff_8in parent="standoff_2in_2_link" number="2" x_loc="0" y_loc="0" z_loc="0.05715"/>
-    <turtlebot_standoff_8in parent="standoff_2in_3_link" number="3" x_loc="0" y_loc="0" z_loc="0.05715"/>
-    <joint name="plate_3_joint" type="fixed">
-      <origin xyz="-0.01316 0 0.2063496" rpy="0 0 0" />
-      <parent link="plate_2_link"/>
-      <child link="plate_3_link" />
-    </joint>
-    <link name="plate_3_link">
-      <inertial>
-        <mass value="12" />
-        <origin xyz="0 0 0" />
-        <inertia ixx="1.0" ixy="0.0" ixz="0.0"
-                 iyy="1.0" iyz="0.0"
-                 izz="1.0" />
-      </inertial>
-      <visual>
-        <origin xyz=" 0 0 0 " rpy="0 0 0" />
-        <geometry>
-          <mesh filename="package://turtlebot_description/meshes/plate_2_logo.dae" scale="${M_SCALE} ${M_SCALE} ${M_SCALE}"/>
-        </geometry>
-      </visual>
-      <collision>
-        <origin xyz="0.0 0.0 0.0" rpy="0 0 0" />
-        <geometry>
-          <mesh filename="package://turtlebot_description/meshes/plate_2_logo.dae"/>
-        </geometry>
-      </collision>
-    </link>
+  <!-- base_footprint is a fictitious link(frame) that is on the ground right below base_link origin, navigation stack depends on this frame -->
+  <link name="base_footprint">
+    <inertial>
+      <mass value="0.0001" />
+      <origin xyz="0 0 0" />
+      <inertia ixx="0.0001" ixy="0.0" ixz="0.0"
+              iyy="0.0001" iyz="0.0"
+              izz="0.0001" />
+    </inertial>
+    <visual>
+      <origin xyz="0 0 0" rpy="0 0 0" />
+      <geometry>
+        <box size="0.001 0.001 0.001" />
+      </geometry>
+      <material name="Green" />
+    </visual>
+    <collision>
+      <origin xyz="0 0 0.017" rpy="0 0 0" />
+      <geometry>
+       <box size="0.001 0.001 0.001" />
+      </geometry>
+    </collision>
+  </link>
+  <link name="base_link">
+    <inertial>
+      <mass value="1" />
+      <origin xyz="0 0 0.0308" />
+      <inertia ixx="1.0" ixy="0.0" ixz="0.0"
+        iyy="1.0" iyz="0.0" izz="1.0" />
+    </inertial>
+    <visual>
+      <origin xyz=" 0 0 0.0308" rpy="0 0 0" />
+      <geometry>
+        <mesh filename="package://turtlebot_description/meshes/create_body.dae"/>
+      </geometry>
+    </visual>
+    <collision>
+      <origin xyz="0.0 0.0 0.0308" rpy="0 0 0" />
+      <geometry>
+        <cylinder length="0.0611632" radius="0.16495"/>
+      </geometry>
+    </collision>
+  </link>
+  <joint name="base_footprint_joint" type="fixed">
+  <!-- NB: While you would think this would make it go up, it is oddly reversed.  This moves the joint to 0,0,0 where we want it for rviz, etc. -->
+    <origin xyz="0 0 0.017" rpy="0 0 0" />
+    <parent link="base_footprint"/>
+    <child link="base_link" />
+  </joint>
+  <link name="left_wheel_link">
+    <inertial>
+      <origin xyz="0 0 0" rpy="0 1.5707 1.5707" />
+      <mass value="0.01" />
+      <inertia ixx="1.0" ixy="0.0" ixz="0.0"
+        iyy="1.0" iyz="0.0" izz="1.0" />
+    </inertial>
+    <visual>
+      <origin xyz="0 0 0" rpy="0 1.5707 1.5707" />
+      <geometry>
+        <cylinder radius="0.033" length = "0.023"/>
+      </geometry>
+    </visual>
+    <collision>
+      <origin xyz="0 0 0" rpy="0 1.5707 1.5707" />
+      <geometry>
+        <cylinder radius="0.033" length = "0.023"/>
+      </geometry>
+    </collision>
+  </link>
+  <joint name="left_wheel_joint" type="continuous">
+    <origin xyz="0 0.13 0.015" rpy="0 0 0"/>
+    <parent link="base_link"/>
+    <child link="left_wheel_link"/>
+    <axis xyz="0 1 0"/>
+  </joint>
+  <link name="right_wheel_link">
+    <inertial>
+      <origin xyz="0 0 0" rpy="0 1.5707 1.5707" />
+      <mass value="0.01" />
+      <inertia ixx="1.0" ixy="0.0" ixz="0.0"
+        iyy="1.0" iyz="0.0" izz="1.0" />
+    </inertial>
+    <visual>
+      <origin xyz="0 0 0" rpy="0 1.5707 1.5707" />
+      <geometry>
+        <cylinder radius="0.033" length = "0.023"/>
+      </geometry>
+    </visual>
+    <collision>
+      <origin xyz="0 0 0" rpy="0 1.5707 1.5707" />
+      <geometry>
+        <cylinder radius="0.033" length = "0.023"/>
+      </geometry>
+    </collision>
+  </link>
+  <joint name="right_wheel_joint" type="continuous">
+    <origin xyz="0 -0.13 0.015" rpy="0 0 0"/>
+    <parent link="base_link"/>
+    <child link="right_wheel_link"/>
+    <axis xyz="0 1 0"/>
+  </joint>
+  <link name="rear_wheel_link">
+    <inertial>
+      <origin xyz="0 0 0" rpy="0 1.5707 1.5707" />
+      <mass value="0.001" />
+      <inertia ixx="1.0" ixy="0.0" ixz="0.0"
+        iyy="1.0" iyz="0.0" izz="1.0" />
+    </inertial>
+    <visual>
+      <origin xyz="0 0 0" rpy="0 1.5707 1.5707"/>
+      <geometry>
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
File: turtlebot_description/urdf/turtlebot_hardware.xacro (robot description, xacro)
@@ -11,21 +11,21 @@
     <link name="spacer_${number}_link">
       <inertial>
-	<mass value="1" />
-	<origin xyz="0 0 0" />
-	<inertia ixx="1.0" ixy="0.0" ixz="0.0"
-		 iyy="1.0" iyz="0.0"
-		 izz="1.0" />
+        <mass value="0.00001" />
+        <origin xyz="0 0 0" />
+        <inertia ixx="1.0" ixy="0.0" ixz="0.0"
+          iyy="1.0" iyz="0.0"
+          izz="1.0" />
       </inertial>
       <visual>
-	<origin xyz=" 0 0 0 " rpy="0 0 0" />
-	<geometry>
-	  <mesh filename="package://turtlebot_description/meshes/68-02403-125_Spacer.dae" scale="${M_SCALE} ${M_SCALE} ${M_SCALE}"/>
-	</geometry>
+        <origin xyz=" 0 0 0 " rpy="0 0 0" />
+        <geometry>
+          <mesh filename="package://turtlebot_description/meshes/68-02403-125_Spacer.dae" scale="${M_SCALE} ${M_SCALE} ${M_SCALE}"/>
+        </geometry>
       </visual>
       <collision>
-	<origin xyz="0.0 0.0 0.0" rpy="0 0 0" />
-	<geometry>
-	  <mesh filename="package://turtlebot_description/meshes/68-02403-125_Spacer.dae"/>
-	</geometry>
+        <origin xyz="0.0 0.0 0.0" rpy="0 0 0" />
+        <geometry>
+          <cylinder length="0.003175" radius=".0127"/>
+        </geometry>
       </collision>
     </link>
@@ -39,21 +39,21 @@
     <link name="standoff_1in_${number}_link">
       <inertial>
-	<mass value="1" />
-	<origin xyz="0 0 0" />
-	<inertia ixx="1.0" ixy="0.0" ixz="0.0"
-		 iyy="1.0" iyz="0.0"
-		 izz="1.0" />
+        <mass value="0.00001" />
+        <origin xyz="0 0 0" />
+        <inertia ixx="1.0" ixy="0.0" ixz="0.0"
+          iyy="1.0" iyz="0.0"
+          izz="1.0" />
       </inertial>
       <visual>
-	<origin xyz=" 0 0 0 " rpy="0 0 0" />
-	<geometry>
-	  <mesh filename="package://turtlebot_description/meshes/68-04552-1000-RA_Turtlebot_M-F_Standoff.dae" scale="${M_SCALE} ${M_SCALE} ${M_SCALE}"/>
-	</geometry>
+        <origin xyz=" 0 0 0 " rpy="0 0 0" />
+        <geometry>
+          <mesh filename="package://turtlebot_description/meshes/68-04552-1000-RA_Turtlebot_M-F_Standoff.dae" scale="${M_SCALE} ${M_SCALE} ${M_SCALE}"/>
+        </geometry>
       </visual>
       <collision>
-	<origin xyz="0.0 0.0 0.0" rpy="0 0 0" />
-	<geometry>
-	  <mesh filename="package://turtlebot_description/meshes/68-04552-1000-RA_Turtlebot_M-F_Standoff.dae"/>
-	</geometry>
+        <origin xyz="0.0 0.0 0.0" rpy="0 0 0" />
+        <geometry>
+          <cylinder length="0.0381" radius="0.011113"/>
+        </geometry>
       </collision>
     </link>
@@ -67,21 +67,21 @@
     <link name="standoff_2in_${number}_link">
       <inertial>
-	<mass value="1" />
-	<origin xyz="0 0 0" />
-	<inertia ixx="1.0" ixy="0.0" ixz="0.0"
-		 iyy="1.0" iyz="0.0"
-		 izz="1.0" />
+        <mass value="0.00001" />
+        <origin xyz="0 0 0" />
+        <inertia ixx="1.0" ixy="0.0" ixz="0.0"
+          iyy="1.0" iyz="0.0"
+          izz="1.0" />
       </inertial>
       <visual>
-	<origin xyz=" 0 0 0 " rpy="0 0 0" />
-	<geometry>
-	  <mesh filename="package://turtlebot_description/meshes/68-04552-2000-RA_Turtlebot_M-F_Standoff.dae" scale="${M_SCALE} ${M_SCALE} ${M_SCALE}"/>
-	</geometry>
+        <origin xyz=" 0 0 0 " rpy="0 0 0" />
+        <geometry>
+          <mesh filename="package://turtlebot_description/meshes/68-04552-2000-RA_Turtlebot_M-F_Standoff.dae" scale="${M_SCALE} ${M_SCALE} ${M_SCALE}"/>
+        </geometry>
       </visual>
       <collision>
-	<origin xyz="0.0 0.0 0.0" rpy="0 0 0" />
-	<geometry>
-	  <mesh filename="package://turtlebot_description/meshes/68-04552-2000-RA_Turtlebot_M-F_Standoff.dae"/>
-	</geometry>
+        <origin xyz="0.0 0.0 0.0" rpy="0 0 0" />
+        <geometry>
+          <cylinder length="0.0635" radius="0.0381"/>
+        </geometry>
       </collision>
     </link>
@@ -95,21 +95,21 @@
     <link name="standoff_8in_${number}_link">
       <inertial>
-	<mass value="1" />
-	<origin xyz="0 0 0" />
-	<inertia ixx="1.0" ixy="0.0" ixz="0.0"
-		 iyy="1.0" iyz="0.0"
-		 izz="1.0" />
+        <mass value="0.00001" />
+        <origin xyz="0 0 0" />
+        <inertia ixx="1.0" ixy="0.0" ixz="0.0"
+          iyy="1.0" iyz="0.0"
+          izz="1.0" />
       </inertial>
       <visual>
-	<origin xyz=" 0 0 0 " rpy="0 0 0" />
-	<geometry>
-	  <mesh filename="package://turtlebot_description/meshes/68-02421-8000-RA_Turtlebot_F-F_Standoff.dae" scale="${M_SCALE} ${M_SCALE} ${M_SCALE}"/>
-	</geometry>
+        <origin xyz=" 0 0 0 " rpy="0 0 0" />
+        <geometry>
+          <mesh filename="package://turtlebot_description/meshes/68-02421-8000-RA_Turtlebot_F-F_Standoff.dae" scale="${M_SCALE} ${M_SCALE} ${M_SCALE}"/>
+        </geometry>
       </visual>
       <collision>
-	<origin xyz="0.0 0.0 0.0" rpy="0 0 0" />
-	<geometry>
-	  <mesh filename="package://turtlebot_description/meshes/68-02421-8000-RA_Turtlebot_F-F_Standoff.dae"/>
-	</geometry>
+        <origin xyz="0.0 0.0 0.0" rpy="0 0 0" />
+        <geometry>
+          <cylinder length="0.2032" radius="0.011113"/>
+        </geometry>
       </collision>
     </link>
@@ -123,21 +123,21 @@
     <link name="standoff_kinect_${number}_link">
       <inertial>
-	<mass value="1" />
-	<origin xyz="0 0 0" />
-	<inertia ixx="1.0" ixy="0.0" ixz="0.0"
-		 iyy="1.0" iyz="0.0"
-		 izz="1.0" />
+        <mass value="0.00001" />
+        <origin xyz="0 0 0" />
+        <inertia ixx="1.0" ixy="0.0" ixz="0.0"
+          iyy="1.0" iyz="0.0"
+          izz="1.0" />
       </inertial>
       <visual>
-	<origin xyz=" 0 0 0 " rpy="0 0 0" />
-	<geometry>
-	  <mesh filename="package://turtlebot_description/meshes/68-04556-RA_Kinect_Standoff_Assy.3ds" scale="${M_SCALE} ${M_SCALE} ${M_SCALE}"/>
-	</geometry>
+        <origin xyz=" 0 0 0 " rpy="0 0 0" />
+        <geometry>
+          <mesh filename="package://turtlebot_description/meshes/68-04556-RA_Kinect_Standoff_Assy.3ds" scale="${M_SCALE} ${M_SCALE} ${M_SCALE}"/>
+        </geometry>
       </visual>
       <collision>
-	<origin xyz="0.0 0.0 0.0" rpy="0 0 0" />
-	<geometry>
-	  <mesh filename="package://turtlebot_description/meshes/68-04556-RA_Kinect_Standoff_Assy.3ds"/>
-	</geometry>
+        <origin xyz="0.0 0.0 0.0" rpy="0 0 0" />
+        <geometry>
+          <cylinder length="0.008585" radius="0.001111"/>
+        </geometry>
       </collision>
     </link>

Commit message: adding extra sensor to urdf

File: turtlebot_description/urdf/turtlebot.xacro (robot description, xacro)
@@ -188,4 +188,24 @@
     </inertial>
   </link>
+  <joint name="laser_joint" type="fixed">
+    <origin xyz="-0.065 0 0.075" rpy="0 0 0" />
+    <parent link="base_link" />
+    <child link="laser" />
+  </joint>
+  <link name="laser">
+    <visual>
+      <geometry>
+        <box size="0.02 0.035 0.002" />
+      </geometry>
+      <material name="Green" />
+    </visual>
+    <inertial>
+      <mass value="0.000001" />
+      <origin xyz="0 0 0" />
+      <inertia ixx="0.0001" ixy="0.0" ixz="0.0"
+        iyy="0.0001" iyz="0.0"
+        izz="0.0001" />
+    </inertial>
+  </link>
   <joint name="plate_0_joint" type="fixed">
     <origin xyz="-0.04334 0  0.06775704" rpy="0 0 0" />
