Commit message: removing rpy from inertial elements of links, to get rid of not supported warning

File: turtlebot_description/urdf/turtlebot.xacro (robot description, xacro)
@@ -126,5 +126,5 @@
   <link name="left_wheel_link">
     <inertial>
-      <origin xyz="0 0 0" rpy="0 1.5707 1.5707" />
+      <origin xyz="0 0 0"/>
       <mass value="0.01" />
       <inertia ixx="1.0" ixy="0.0" ixz="0.0"
@@ -152,5 +152,5 @@
   <link name="right_wheel_link">
     <inertial>
-      <origin xyz="0 0 0" rpy="0 1.5707 1.5707" />
+      <origin xyz="0 0 0"/>
       <mass value="0.01" />
       <inertia ixx="1.0" ixy="0.0" ixz="0.0"
@@ -178,5 +178,5 @@
   <link name="rear_wheel_link">
     <inertial>
-      <origin xyz="0 0 0" rpy="0 1.5707 1.5707" />
+      <origin xyz="0 0 0"/>
       <mass value="0.001" />
       <inertia ixx="1.0" ixy="0.0" ixz="0.0"
@@ -204,5 +204,5 @@
   <link name="front_wheel_link">
     <inertial>
-      <origin xyz="0 0 0" rpy="0 1.5707 1.5707" />
+      <origin xyz="0 0 0" />
       <mass value="0.01" />
       <inertia ixx="1.0" ixy="0.0" ixz="0.0"

Commit message: updating urdf to reflect production turtlebot changes

File: turtlebot_description/urdf/turtlebot.xacro (robot description, xacro)
@@ -298,10 +298,10 @@
     </collision>
   </link>
-  <turtlebot_standoff_1in parent="base_link" number="0" x_loc="0.0676402" y_loc="0.1314196" z_loc="0.0709803"/>
-  <turtlebot_standoff_1in parent="base_link" number="1" x_loc="0.0676402" y_loc="-0.1314196" z_loc="0.0709803"/>
-  <turtlebot_standoff_1in parent="base_link" number="2" x_loc="-0.052832" y_loc="-0.1314196" z_loc="0.0709803"/>
-  <turtlebot_standoff_1in parent="base_link" number="3" x_loc="-0.052832" y_loc="0.1314196" z_loc="0.0709803"/>
+  <turtlebot_standoff_2in parent="base_link" number="0" x_loc="0.0676402" y_loc="0.1314196" z_loc="0.0709803"/>
+  <turtlebot_standoff_2in parent="base_link" number="1" x_loc="0.0676402" y_loc="-0.1314196" z_loc="0.0709803"/>
+  <turtlebot_standoff_2in parent="base_link" number="2" x_loc="-0.052832" y_loc="-0.1314196" z_loc="0.0709803"/>
+  <turtlebot_standoff_2in parent="base_link" number="3" x_loc="-0.052832" y_loc="0.1314196" z_loc="0.0709803"/>
   <joint name="plate_1_joint" type="fixed">
-    <origin xyz="0.04068 0 0.0318008" rpy="0 0 0" />
+    <origin xyz="0.04068 0 0.05715" rpy="0 0 0" />
     <parent link="plate_0_link"/>
     <child link="plate_1_link" />
@@ -328,8 +328,8 @@
     </collision>
   </link>
-  <turtlebot_standoff_2in parent="standoff_1in_0_link" number="0" x_loc="0" y_loc="0" z_loc="0.0318008"/>
-  <turtlebot_standoff_2in parent="standoff_1in_1_link" number="1" x_loc="0" y_loc="0" z_loc="0.0318008"/>
-  <turtlebot_standoff_2in parent="standoff_1in_2_link" number="2" x_loc="0" y_loc="0" z_loc="0.0318008"/>
-  <turtlebot_standoff_2in parent="standoff_1in_3_link" number="3" x_loc="0" y_loc="0" z_loc="0.0318008"/>
+  <turtlebot_standoff_2in parent="standoff_2in_0_link" number="4" x_loc="0" y_loc="0" z_loc="0.05715"/>
+  <turtlebot_standoff_2in parent="standoff_2in_1_link" number="5" x_loc="0" y_loc="0" z_loc="0.05715"/>
+  <turtlebot_standoff_2in parent="standoff_2in_2_link" number="6" x_loc="0" y_loc="0" z_loc="0.05715"/>
+  <turtlebot_standoff_2in parent="standoff_2in_3_link" number="7" x_loc="0" y_loc="0" z_loc="0.05715"/>
   <joint name="plate_2_joint" type="fixed">
     <origin xyz="0 0 0.0572008" rpy="0 0 0" />
@@ -442,8 +442,8 @@
   <turtlebot_standoff_kinect parent="plate_2_link" number="0" x_loc="-0.1024382" y_loc="0.098" z_loc="0.0032004"/>
   <turtlebot_standoff_kinect parent="plate_2_link" number="1" x_loc="-0.1024382" y_loc="-0.098" z_loc="0.0032004"/>
-  <turtlebot_standoff_8in parent="standoff_2in_0_link" number="0" x_loc="0" y_loc="0" z_loc="0.05715"/>
-  <turtlebot_standoff_8in parent="standoff_2in_1_link" number="1" x_loc="0" y_loc="0" z_loc="0.05715"/>
-  <turtlebot_standoff_8in parent="standoff_2in_2_link" number="2" x_loc="0" y_loc="0" z_loc="0.05715"/>
-  <turtlebot_standoff_8in parent="standoff_2in_3_link" number="3" x_loc="0" y_loc="0" z_loc="0.05715"/>
+  <turtlebot_standoff_8in parent="standoff_2in_4_link" number="0" x_loc="0" y_loc="0" z_loc="0.05715"/>
+  <turtlebot_standoff_8in parent="standoff_2in_5_link" number="1" x_loc="0" y_loc="0" z_loc="0.05715"/>
+  <turtlebot_standoff_8in parent="standoff_2in_6_link" number="2" x_loc="0" y_loc="0" z_loc="0.05715"/>
+  <turtlebot_standoff_8in parent="standoff_2in_7_link" number="3" x_loc="0" y_loc="0" z_loc="0.05715"/>
   <joint name="plate_3_joint" type="fixed">
     <origin xyz="-0.01316 0 0.2063496" rpy="0 0 0" />

Commit message: add space for calibration

File: turtlebot_description/urdf/turtlebot.xacro (robot description, xacro)
@@ -3,4 +3,5 @@
   <include filename="$(find turtlebot_description)/urdf/turtlebot_hardware.xacro" />
   <include filename="$(find turtlebot_description)/urdf/gazebo.urdf.xacro"/>
+  <include filename="$(find turtlebot_description)/urdf/turtlebot_calibration.xacro" />
   <material name="Green">
     <color rgba="0.0 0.8 0.0 1.0"/>
@@ -359,6 +360,7 @@
   </link>
   <joint name="base_kinect_joint" type="fixed">
-    <origin xyz="-0.0844382 0 0.1047496" rpy="0 0 0" />
-    <parent link="plate_2_link" />
+    <origin xyz="${turtlebot_calib_cam_x} ${turtlebot_calib_cam_y} ${turtlebot_calib_cam_z}"
+            rpy="${turtlebot_calib_cam_rr} ${turtlebot_calib_cam_rp} ${turtlebot_calib_cam_ry}" />
+    <parent link="${turtlebot_kinect_frame_name}" />
     <child link="kinect_link" />
   </joint>

Commit message: Changed rear_wheel_link to be fixed to fix the robot model.
--HG--
branch : diamondback_development
extra : transplant_source : %8E%2B%98W%E5%B6%5DjI%E7%03i%8A%FAn%AF%C8%B1E%40

File: turtlebot_description/urdf/turtlebot.xacro (robot description, xacro)
@@ -196,5 +196,5 @@
     </collision>
   </link>
-  <joint name="rear_castor_joint" type="continuous">
+  <joint name="rear_castor_joint" type="fixed">
     <origin xyz="-0.13 0 0.0" rpy="0 0 0"/>
     <parent link="base_link"/>

Commit message: Changed rear_wheel_link to be fixed to fix the robot model.

File: turtlebot_description/urdf/turtlebot.xacro (robot description, xacro)
@@ -197,5 +197,5 @@
     </collision>
   </link>
-  <joint name="rear_castor_joint" type="continuous">
+  <joint name="rear_castor_joint" type="fixed">
     <origin xyz="-0.13 0 0.0" rpy="0 0 0"/>
     <parent link="base_link"/>

Commit message: fixed joints get reduced, breaking plugin looking for the joint in simulation

File: turtlebot_description/urdf/turtlebot.xacro (robot description, xacro)
@@ -197,5 +197,5 @@
     </collision>
   </link>
-  <joint name="rear_castor_joint" type="fixed">
+  <joint name="rear_castor_joint" type="continuous">
     <origin xyz="-0.13 0 0.0" rpy="0 0 0"/>
     <parent link="base_link"/>

Commit message: change back to fixed, not sure why, but must be useful?

File: turtlebot_description/urdf/turtlebot.xacro (robot description, xacro)
@@ -197,5 +197,6 @@
     </collision>
   </link>
-  <joint name="rear_castor_joint" type="continuous">
+  <!-- not sure why this is set to fixed -->
+  <joint name="rear_castor_joint" type="fixed">
     <origin xyz="-0.13 0 0.0" rpy="0 0 0"/>
     <parent link="base_link"/>

Commit message: Switching to new-style xacro:macro's
--HG--
branch : tbot_improve

File: turtlebot_description/urdf/turtlebot.xacro (robot description, xacro)
@@ -16,5 +16,5 @@
   <property name="base_x" value="0.33" />
   <property name="base_y" value="0.33" />
-  <macro name="turtlebot">
+  <xacro:macro name="turtlebot">
   <!-- base_footprint is a fictitious link(frame) that is on the ground right below base_link origin, navigation stack depends on this frame -->
   <link name="base_footprint">
@@ -488,4 +488,4 @@
     </sensor:ray>
   </gazebo>
-  </macro> <!--turtlebot -->
+  </xacro:macro> <!--turtlebot -->
 </robot>

File: turtlebot_description/urdf/turtlebot_hardware.xacro (robot description, xacro)
@@ -1,7 +1,7 @@
 <?xml version="1.0"?>
-<robot>
+<robot name="turtlebot_hardware" xmlns:xacro="http://ros.org/wiki/xacro">
   <property name="M_PI" value="3.14159"/>
   <property name="M_SCALE" value="0.001"/>
-  <macro name="turtlebot_spacer" params="parent number x_loc y_loc z_loc">
+  <xacro:macro name="turtlebot_spacer" params="parent number x_loc y_loc z_loc">
     <joint name="spacer_${number}_joint" type="fixed">
       <origin xyz="${x_loc} ${y_loc} ${z_loc}" rpy="0 0 0" />
@@ -30,6 +30,6 @@
       </collision>
     </link>
-  </macro>
-  <macro name="turtlebot_standoff_1in" params="parent number x_loc y_loc z_loc">
+  </xacro:macro>
+  <xacro:macro name="turtlebot_standoff_1in" params="parent number x_loc y_loc z_loc">
     <joint name="standoff_1in_${number}_joint" type="fixed">
       <origin xyz="${x_loc} ${y_loc} ${z_loc}" rpy="0 0 0" />
@@ -58,6 +58,6 @@
       </collision>
     </link>
-  </macro>
-  <macro name="turtlebot_standoff_2in" params="parent number x_loc y_loc z_loc">
+  </xacro:macro>
+  <xacro:macro name="turtlebot_standoff_2in" params="parent number x_loc y_loc z_loc">
     <joint name="standoff_2in_${number}_joint" type="fixed">
       <origin xyz="${x_loc} ${y_loc} ${z_loc}" rpy="0 0 0" />
@@ -86,6 +86,6 @@
       </collision>
     </link>
-  </macro>
-  <macro name="turtlebot_standoff_8in" params="parent number x_loc y_loc z_loc">
+  </xacro:macro>
+  <xacro:macro name="turtlebot_standoff_8in" params="parent number x_loc y_loc z_loc">
     <joint name="standoff_8in_${number}_joint" type="fixed">
       <origin xyz="${x_loc} ${y_loc} ${z_loc}" rpy="0 0 0" />
@@ -114,6 +114,6 @@
       </collision>
     </link>
-  </macro>
-  <macro name="turtlebot_standoff_kinect" params="parent number x_loc y_loc z_loc">
+  </xacro:macro>
+  <xacro:macro name="turtlebot_standoff_kinect" params="parent number x_loc y_loc z_loc">
     <joint name="standoff_kinect_${number}_joint" type="fixed">
       <origin xyz="${x_loc} ${y_loc} ${z_loc}" rpy="0 0 0" />
@@ -142,4 +142,4 @@
       </collision>
     </link>
-  </macro>
+  </xacro:macro>
 </robot>
