Commit message: Added sensors for the cliff sensors

File: turtlebot_description/urdf/gazebo.urdf.xacro (robot description, xacro)
@@ -11,7 +11,73 @@
       <wheel_separation>.260</wheel_separation>
       <wheel_diameter>0.066</wheel_diameter>
+      <base_geom>base_link_geom_base_link</base_geom>
       <updateRate>40</updateRate>
       <torque>0.1</torque>
     </controller:gazebo_ros_create>
+  </gazebo>
+  <gazebo reference="wall_sensor_link">
+    <sensor:ray name="wall_sensor">
+      <alwaysActive>true</alwaysActive>
+      <rayCount>1</rayCount>
+      <rangeCount>1</rangeCount>
+      <resRange>0.1</resRange>
+      <minAngle>0</minAngle>
+      <maxAngle>0</maxAngle>
+      <minRange>0.0160</minRange>
+      <maxRange>0.04</maxRange>
+      <displayRays>fan</displayRays>
+    </sensor:ray>
+  </gazebo>
+  <gazebo reference="left_cliff_sensor_link">
+    <sensor:ray name="left_cliff_sensor">
+      <alwaysActive>true</alwaysActive>
+      <rayCount>1</rayCount>
+      <rangeCount>1</rangeCount>
+      <resRange>0.1</resRange>
+      <minAngle>0</minAngle>
+      <maxAngle>0</maxAngle>
+      <minRange>0.01</minRange>
+      <maxRange>0.04</maxRange>
+      <displayRays>fan</displayRays>
+    </sensor:ray>
+  </gazebo>
+  <gazebo reference="right_cliff_sensor_link">
+    <sensor:ray name="right_cliff_sensor">
+      <alwaysActive>true</alwaysActive>
+      <rayCount>1</rayCount>
+      <rangeCount>1</rangeCount>
+      <resRange>0.1</resRange>
+      <minAngle>0</minAngle>
+      <maxAngle>0</maxAngle>
+      <minRange>0.01</minRange>
+      <maxRange>0.04</maxRange>
+      <displayRays>fan</displayRays>
+    </sensor:ray>
+  </gazebo>
+  <gazebo reference="leftfront_cliff_sensor_link">
+    <sensor:ray name="leftfront_cliff_sensor">
+      <alwaysActive>true</alwaysActive>
+      <rayCount>1</rayCount>
+      <rangeCount>1</rangeCount>
+      <resRange>0.1</resRange>
+      <minAngle>0</minAngle>
+      <maxAngle>0</maxAngle>
+      <minRange>0.01</minRange>
+      <maxRange>0.04</maxRange>
+      <displayRays>fan</displayRays>
+    </sensor:ray>
+  </gazebo>
+  <gazebo reference="rightfront_cliff_sensor_link">
+    <sensor:ray name="rightfront_cliff_sensor">
+      <alwaysActive>true</alwaysActive>
+      <rayCount>1</rayCount>
+      <rangeCount>1</rangeCount>
+      <resRange>0.1</resRange>
+      <minAngle>0</minAngle>
+      <maxAngle>0</maxAngle>
+      <minRange>0.01</minRange>
+      <maxRange>0.04</maxRange>
+      <displayRays>fan</displayRays>
+    </sensor:ray>
   </gazebo>
   <gazebo reference="kinect_link">

File: turtlebot_description/urdf/turtlebot.xacro (robot description, xacro)
@@ -54,9 +54,73 @@
     </collision>
   </link>
+  <link name="wall_sensor_link">
+    <inertial>
+      <mass value="0" />
+      <origin xyz="0 0 0"/>
+      <inertia ixx="1.0" ixy="0.0" ixz="0.0"
+        iyy="1.0" iyz="0.0" izz="1.0" />
+    </inertial>
+  </link>
+  <link name="left_cliff_sensor_link">
+    <inertial>
+      <mass value="0" />
+      <origin xyz="0 0 0"/>
+      <inertia ixx="1.0" ixy="0.0" ixz="0.0"
+        iyy="1.0" iyz="0.0" izz="1.0" />
+    </inertial>
+  </link>
+  <link name="right_cliff_sensor_link">
+    <inertial>
+      <mass value="0" />
+      <origin xyz="0 0 0"/>
+      <inertia ixx="1.0" ixy="0.0" ixz="0.0"
+        iyy="1.0" iyz="0.0" izz="1.0" />
+    </inertial>
+  </link>
+  <link name="leftfront_cliff_sensor_link">
+    <inertial>
+      <mass value="0" />
+      <origin xyz="0 0 0"/>
+      <inertia ixx="1.0" ixy="0.0" ixz="0.0"
+        iyy="1.0" iyz="0.0" izz="1.0" />
+    </inertial>
+  </link>
+  <link name="rightfront_cliff_sensor_link">
+    <inertial>
+      <mass value="0" />
+      <origin xyz="0 0 0"/>
+      <inertia ixx="1.0" ixy="0.0" ixz="0.0"
+        iyy="1.0" iyz="0.0" izz="1.0" />
+    </inertial>
+  </link>
   <joint name="base_footprint_joint" type="fixed">
-  <!-- NB: While you would think this would make it go up, it is oddly reversed.  This moves the joint to 0,0,0 where we want it for rviz, etc. -->
     <origin xyz="0 0 0.017" rpy="0 0 0" />
     <parent link="base_footprint"/>
     <child link="base_link" />
+  </joint>
+  <joint name="base_wall_sensor_joint" type="fixed">
+    <origin xyz="0.09 -0.120 0.042" rpy="0 0 -1.0" />
+    <parent link="base_link"/>
+    <child link="wall_sensor_link" />
+  </joint>
+  <joint name="base_left_cliff_sensor_joint" type="fixed">
+    <origin xyz="0.07 0.14 0.01" rpy="0 1.57079 0" />
+    <parent link="base_link"/>
+    <child link="left_cliff_sensor_link" />
+  </joint>
+  <joint name="base_right_cliff_sensor_joint" type="fixed">
+    <origin xyz="0.07 -0.14 0.01" rpy="0 1.57079 0" />
+    <parent link="base_link"/>
+    <child link="right_cliff_sensor_link" />
+  </joint>
+  <joint name="base_leftfront_cliff_sensor_joint" type="fixed">
+    <origin xyz="0.15 0.04 0.01" rpy="0 1.57079 0" />
+    <parent link="base_link"/>
+    <child link="leftfront_cliff_sensor_link" />
+  </joint>
+  <joint name="base_rightfront_cliff_sensor_joint" type="fixed">
+    <origin xyz="0.15 -0.04 0.01" rpy="0 1.57079 0" />
+    <parent link="base_link"/>
+    <child link="rightfront_cliff_sensor_link" />
   </joint>
   <link name="left_wheel_link">

Commit message: Made sensor links have non-zero mass. A zero-mass caused urdf2gazebo to ignore the sensor links

File: turtlebot_description/urdf/gazebo.urdf.xacro (robot description, xacro)
@@ -26,5 +26,5 @@
       <minRange>0.0160</minRange>
       <maxRange>0.04</maxRange>
-      <displayRays>fan</displayRays>
+      <displayRays>false</displayRays>
     </sensor:ray>
   </gazebo>
@@ -39,5 +39,5 @@
       <minRange>0.01</minRange>
       <maxRange>0.04</maxRange>
-      <displayRays>fan</displayRays>
+      <displayRays>false<displayRays>
     </sensor:ray>
   </gazebo>
@@ -52,5 +52,5 @@
       <minRange>0.01</minRange>
       <maxRange>0.04</maxRange>
-      <displayRays>fan</displayRays>
+      <displayRays>false</displayRays>
     </sensor:ray>
   </gazebo>
@@ -65,5 +65,5 @@
       <minRange>0.01</minRange>
       <maxRange>0.04</maxRange>
-      <displayRays>fan</displayRays>
+      <displayRays>false</displayRays>
     </sensor:ray>
   </gazebo>

File: turtlebot_description/urdf/turtlebot.xacro (robot description, xacro)
@@ -56,5 +56,5 @@
   <link name="wall_sensor_link">
     <inertial>
-      <mass value="0" />
+      <mass value="0.01" />
       <origin xyz="0 0 0"/>
       <inertia ixx="1.0" ixy="0.0" ixz="0.0"
@@ -64,5 +64,5 @@
   <link name="left_cliff_sensor_link">
     <inertial>
-      <mass value="0" />
+      <mass value="0.01" />
       <origin xyz="0 0 0"/>
       <inertia ixx="1.0" ixy="0.0" ixz="0.0"
@@ -72,5 +72,5 @@
   <link name="right_cliff_sensor_link">
     <inertial>
-      <mass value="0" />
+      <mass value="0.01" />
       <origin xyz="0 0 0"/>
       <inertia ixx="1.0" ixy="0.0" ixz="0.0"
@@ -80,5 +80,5 @@
   <link name="leftfront_cliff_sensor_link">
     <inertial>
-      <mass value="0" />
+      <mass value="0.01" />
       <origin xyz="0 0 0"/>
       <inertia ixx="1.0" ixy="0.0" ixz="0.0"
@@ -88,5 +88,5 @@
   <link name="rightfront_cliff_sensor_link">
     <inertial>
-      <mass value="0" />
+      <mass value="0.01" />
       <origin xyz="0 0 0"/>
       <inertia ixx="1.0" ixy="0.0" ixz="0.0"

Commit message: fix masses for turtlebot

File: turtlebot_description/urdf/gazebo.urdf.xacro (robot description, xacro)
@@ -13,5 +13,5 @@
       <base_geom>base_link_geom_base_link</base_geom>
       <updateRate>40</updateRate>
-      <torque>0.1</torque>
+      <torque>1.0</torque>
     </controller:gazebo_ros_create>
   </gazebo>
@@ -105,15 +105,29 @@
     </sensor:camera>
   </gazebo>
+  <gazebo reference="left_wheel_link">
+    <mu1 value="10.0"/>
+    <mu2 value="0.5"/>
+    <kp value="100000000.0"/>
+    <kd value="10000.0"/>
+    <fdir1 value="0 1 0"/>
+  </gazebo>
+  <gazebo reference="right_wheel_link">
+    <mu1 value="10.0"/>
+    <mu2 value="0.5"/>
+    <kp value="100000000.0"/>
+    <kd value="10000.0"/>
+    <fdir1 value="0 1 0"/>
+  </gazebo>
   <gazebo reference="rear_wheel_link">
     <mu1 value="0"/>
     <mu2 value="0"/>
-    <kp value="100000.0"/>
-    <kd value="1.0"/>
+    <kp value="100000000.0"/>
+    <kd value="1000.0"/>
   </gazebo>
   <gazebo reference="front_wheel_link">
     <mu1 value="0"/>
     <mu2 value="0"/>
-    <kp value="100000.0"/>
-    <kd value="1.0"/>
+    <kp value="100000000.0"/>
+    <kd value="1000.0"/>
   </gazebo>
 </robot>

File: turtlebot_description/urdf/turtlebot.xacro (robot description, xacro)
@@ -38,50 +38,50 @@
       <mass value="1" />
       <origin xyz="0 0 0.0308" />
+      <inertia ixx="0.1" ixy="0.0" ixz="0.0"
+        iyy="0.1" iyz="0.0" izz="0.1" />
+    </inertial>
+    <visual>
+      <origin xyz=" 0 0 0.0308" rpy="0 0 0" />
+      <geometry>
+        <mesh filename="package://turtlebot_description/meshes/create_body.dae"/>
+      </geometry>
+    </visual>
+    <collision>
+      <origin xyz="0.0 0.0 0.0308" rpy="0 0 0" />
+      <geometry>
+        <cylinder length="0.0611632" radius="0.16495"/>
+      </geometry>
+    </collision>
+  </link>
+  <link name="wall_sensor_link">
+    <inertial>
+      <mass value="0.01" />
+      <origin xyz="0 0 0"/>
+      <inertia ixx="0.001" ixy="0.0" ixz="0.0"
+        iyy="0.001" iyz="0.0" izz="0.001" />
+    </inertial>
+  </link>
+  <link name="left_cliff_sensor_link">
+    <inertial>
+      <mass value="0.01" />
+      <origin xyz="0 0 0"/>
+      <inertia ixx="0.001" ixy="0.0" ixz="0.0"
+        iyy="0.001" iyz="0.0" izz="0.001" />
+    </inertial>
+  </link>
+  <link name="right_cliff_sensor_link">
+    <inertial>
+      <mass value="0.01" />
+      <origin xyz="0 0 0"/>
+      <inertia ixx="0.001" ixy="0.0" ixz="0.0"
+        iyy="0.001" iyz="0.0" izz="0.001" />
+    </inertial>
+  </link>
+  <link name="leftfront_cliff_sensor_link">
+    <inertial>
+      <mass value="0.01" />
+      <origin xyz="0 0 0"/>
       <inertia ixx="1.0" ixy="0.0" ixz="0.0"
-        iyy="1.0" iyz="0.0" izz="1.0" />
-    </inertial>
-    <visual>
-      <origin xyz=" 0 0 0.0308" rpy="0 0 0" />
-      <geometry>
-        <mesh filename="package://turtlebot_description/meshes/create_body.dae"/>
-      </geometry>
-    </visual>
-    <collision>
-      <origin xyz="0.0 0.0 0.0308" rpy="0 0 0" />
-      <geometry>
-        <cylinder length="0.0611632" radius="0.16495"/>
-      </geometry>
-    </collision>
-  </link>
-  <link name="wall_sensor_link">
-    <inertial>
-      <mass value="0.01" />
-      <origin xyz="0 0 0"/>
-      <inertia ixx="1.0" ixy="0.0" ixz="0.0"
-        iyy="1.0" iyz="0.0" izz="1.0" />
-    </inertial>
-  </link>
-  <link name="left_cliff_sensor_link">
-    <inertial>
-      <mass value="0.01" />
-      <origin xyz="0 0 0"/>
-      <inertia ixx="1.0" ixy="0.0" ixz="0.0"
-        iyy="1.0" iyz="0.0" izz="1.0" />
-    </inertial>
-  </link>
-  <link name="right_cliff_sensor_link">
-    <inertial>
-      <mass value="0.01" />
-      <origin xyz="0 0 0"/>
-      <inertia ixx="1.0" ixy="0.0" ixz="0.0"
-        iyy="1.0" iyz="0.0" izz="1.0" />
-    </inertial>
-  </link>
-  <link name="leftfront_cliff_sensor_link">
-    <inertial>
-      <mass value="0.01" />
-      <origin xyz="0 0 0"/>
-      <inertia ixx="1.0" ixy="0.0" ixz="0.0"
-        iyy="1.0" iyz="0.0" izz="1.0" />
+        iyy="0.1" iyz="0.0" izz="0.1" />
     </inertial>
   </link>
@@ -90,6 +90,6 @@
       <mass value="0.01" />
       <origin xyz="0 0 0"/>
-      <inertia ixx="1.0" ixy="0.0" ixz="0.0"
-        iyy="1.0" iyz="0.0" izz="1.0" />
+      <inertia ixx="0.001" ixy="0.0" ixz="0.0"
+        iyy="0.001" iyz="0.0" izz="0.001" />
     </inertial>
   </link>
@@ -128,6 +128,6 @@
       <origin xyz="0 0 0"/>
       <mass value="0.01" />
-      <inertia ixx="1.0" ixy="0.0" ixz="0.0"
-        iyy="1.0" iyz="0.0" izz="1.0" />
+      <inertia ixx="0.001" ixy="0.0" ixz="0.0"
+        iyy="0.001" iyz="0.0" izz="0.001" />
     </inertial>
     <visual>
@@ -154,6 +154,6 @@
       <origin xyz="0 0 0"/>
       <mass value="0.01" />
-      <inertia ixx="1.0" ixy="0.0" ixz="0.0"
-        iyy="1.0" iyz="0.0" izz="1.0" />
+      <inertia ixx="0.001" ixy="0.0" ixz="0.0"
+        iyy="0.001" iyz="0.0" izz="0.001" />
     </inertial>
     <visual>
@@ -180,6 +180,6 @@
       <origin xyz="0 0 0"/>
       <mass value="0.001" />
-      <inertia ixx="1.0" ixy="0.0" ixz="0.0"
-        iyy="1.0" iyz="0.0" izz="1.0" />
+      <inertia ixx="0.0001" ixy="0.0" ixz="0.0"
+        iyy="0.0001" iyz="0.0" izz="0.0001" />
     </inertial>
     <visual>
@@ -206,6 +206,6 @@
       <origin xyz="0 0 0" />
       <mass value="0.01" />
-      <inertia ixx="1.0" ixy="0.0" ixz="0.0"
-        iyy="1.0" iyz="0.0" izz="1.0" />
+      <inertia ixx="0.001" ixy="0.0" ixz="0.0"
+        iyy="0.001" iyz="0.0" izz="0.001" />
     </inertial>
     <visual>
@@ -245,5 +245,5 @@
     </visual>
     <inertial>
-      <mass value="0.000001" />
+      <mass value="0.001" />
       <origin xyz="0 0 0" />
       <inertia ixx="0.0001" ixy="0.0" ixz="0.0"
@@ -265,5 +265,5 @@
     </visual>
     <inertial>
-      <mass value="0.000001" />
+      <mass value="0.001" />
       <origin xyz="0 0 0" />
       <inertia ixx="0.0001" ixy="0.0" ixz="0.0"
@@ -281,7 +281,7 @@
       <mass value="0.01" />
       <origin xyz="0 0 0" />
-      <inertia ixx="1.0" ixy="0.0" ixz="0.0"
-        iyy="1.0" iyz="0.0"
-        izz="1.0" />
+      <inertia ixx="0.1" ixy="0.0" ixz="0.0"
+        iyy="0.1" iyz="0.0"
+        izz="0.1" />
     </inertial>
     <visual>
@@ -311,7 +311,7 @@
       <mass value="0.1" />
       <origin xyz="0 0 0" />
-      <inertia ixx="1.0" ixy="0.0" ixz="0.0"
-        iyy="1.0" iyz="0.0"
-        izz="1.0" />
+      <inertia ixx="0.01" ixy="0.0" ixz="0.0"
+        iyy="0.01" iyz="0.0"
+        izz="0.01" />
     </inertial>
     <visual>
@@ -341,7 +341,7 @@
       <mass value="0.01" />
       <origin xyz="0 0 0" />
-      <inertia ixx="1.0" ixy="0.0" ixz="0.0"
-        iyy="1.0" iyz="0.0"
-        izz="1.0" />
+      <inertia ixx="0.001" ixy="0.0" ixz="0.0"
+        iyy="0.001" iyz="0.0"
+        izz="0.001" />
     </inertial>
     <visual>
@@ -365,9 +365,9 @@
   <link name="kinect_link">
     <inertial>
-      <mass value="0.00001" />
-      <origin xyz="0 0 0" />
-      <inertia ixx="1.0" ixy="0.0" ixz="0.0"
-        iyy="1.0" iyz="0.0"
-        izz="1.0" />
+      <mass value="0.01" />
+      <origin xyz="0 0 0" />
+      <inertia ixx="0.001" ixy="0.0" ixz="0.0"
+        iyy="0.001" iyz="0.0"
+        izz="0.001" />
     </inertial>
     <visual>
@@ -391,9 +391,9 @@
   <link name="kinect_depth_frame">
     <inertial>
-      <mass value="0.000001" />
-      <origin xyz="0 0 0" />
-      <inertia ixx="0.0001" ixy="0.0" ixz="0.0"
-        iyy="0.0001" iyz="0.0"
-        izz="0.0001" />
+      <mass value="0.01" />
+      <origin xyz="0 0 0" />
+      <inertia ixx="0.001" ixy="0.0" ixz="0.0"
+        iyy="0.001" iyz="0.0"
+        izz="0.001" />
     </inertial>
   </link>
@@ -405,5 +405,5 @@
   <link name="kinect_depth_optical_frame">
     <inertial>
-      <mass value="0.000001" />
+      <mass value="0.001" />
       <origin xyz="0 0 0" />
       <inertia ixx="0.0001" ixy="0.0" ixz="0.0"
@@ -419,5 +419,5 @@
   <link name="kinect_rgb_frame">
     <inertial>
-      <mass value="0.000001" />
+      <mass value="0.001" />
       <origin xyz="0 0 0" />
       <inertia ixx="0.0001" ixy="0.0" ixz="0.0"
@@ -433,5 +433,5 @@
   <link name="kinect_rgb_optical_frame">
     <inertial>
-      <mass value="0.000001" />
+      <mass value="0.001" />
       <origin xyz="0 0 0" />
       <inertia ixx="0.0001" ixy="0.0" ixz="0.0"
@@ -455,7 +455,7 @@
       <mass value="0.01" />
       <origin xyz="0 0 0" />
-      <inertia ixx="1.0" ixy="0.0" ixz="0.0"
-        iyy="1.0" iyz="0.0"
-        izz="1.0" />
+      <inertia ixx="0.0001" ixy="0.0" ixz="0.0"
+        iyy="0.0001" iyz="0.0"
+        izz="0.0001" />
     </inertial>
     <visual>

File: turtlebot_description/urdf/turtlebot_hardware.xacro (robot description, xacro)
@@ -11,9 +11,9 @@
     <link name="spacer_${number}_link">
       <inertial>
-        <mass value="0.00001" />
+        <mass value="0.001" />
         <origin xyz="0 0 0" />
-        <inertia ixx="1.0" ixy="0.0" ixz="0.0"
-          iyy="1.0" iyz="0.0"
-          izz="1.0" />
+        <inertia ixx="0.0001" ixy="0.0" ixz="0.0"
+          iyy="0.0001" iyz="0.0"
+          izz="0.0001" />
       </inertial>
       <visual>
@@ -39,9 +39,9 @@
     <link name="standoff_1in_${number}_link">
       <inertial>
-        <mass value="0.00001" />
+        <mass value="0.001" />
         <origin xyz="0 0 0" />
-        <inertia ixx="1.0" ixy="0.0" ixz="0.0"
-          iyy="1.0" iyz="0.0"
-          izz="1.0" />
+        <inertia ixx="0.0001" ixy="0.0" ixz="0.0"
+          iyy="0.0001" iyz="0.0"
+          izz="0.0001" />
       </inertial>
       <visual>
@@ -67,9 +67,9 @@
     <link name="standoff_2in_${number}_link">
       <inertial>
-        <mass value="0.00001" />
+        <mass value="0.001" />
         <origin xyz="0 0 0" />
-        <inertia ixx="1.0" ixy="0.0" ixz="0.0"
-          iyy="1.0" iyz="0.0"
-          izz="1.0" />
+        <inertia ixx="0.0001" ixy="0.0" ixz="0.0"
+          iyy="0.0001" iyz="0.0"
+          izz="0.0001" />
       </inertial>
       <visual>
@@ -95,9 +95,9 @@
     <link name="standoff_8in_${number}_link">
       <inertial>
-        <mass value="0.00001" />
+        <mass value="0.001" />
         <origin xyz="0 0 0" />
-        <inertia ixx="1.0" ixy="0.0" ixz="0.0"
-          iyy="1.0" iyz="0.0"
-          izz="1.0" />
+        <inertia ixx="0.0001" ixy="0.0" ixz="0.0"
+          iyy="0.0001" iyz="0.0"
+          izz="0.0001" />
       </inertial>
       <visual>
@@ -123,9 +123,9 @@
     <link name="standoff_kinect_${number}_link">
       <inertial>
-        <mass value="0.00001" />
+        <mass value="0.001" />
         <origin xyz="0 0 0" />
-        <inertia ixx="1.0" ixy="0.0" ixz="0.0"
-          iyy="1.0" iyz="0.0"
-          izz="1.0" />
+        <inertia ixx="0.0001" ixy="0.0" ixz="0.0"
+          iyy="0.0001" iyz="0.0"
+          izz="0.0001" />
       </inertial>
       <visual>

Commit message: making casters fixed.  fix simulation params, now the robot is controllable.

File: turtlebot_description/urdf/gazebo.urdf.xacro (robot description, xacro)
@@ -106,16 +106,16 @@
   </gazebo>
   <gazebo reference="left_wheel_link">
-    <mu1 value="10.0"/>
-    <mu2 value="0.5"/>
+    <mu1 value="10"/>
+    <mu2 value="10"/>
     <kp value="100000000.0"/>
     <kd value="10000.0"/>
-    <fdir1 value="0 1 0"/>
+    <fdir value="1 0 0"/>
   </gazebo>
   <gazebo reference="right_wheel_link">
-    <mu1 value="10.0"/>
-    <mu2 value="0.5"/>
+    <mu1 value="10"/>
+    <mu2 value="10"/>
     <kp value="100000000.0"/>
     <kd value="10000.0"/>
-    <fdir1 value="0 1 0"/>
+    <fdir value="1 0 0"/>
   </gazebo>
   <gazebo reference="rear_wheel_link">
@@ -123,5 +123,5 @@
     <mu2 value="0"/>
     <kp value="100000000.0"/>
-    <kd value="1000.0"/>
+    <kd value="10000.0"/>
   </gazebo>
   <gazebo reference="front_wheel_link">
@@ -129,5 +129,5 @@
     <mu2 value="0"/>
     <kp value="100000000.0"/>
-    <kd value="1000.0"/>
+    <kd value="10000.0"/>
   </gazebo>
 </robot>

File: turtlebot_description/urdf/turtlebot.xacro (robot description, xacro)
@@ -37,8 +37,8 @@
   <link name="base_link">
     <inertial>
-      <mass value="1" />
-      <origin xyz="0 0 0.0308" />
-      <inertia ixx="0.1" ixy="0.0" ixz="0.0"
-        iyy="0.1" iyz="0.0" izz="0.1" />
+      <mass value="2" />
+      <origin xyz="0 0 0.0" />
+      <inertia ixx="0.01" ixy="0.0" ixz="0.0"
+        iyy="0.01" iyz="0.0" izz="0.5" />
     </inertial>
     <visual>
@@ -51,5 +51,5 @@
       <origin xyz="0.0 0.0 0.0308" rpy="0 0 0" />
       <geometry>
-        <cylinder length="0.0611632" radius="0.16495"/>
+        <cylinder length="0.0611632" radius="0.016495"/>
       </geometry>
     </collision>
@@ -84,5 +84,5 @@
       <origin xyz="0 0 0"/>
       <inertia ixx="1.0" ixy="0.0" ixz="0.0"
-        iyy="0.1" iyz="0.0" izz="0.1" />
+        iyy="0.01" iyz="0.0" izz="0.01" />
     </inertial>
   </link>
@@ -187,15 +187,15 @@
       <origin xyz="0 0 0" rpy="0 1.5707 1.5707"/>
       <geometry>
-        <sphere radius="0.018" />
-      </geometry>
-    </visual>
-    <collision>
-      <origin xyz="0 0 0" rpy="0 1.5707 1.5707" />
-      <geometry>
-        <sphere radius="0.018" />
-      </geometry>
-    </collision>
-  </link>
-  <!-- not sure why this is set to fixed -->
+        <sphere radius="0.015" />
+      </geometry>
+    </visual>
+    <collision>
+      <origin xyz="0 0 0" rpy="0 1.5707 1.5707" />
+      <geometry>
+        <sphere radius="0.015" />
+      </geometry>
+    </collision>
+  </link>
+  <!-- fixed because there's no transmission -->
   <joint name="rear_castor_joint" type="fixed">
     <origin xyz="-0.13 0 0.0" rpy="0 0 0"/>
@@ -224,5 +224,6 @@
     </collision>
   </link>
-  <joint name="front_castor_joint" type="continuous">
+  <!-- fixed because there's no transmission -->
+  <joint name="front_castor_joint" type="fixed">
     <origin xyz="0.13 0 0.0" rpy="0 0 0"/>
     <parent link="base_link"/>
@@ -283,7 +284,7 @@
       <mass value="0.01" />
       <origin xyz="0 0 0" />
-      <inertia ixx="0.1" ixy="0.0" ixz="0.0"
-        iyy="0.1" iyz="0.0"
-        izz="0.1" />
+      <inertia ixx="0.01" ixy="0.0" ixz="0.0"
+        iyy="0.01" iyz="0.0"
+        izz="0.01" />
     </inertial>
     <visual>
