Commit message: Refactored URDF for TBot to allow replacement of Kinect
--HG--
branch : tbot_improve
rename : turtlebot_description/urdf/turtlebot_hardware.xacro => turtlebot_description/urdf/turtlebot_hardware.urdf.xacro

File: turtlebot_description/urdf/gazebo.urdf.xacro (robot description, xacro)
@@ -1,4 +1,70 @@
 <?xml version="1.0"?>
-<robot xmlns:controller="http://playerstage.sourceforge.net/gazebo/xmlschema/#controller" xmlns:interface="http://playerstage.sourceforge.net/gazebo/xmlschema/#interface" xmlns:sensor="http://playerstage.sourceforge.net/gazebo/xmlschema/#sensor" name="turtlebot_gazebo">
+<robot xmlns:controller="http://playerstage.sourceforge.net/gazebo/xmlschema/#controller" xmlns:interface="http://playerstage.sourceforge.net/gazebo/xmlschema/#interface" xmlns:sensor="http://playerstage.sourceforge.net/gazebo/xmlschema/#sensor" xmlns:xacro="http://ros.org/wiki/xacro" name="turtlebot_gazebo">
+<xacro:macro name="turtlebot_sim_kinect">
+  <gazebo reference="kinect_link">
+    <sensor:camera name="kinect_camera">
+      <imageFormat>R8G8B8</imageFormat>
+      <imageSize>640 480</imageSize>
+      <hfov>60</hfov>
+      <nearClip>0.05</nearClip>
+      <farClip>3</farClip>
+      <updateRate>20</updateRate>
+      <baseline>0.1</baseline>
+      <controller:gazebo_ros_openni_kinect name="kinect_camera_controller" plugin="libgazebo_ros_openni_kinect.so">
+        <alwaysOn>true</alwaysOn>
+        <updateRate>20</updateRate>
+        <imageTopicName>/camera/image_raw</imageTopicName>
+        <pointCloudTopicName>/camera/depth/points</pointCloudTopicName>
+        <cameraInfoTopicName>/camera/camera_info</cameraInfoTopicName>
+        <frameName>kinect_depth_optical_frame</frameName>
+        <distortion_k1>0.0</distortion_k1>
+        <distortion_k2>0.0</distortion_k2>
+        <distortion_k3>0.0</distortion_k3>
+        <distortion_t1>0.0</distortion_t1>
+        <distortion_t2>0.0</distortion_t2>
+      </controller:gazebo_ros_openni_kinect>
+    </sensor:camera>
+  </gazebo>
+</xacro:macro>
+<xacro:macro name="turtlebot_sim_imu">
+  <gazebo>
+    <controller:gazebo_ros_imu name="imu_controller" plugin="libgazebo_ros_imu.so">
+      <alwaysOn>true</alwaysOn>
+      <updateRate>30</updateRate>
+      <bodyName>gyro_link</bodyName>
+      <topicName>imu/data</topicName>
+      <gaussianNoise>${0.0017*0.0017}</gaussianNoise>
+      <xyzOffsets>0 0 0</xyzOffsets>
+      <rpyOffsets>0 0 0</rpyOffsets>
+      <interface:position name="imu_position"/>
+    </controller:gazebo_ros_imu>
+  </gazebo>
+</xacro:macro>
+<xacro:macro name="turtlebot_sim_laser">
+  <gazebo reference="laser">
+    <sensor:ray name="laser">
+      <rayCount>180</rayCount>
+      <rangeCount>180</rangeCount>
+      <laserCount>1</laserCount>
+      <origin>0.0 0.0 0.0</origin>
+      <displayRays>false</displayRays>
+      <minAngle>-130</minAngle>
+      <maxAngle>130</maxAngle>
+      <minRange>0.08</minRange>
+      <maxRange>10.0</maxRange>
+      <resRange>0.01</resRange>
+      <updateRate>20</updateRate>
+      <controller:gazebo_ros_laser name="gazebo_ros_laser_controller" plugin="libgazebo_ros_laser.so">
+	<gaussianNoise>0.005</gaussianNoise>
+	<alwaysOn>true</alwaysOn>
+	<updateRate>20</updateRate>
+	<topicName>scan</topicName>
+	<frameName>laser</frameName>
+	<interface:laser name="gazebo_ros_laser_iface" />
+      </controller:gazebo_ros_laser>
+    </sensor:ray>
+  </gazebo>
+</xacro:macro>
+<xacro:macro name="turtlebot_sim_create">
   <gazebo>
     <controller:gazebo_ros_create name="create_controller" plugin="libgazebo_ros_create.so">
@@ -16,4 +82,6 @@
     </controller:gazebo_ros_create>
   </gazebo>
+</xacro:macro>
+<xacro:macro name="turtlebot_sim_wall_sensors">
   <gazebo reference="wall_sensor_link">
     <sensor:ray name="wall_sensor">
@@ -81,28 +149,4 @@
     </sensor:ray>
   </gazebo>
-  <gazebo reference="kinect_link">
-    <sensor:camera name="kinect_camera">
-      <imageFormat>R8G8B8</imageFormat>
-      <imageSize>640 480</imageSize>
-      <hfov>60</hfov>
-      <nearClip>0.05</nearClip>
-      <farClip>3</farClip>
-      <updateRate>20</updateRate>
-      <baseline>0.1</baseline>
-      <controller:gazebo_ros_openni_kinect name="kinect_camera_controller" plugin="libgazebo_ros_openni_kinect.so">
-        <alwaysOn>true</alwaysOn>
-        <updateRate>20</updateRate>
-        <imageTopicName>/camera/image_raw</imageTopicName>
-        <pointCloudTopicName>/camera/depth/points</pointCloudTopicName>
-        <cameraInfoTopicName>/camera/camera_info</cameraInfoTopicName>
-        <frameName>kinect_depth_optical_frame</frameName>
-        <distortion_k1>0.00000001</distortion_k1>
-        <distortion_k2>0.00000001</distortion_k2>
-        <distortion_k3>0.00000001</distortion_k3>
-        <distortion_t1>0.00000001</distortion_t1>
-        <distortion_t2>0.00000001</distortion_t2>
-      </controller:gazebo_ros_openni_kinect>
-    </sensor:camera>
-  </gazebo>
   <gazebo reference="left_wheel_link">
     <mu1 value="10"/>
@@ -131,3 +175,4 @@
     <kd value="10000.0"/>
   </gazebo>
+</xacro:macro>
 </robot>

File: turtlebot_description/urdf/turtlebot.xacro (robot description, xacro)
@@ -5,487 +5,14 @@
        xmlns:interface="http://playerstage.sourceforge.net/gazebo/xmlschema/#interface"
        xmlns:xacro="http://ros.org/wiki/xacro">
-  <include filename="$(find turtlebot_description)/urdf/turtlebot_hardware.xacro" />
-  <include filename="$(find turtlebot_description)/urdf/gazebo.urdf.xacro"/>
-  <include filename="$(find turtlebot_description)/urdf/turtlebot_calibration.xacro" />
-  <include filename="$(find turtlebot_description)/urdf/sensors/microstrain_3dmgx2_imu.urdf.xacro"/>
-  <material name="Green">
-    <color rgba="0.0 0.8 0.0 1.0"/>
-  </material>
+  <include filename="$(find turtlebot_description)/urdf/turtlebot_hardware.urdf.xacro" />
+  <include filename="$(find turtlebot_description)/urdf/turtlebot_body.urdf.xacro" />
+  <include filename="$(find turtlebot_description)/urdf/turtlebot_kinect.urdf.xacro" />
   <property name="M_PI" value="3.14159"/>
   <property name="SCALE" value="0.0254"/>
-  <property name="base_x" value="0.33" />
-  <property name="base_y" value="0.33" />
   <xacro:macro name="turtlebot">
-  <!-- base_footprint is a fictitious link(frame) that is on the ground right below base_link origin, navigation stack depends on this frame -->
-  <link name="base_footprint">
-    <inertial>
-      <mass value="0.0001" />
-      <origin xyz="0 0 0" />
-      <inertia ixx="0.0001" ixy="0.0" ixz="0.0"
-              iyy="0.0001" iyz="0.0"
-              izz="0.0001" />
-    </inertial>
-    <visual>
-      <origin xyz="0 0 0" rpy="0 0 0" />
-      <geometry>
-        <box size="0.001 0.001 0.001" />
-      </geometry>
-      <material name="Green" />
-    </visual>
-    <collision>
-      <origin xyz="0 0 0.017" rpy="0 0 0" />
-      <geometry>
-       <box size="0.001 0.001 0.001" />
-      </geometry>
-    </collision>
-  </link>
-  <link name="base_link">
-    <inertial>
-      <mass value="2" />
-      <origin xyz="0 0 0.0" />
-      <inertia ixx="0.01" ixy="0.0" ixz="0.0"
-        iyy="0.01" iyz="0.0" izz="0.5" />
-    </inertial>
-    <visual>
-      <origin xyz=" 0 0 0.0308" rpy="0 0 0" />
-      <geometry>
-        <mesh filename="package://turtlebot_description/meshes/create_body.dae"/>
-      </geometry>
-    </visual>
-    <collision>
-      <origin xyz="0.0 0.0 0.0308" rpy="0 0 0" />
-      <geometry>
-        <cylinder length="0.0611632" radius="0.016495"/>
-      </geometry>
-    </collision>
-  </link>
-  <link name="wall_sensor_link">
-    <inertial>
-      <mass value="0.01" />
-      <origin xyz="0 0 0"/>
-      <inertia ixx="0.001" ixy="0.0" ixz="0.0"
-        iyy="0.001" iyz="0.0" izz="0.001" />
-    </inertial>
-  </link>
-  <link name="left_cliff_sensor_link">
-    <inertial>
-      <mass value="0.01" />
-      <origin xyz="0 0 0"/>
-      <inertia ixx="0.001" ixy="0.0" ixz="0.0"
-        iyy="0.001" iyz="0.0" izz="0.001" />
-    </inertial>
-  </link>
-  <link name="right_cliff_sensor_link">
-    <inertial>
-      <mass value="0.01" />
-      <origin xyz="0 0 0"/>
-      <inertia ixx="0.001" ixy="0.0" ixz="0.0"
-        iyy="0.001" iyz="0.0" izz="0.001" />
-    </inertial>
-  </link>
-  <link name="leftfront_cliff_sensor_link">
-    <inertial>
-      <mass value="0.01" />
-      <origin xyz="0 0 0"/>
-      <inertia ixx="1.0" ixy="0.0" ixz="0.0"
-        iyy="0.01" iyz="0.0" izz="0.01" />
-    </inertial>
-  </link>
-  <link name="rightfront_cliff_sensor_link">
-    <inertial>
-      <mass value="0.01" />
-      <origin xyz="0 0 0"/>
-      <inertia ixx="0.001" ixy="0.0" ixz="0.0"
-        iyy="0.001" iyz="0.0" izz="0.001" />
-    </inertial>
-  </link>
-  <joint name="base_footprint_joint" type="fixed">
-    <origin xyz="0 0 0.017" rpy="0 0 0" />
-    <parent link="base_footprint"/>
-    <child link="base_link" />
-  </joint>
-  <joint name="base_wall_sensor_joint" type="fixed">
-    <origin xyz="0.09 -0.120 0.042" rpy="0 0 -1.0" />
-    <parent link="base_link"/>
-    <child link="wall_sensor_link" />
-  </joint>
-  <joint name="base_left_cliff_sensor_joint" type="fixed">
-    <origin xyz="0.07 0.14 0.01" rpy="0 1.57079 0" />
-    <parent link="base_link"/>
-    <child link="left_cliff_sensor_link" />
-  </joint>
-  <joint name="base_right_cliff_sensor_joint" type="fixed">
-    <origin xyz="0.07 -0.14 0.01" rpy="0 1.57079 0" />
-    <parent link="base_link"/>
-    <child link="right_cliff_sensor_link" />
-  </joint>
-  <joint name="base_leftfront_cliff_sensor_joint" type="fixed">
-    <origin xyz="0.15 0.04 0.01" rpy="0 1.57079 0" />
-    <parent link="base_link"/>
-    <child link="leftfront_cliff_sensor_link" />
-  </joint>
-  <joint name="base_rightfront_cliff_sensor_joint" type="fixed">
-    <origin xyz="0.15 -0.04 0.01" rpy="0 1.57079 0" />
-    <parent link="base_link"/>
-    <child link="rightfront_cliff_sensor_link" />
-  </joint>
-  <link name="left_wheel_link">
-    <inertial>
-      <origin xyz="0 0 0"/>
-      <mass value="0.01" />
-      <inertia ixx="0.001" ixy="0.0" ixz="0.0"
-        iyy="0.001" iyz="0.0" izz="0.001" />
-    </inertial>
-    <visual>
-      <origin xyz="0 0 0" rpy="0 1.5707 1.5707" />
-      <geometry>
-        <cylinder radius="0.033" length = "0.023"/>
-      </geometry>
-    </visual>
-    <collision>
-      <origin xyz="0 0 0" rpy="0 1.5707 1.5707" />
-      <geometry>
-        <cylinder radius="0.033" length = "0.023"/>
-      </geometry>
-    </collision>
-  </link>
-  <joint name="left_wheel_joint" type="continuous">
-    <origin xyz="0 0.13 0.015" rpy="0 0 0"/>
-    <parent link="base_link"/>
-    <child link="left_wheel_link"/>
-    <axis xyz="0 1 0"/>
-  </joint>
-  <link name="right_wheel_link">
-    <inertial>
-      <origin xyz="0 0 0"/>
-      <mass value="0.01" />
-      <inertia ixx="0.001" ixy="0.0" ixz="0.0"
-        iyy="0.001" iyz="0.0" izz="0.001" />
-    </inertial>
-    <visual>
-      <origin xyz="0 0 0" rpy="0 1.5707 1.5707" />
-      <geometry>
-        <cylinder radius="0.033" length = "0.023"/>
-      </geometry>
-    </visual>
-    <collision>
-      <origin xyz="0 0 0" rpy="0 1.5707 1.5707" />
-      <geometry>
-        <cylinder radius="0.033" length = "0.023"/>
-      </geometry>
-    </collision>
-  </link>
-  <joint name="right_wheel_joint" type="continuous">
-    <origin xyz="0 -0.13 0.015" rpy="0 0 0"/>
-    <parent link="base_link"/>
-    <child link="right_wheel_link"/>
-    <axis xyz="0 1 0"/>
-  </joint>
-  <link name="rear_wheel_link">
-    <inertial>
-      <origin xyz="0 0 0"/>
-      <mass value="0.001" />
-      <inertia ixx="0.0001" ixy="0.0" ixz="0.0"
-        iyy="0.0001" iyz="0.0" izz="0.0001" />
-    </inertial>
-    <visual>
-      <origin xyz="0 0 0" rpy="0 1.5707 1.5707"/>
-      <geometry>
-        <sphere radius="0.015" />
-      </geometry>
-    </visual>
-    <collision>
-      <origin xyz="0 0 0" rpy="0 1.5707 1.5707" />
-      <geometry>
-        <sphere radius="0.015" />
-      </geometry>
-    </collision>
-  </link>
-  <!-- fixed because there's no transmission -->
-  <joint name="rear_castor_joint" type="fixed">
-    <origin xyz="-0.13 0 0.0" rpy="0 0 0"/>
-    <parent link="base_link"/>
-    <child link="rear_wheel_link"/>
-    <axis xyz="0 1 0"/>
-  </joint>
-  <link name="front_wheel_link">
-    <inertial>
-      <origin xyz="0 0 0" />
-      <mass value="0.01" />
-      <inertia ixx="0.001" ixy="0.0" ixz="0.0"
-        iyy="0.001" iyz="0.0" izz="0.001" />
-    </inertial>
-    <visual>
-      <origin xyz="0 0 0" rpy="0 1.5707 1.5707"/>
-      <geometry>
-        <sphere radius="0.018" />
-      </geometry>
-    </visual>
-    <collision>
-      <origin xyz="0 0 0" rpy="0 1.5707 1.5707" />
-      <geometry>
-        <sphere radius="0.018" />
-      </geometry>
-    </collision>
-  </link>
-  <!-- fixed because there's no transmission -->
-  <joint name="front_castor_joint" type="fixed">
-    <origin xyz="0.13 0 0.0" rpy="0 0 0"/>
-    <parent link="base_link"/>
-    <child link="front_wheel_link"/>
-    <axis xyz="0 1 0"/>
-  </joint>
-  <turtlebot_spacer parent="base_link" number="0" x_loc="-0.00254" y_loc="0.1114679" z_loc="0.062992"/>
-  <turtlebot_spacer parent="base_link" number="1" x_loc="-0.00254" y_loc="-0.1114679" z_loc="0.062992"/>
-  <turtlebot_spacer parent="base_link" number="2" x_loc="-0.07239" y_loc="-0.1114679" z_loc="0.062992"/>
-  <turtlebot_spacer parent="base_link" number="3" x_loc="-0.07239" y_loc="0.1114679" z_loc="0.062992"/>
- <xacro:microstrain_3dmgx2_imu_v0 name="gyro" parent="base" imu_topic="imu/data" update_rate="100.0" stdev="0.00017">
-   <origin xyz="0 0 0.04" rpy="0 0 0" />
- </xacro:microstrain_3dmgx2_imu_v0>
-  <joint name="laser_joint" type="fixed">
-    <origin xyz="-0.065 0 0.075" rpy="0 0 0" />
-    <parent link="base_link" />
-    <child link="laser" />
-  </joint>
-  <link name="laser">
-    <visual>
-      <geometry>
-        <box size="0.02 0.035 0.002" />
-      </geometry>
-      <material name="Green" />
-    </visual>
-    <inertial>
-      <mass value="0.001" />
-      <origin xyz="0 0 0" />
-      <inertia ixx="0.0001" ixy="0.0" ixz="0.0"
-        iyy="0.0001" iyz="0.0"
-        izz="0.0001" />
-    </inertial>
-  </link>
-  <joint name="plate_0_joint" type="fixed">
-    <origin xyz="-0.04334 0  0.06775704" rpy="0 0 0" />
-    <parent link="base_link"/>
-    <child link="plate_0_link" />
-  </joint>
-  <link name="plate_0_link">
-    <inertial>
-      <mass value="0.01" />
-      <origin xyz="0 0 0" />
-      <inertia ixx="0.01" ixy="0.0" ixz="0.0"
-        iyy="0.01" iyz="0.0"
-        izz="0.01" />
-    </inertial>
-    <visual>
-      <origin xyz=" 0 0 0 " rpy="0 0 0" />
-      <geometry>
-        <mesh filename="package://turtlebot_description/meshes/plate_0_logo.dae"/>
-      </geometry>
-    </visual>
-    <collision>
-      <origin xyz="0.0 0.0 0.0" rpy="0 0 0" />
-      <geometry>
-        <box size="0.233502 0.314845 0.006401"/>
-      </geometry>
-    </collision>
-  </link>
-  <turtlebot_standoff_2in parent="base_link" number="0" x_loc="0.0676402" y_loc="0.1314196" z_loc="0.0709803"/>
-  <turtlebot_standoff_2in parent="base_link" number="1" x_loc="0.0676402" y_loc="-0.1314196" z_loc="0.0709803"/>
-  <turtlebot_standoff_2in parent="base_link" number="2" x_loc="-0.052832" y_loc="-0.1314196" z_loc="0.0709803"/>
-  <turtlebot_standoff_2in parent="base_link" number="3" x_loc="-0.052832" y_loc="0.1314196" z_loc="0.0709803"/>
-  <joint name="plate_1_joint" type="fixed">
-    <origin xyz="0.04068 0 0.05715" rpy="0 0 0" />
-    <parent link="plate_0_link"/>
-    <child link="plate_1_link" />
-  </joint>
-  <link name="plate_1_link">
-    <inertial>
-      <mass value="0.1" />
-      <origin xyz="0 0 0" />
-      <inertia ixx="0.01" ixy="0.0" ixz="0.0"
-        iyy="0.01" iyz="0.0"
-        izz="0.01" />
-    </inertial>
-    <visual>
-      <origin xyz=" 0 0 0 " rpy="0 0 0" />
-      <geometry>
-        <mesh filename="package://turtlebot_description/meshes/plate_1_logo.dae"/>
-      </geometry>
-    </visual>
-    <collision>
-      <origin xyz="0.0 0.0 0.0" rpy="0 0 0" />
-      <geometry>
-        <box size="0.314856 0.314856 0.006401"/>
-      </geometry>
-    </collision>
-  </link>
-  <turtlebot_standoff_2in parent="standoff_2in_0_link" number="4" x_loc="0" y_loc="0" z_loc="0.05715"/>
-  <turtlebot_standoff_2in parent="standoff_2in_1_link" number="5" x_loc="0" y_loc="0" z_loc="0.05715"/>
-  <turtlebot_standoff_2in parent="standoff_2in_2_link" number="6" x_loc="0" y_loc="0" z_loc="0.05715"/>
-  <turtlebot_standoff_2in parent="standoff_2in_3_link" number="7" x_loc="0" y_loc="0" z_loc="0.05715"/>
-  <joint name="plate_2_joint" type="fixed">
-    <origin xyz="0 0 0.0572008" rpy="0 0 0" />
-    <parent link="plate_1_link"/>
-    <child link="plate_2_link" />
-  </joint>
-  <link name="plate_2_link">
-    <inertial>
-      <mass value="0.01" />
-      <origin xyz="0 0 0" />
-      <inertia ixx="0.001" ixy="0.0" ixz="0.0"
-        iyy="0.001" iyz="0.0"
-        izz="0.001" />
-    </inertial>
-    <visual>
-      <origin xyz=" 0 0 0 " rpy="0 0 0" />
-      <geometry>
-        <mesh filename="package://turtlebot_description/meshes/plate_1_logo.dae"/>
-      </geometry>
-    </visual>
-    <collision>
-      <origin xyz="0.0 0.0 0.0" rpy="0 0 0" />
-      <geometry>
-        <box size="0.314856 0.314856 0.006401"/>
-      </geometry>
-    </collision>
-  </link>
-  <joint name="base_kinect_joint" type="fixed">
-    <origin xyz="${turtlebot_calib_cam_x} ${turtlebot_calib_cam_y} ${turtlebot_calib_cam_z}"
-            rpy="${turtlebot_calib_cam_rr} ${turtlebot_calib_cam_rp} ${turtlebot_calib_cam_ry}" />
-    <parent link="${turtlebot_kinect_frame_name}" />
-    <child link="kinect_link" />
-  </joint>
-  <link name="kinect_link">
-    <inertial>
-      <mass value="0.01" />
-      <origin xyz="0 0 0" />
-      <inertia ixx="0.001" ixy="0.0" ixz="0.0"
-        iyy="0.001" iyz="0.0"
-        izz="0.001" />
-    </inertial>
-    <visual>
-      <origin xyz=" 0 0 0 " rpy="0 0 0" />
-      <geometry>
-        <mesh filename="package://turtlebot_description/meshes/kinect.dae"/>
-      </geometry>
-    </visual>
-    <collision>
-      <origin xyz="0.0 0.0 0.0" rpy="0 0 0" />
-      <geometry>
-        <box size="0.0730 .2760 0.0720"/>
-      </geometry>
-    </collision>
-  </link>
-  <joint name="kinect_depth_joint" type="fixed">
-    <origin xyz="0 0.018 0" rpy="0 0 0" />
-    <parent link="kinect_link" />
-    <child link="kinect_depth_frame" />
-  </joint>
-  <link name="kinect_depth_frame">
-    <inertial>
-      <mass value="0.01" />
-      <origin xyz="0 0 0" />
-      <inertia ixx="0.001" ixy="0.0" ixz="0.0"
-        iyy="0.001" iyz="0.0"
-        izz="0.001" />
-    </inertial>
-  </link>
-  <joint name="kinect_depth_optical_joint" type="fixed">
-    <origin xyz="0 0 0" rpy="${-M_PI/2} 0 ${-M_PI/2}" />
-    <parent link="kinect_depth_frame" />
-    <child link="kinect_depth_optical_frame" />
-  </joint>
-  <link name="kinect_depth_optical_frame">
-    <inertial>
-      <mass value="0.001" />
-      <origin xyz="0 0 0" />
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