Commit message: cleanup kinect/camera naming stuffs

File: turtlebot_description/urdf/asus_xtion_pro.urdf.xacro (robot description, xacro)
@@ -6,11 +6,11 @@
 <!-- Macro for ASUS Xtion PRO on Turtlebot. Uses Kinect frame names, but they have moved -->
 <xacro:macro name="turtlebot_xtion_pro">
-  <joint name="base_kinect_joint" type="fixed">
+  <joint name="base_camera_joint" type="fixed">
     <origin xyz="${turtlebot_calib_cam_x} ${turtlebot_calib_cam_y} 0.124"
             rpy="${turtlebot_calib_cam_rr} ${turtlebot_calib_cam_rp} ${turtlebot_calib_cam_ry}" />
-    <parent link="${turtlebot_kinect_frame_name}" />
-    <child link="kinect_link" />
+    <parent link="${turtlebot_camera_parent_name}" />
+    <child link="camera_link" />
   </joint>
-  <link name="kinect_link">
+  <link name="camera_link">
     <inertial>
       <mass value="0.01" />
@@ -33,10 +33,10 @@
     </collision>
   </link>
-  <joint name="kinect_depth_joint" type="fixed">
+  <joint name="camera_depth_joint" type="fixed">
     <origin xyz="0 0.049 0" rpy="0 0 0" />
-    <parent link="kinect_link" />
-    <child link="kinect_depth_frame" />
+    <parent link="camera_link" />
+    <child link="camera_depth_frame" />
   </joint>
-  <link name="kinect_depth_frame">
+  <link name="camera_depth_frame">
     <inertial>
       <mass value="0.01" />
@@ -47,10 +47,10 @@
     </inertial>
   </link>
-  <joint name="kinect_depth_optical_joint" type="fixed">
+  <joint name="camera_depth_optical_joint" type="fixed">
     <origin xyz="0 0 0" rpy="${-M_PI/2} 0 ${-M_PI/2}" />
-    <parent link="kinect_depth_frame" />
-    <child link="kinect_depth_optical_frame" />
+    <parent link="camera_depth_frame" />
+    <child link="camera_depth_optical_frame" />
   </joint>
-  <link name="kinect_depth_optical_frame">
+  <link name="camera_depth_optical_frame">
     <inertial>
       <mass value="0.001" />
@@ -61,10 +61,10 @@
     </inertial>
   </link>
-  <joint name="kinect_rgb_joint" type="fixed">
+  <joint name="camera_rgb_joint" type="fixed">
     <origin xyz="0 0.022 0" rpy="0 0 0" />
-    <parent link="kinect_link" />
-    <child link="kinect_rgb_frame" />
+    <parent link="camera_link" />
+    <child link="camera_rgb_frame" />
   </joint>
-  <link name="kinect_rgb_frame">
+  <link name="camera_rgb_frame">
     <inertial>
       <mass value="0.001" />
@@ -75,10 +75,10 @@
     </inertial>
   </link>
-  <joint name="kinect_rgb_optical_joint" type="fixed">
+  <joint name="camera_rgb_optical_joint" type="fixed">
     <origin xyz="0 0 0" rpy="${-M_PI/2} 0 ${-M_PI/2}" />
-    <parent link="kinect_rgb_frame" />
-    <child link="kinect_rgb_optical_frame" />
+    <parent link="camera_rgb_frame" />
+    <child link="camera_rgb_optical_frame" />
   </joint>
-  <link name="kinect_rgb_optical_frame">
+  <link name="camera_rgb_optical_frame">
     <inertial>
       <mass value="0.001" />

File: turtlebot_description/urdf/turtlebot_calibration.xacro (robot description, xacro)
@@ -7,4 +7,4 @@
   <property name="turtlebot_calib_cam_rp" value="0" />
   <property name="turtlebot_calib_cam_ry" value="0" />
-  <property name="turtlebot_kinect_frame_name" value="plate_2_link" />
+  <property name="turtlebot_camera_parent_name" value="plate_2_link" />
 </robot>

File: turtlebot_description/urdf/turtlebot_kinect.urdf.xacro (robot description, xacro)
@@ -5,11 +5,11 @@
   <include filename="$(find turtlebot_description)/urdf/turtlebot_calibration.xacro" />
 <xacro:macro name="turtlebot_kinect">
-  <joint name="base_kinect_joint" type="fixed">
+  <joint name="base_camera_joint" type="fixed">
     <origin xyz="${turtlebot_calib_cam_x} ${turtlebot_calib_cam_y} ${turtlebot_calib_cam_z}"
             rpy="${turtlebot_calib_cam_rr} ${turtlebot_calib_cam_rp} ${turtlebot_calib_cam_ry}" />
-    <parent link="${turtlebot_kinect_frame_name}" />
-    <child link="kinect_link" />
+    <parent link="${turtlebot_camera_parent_name}" />
+    <child link="camera_link" />
   </joint>
-  <link name="kinect_link">
+  <link name="camera_link">
     <inertial>
       <mass value="0.01" />
@@ -32,10 +32,10 @@
     </collision>
   </link>
-  <joint name="kinect_depth_joint" type="fixed">
+  <joint name="camera_depth_joint" type="fixed">
     <origin xyz="0 0.018 0" rpy="0 0 0" />
-    <parent link="kinect_link" />
-    <child link="kinect_depth_frame" />
+    <parent link="camera_link" />
+    <child link="camera_depth_frame" />
   </joint>
-  <link name="kinect_depth_frame">
+  <link name="camera_depth_frame">
     <inertial>
       <mass value="0.01" />
@@ -46,10 +46,10 @@
     </inertial>
   </link>
-  <joint name="kinect_depth_optical_joint" type="fixed">
+  <joint name="camera_depth_optical_joint" type="fixed">
     <origin xyz="0 0 0" rpy="${-M_PI/2} 0 ${-M_PI/2}" />
-    <parent link="kinect_depth_frame" />
-    <child link="kinect_depth_optical_frame" />
+    <parent link="camera_depth_frame" />
+    <child link="camera_depth_optical_frame" />
   </joint>
-  <link name="kinect_depth_optical_frame">
+  <link name="camera_depth_optical_frame">
     <inertial>
       <mass value="0.001" />
@@ -60,10 +60,10 @@
     </inertial>
   </link>
-  <joint name="kinect_rgb_joint" type="fixed">
+  <joint name="camera_rgb_joint" type="fixed">
     <origin xyz="0 -0.005 0" rpy="0 0 0" />
-    <parent link="kinect_link" />
-    <child link="kinect_rgb_frame" />
+    <parent link="camera_link" />
+    <child link="camera_rgb_frame" />
   </joint>
-  <link name="kinect_rgb_frame">
+  <link name="camera_rgb_frame">
     <inertial>
       <mass value="0.001" />
@@ -74,10 +74,10 @@
     </inertial>
   </link>
-  <joint name="kinect_rgb_optical_joint" type="fixed">
+  <joint name="camera_rgb_optical_joint" type="fixed">
     <origin xyz="0 0 0" rpy="${-M_PI/2} 0 ${-M_PI/2}" />
-    <parent link="kinect_rgb_frame" />
-    <child link="kinect_rgb_optical_frame" />
+    <parent link="camera_rgb_frame" />
+    <child link="camera_rgb_optical_frame" />
   </joint>
-  <link name="kinect_rgb_optical_frame">
+  <link name="camera_rgb_optical_frame">
     <inertial>
       <mass value="0.001" />
