Commit message: adds minor name adjustments

File: turtlebot_description/urdf/kinect_turtlebot2.urdf.xacro (robot description, xacro)
@@ -7,6 +7,5 @@
                                 xmlns:interface="http://playerstage.sourceforge.net/gazebo/xmlschema/#interface"
                                 xmlns:sensor="http://playerstage.sourceforge.net/gazebo/xmlschema/#sensor">
-  <include filename="$(find kobuki_description)/urdf/common_properties.urdf.xacro"/>
-<!--   <include filename="$(find kobuki_description)/urdf/kobuki_gazebo.urdf.xacro"/> -->
+  <include filename="$(find turtlebot_description)/urdf/common_properties.urdf.xacro"/>
   <!-- Xacro properties -->
   <xacro:property name="M_SCALE" value="0.001"/>
@@ -28,5 +27,5 @@
         <origin xyz="0 0 0" rpy="${-M_PI/2} 0 0"/>
         <geometry>
-          <mesh filename="package://kobuki_description/meshes/turtlebot2_stack/high_res/poll_kinect.stl" scale="${M_SCALE} ${M_SCALE} ${M_SCALE}"/>
+          <mesh filename="package://turtlebot_description/meshes/turtlebot2_stack/pole_kinect.stl" scale="${M_SCALE} ${M_SCALE} ${M_SCALE}"/>
         </geometry>
         <xacro:insert_block name="material_light_grey"/>
@@ -60,5 +59,5 @@
 	      <origin xyz="0 0 0" rpy="0 0 0"/>
 	      <geometry>
-	        <mesh filename="package://kobuki_description/meshes/kinect.dae"/>
+	        <mesh filename="package://turtlebot_description/meshes/kinect.dae"/>
 	      </geometry>
         <xacro:insert_block name="material_light_grey"/>

File: turtlebot_description/urdf/turtlebot2_stack.urdf.xacro (robot description, xacro)
@@ -4,5 +4,5 @@
  -->
 <robot name="turtlebot2_stack" xmlns:xacro="http://ros.org/wiki/xacro">
-  <include filename="$(find kobuki_description)/urdf/common_properties.urdf.xacro"/>
+  <include filename="$(find turtlebot_description)/urdf/common_properties.urdf.xacro"/>
   <!-- Xacro properties -->
   <xacro:property name="M_SCALE" value="0.001"/>
@@ -18,5 +18,5 @@
         <origin xyz="0 0 0" rpy="${M_PI/2} 0 ${M_PI/2}"/>
         <geometry>
-          <mesh filename="package://kobuki_description/meshes/turtlebot2_stack/high_res/poll_1st.stl" scale="${M_SCALE} ${M_SCALE} ${M_SCALE}"/>
+          <mesh filename="package://turtlebot_description/meshes/turtlebot2_stack/pole_bottom.stl" scale="${M_SCALE} ${M_SCALE} ${M_SCALE}"/>
         </geometry>
         <xacro:insert_block name="material_light_grey"/>
@@ -47,5 +47,5 @@
         <origin xyz="0 0 0" rpy="${-M_PI/2} 0 0"/>
         <geometry>
-          <mesh filename="package://kobuki_description/meshes/turtlebot2_stack/high_res/poll_2nd.stl" scale="${M_SCALE} ${M_SCALE} ${M_SCALE}"/>
+          <mesh filename="package://turtlebot_description/meshes/turtlebot2_stack/pole_middle.stl" scale="${M_SCALE} ${M_SCALE} ${M_SCALE}"/>
         </geometry>
         <xacro:insert_block name="material_light_grey"/>
@@ -76,5 +76,5 @@
         <origin xyz=" 0 0 0" rpy="${M_PI/2} 0 ${M_PI/2}"/>
         <geometry>
-          <mesh filename="package://kobuki_description/meshes/turtlebot2_stack/high_res/poll_3rd.stl" scale="${M_SCALE} ${M_SCALE} ${M_SCALE}"/>
+          <mesh filename="package://turtlebot_description/meshes/turtlebot2_stack/pole_top.stl" scale="${M_SCALE} ${M_SCALE} ${M_SCALE}"/>
         </geometry>
         <xacro:insert_block name="material_light_grey"/>
@@ -93,33 +93,4 @@
                  izz="0.0001"/>
       </inertial>
-    </link>
-  </xacro:macro>
-  <xacro:macro name="stack_xtion_pole" params="parent number x_loc y_loc z_loc">
-    <joint name="pole_xtion${number}_joint" type="fixed">
-      <origin xyz="${x_loc} ${y_loc} ${z_loc}" rpy="0 0 0"/>
-      <parent link="${parent}"/>
-      <child link="pole_xtion_${number}_link"/>
-    </joint>
-    <link name="pole_xtion_${number}_link">
-      <inertial>
-        <mass value="0.001"/>
-        <origin xyz="0 0 0"/>
-        <inertia ixx="0.0001" ixy="0.0" ixz="0.0"
-                 iyy="0.0001" iyz="0.0"
-                 izz="0.0001"/>
-      </inertial>
-      <visual>
-        <origin xyz=" 0 0 0 " rpy="0 0 0"/>
-        <geometry>
-          <mesh filename="package://kobuki_description/meshes/turtlebot2_stack/high_res/poll_kinect.stl" scale="${M_SCALE} ${M_SCALE} ${M_SCALE}"/>
-        </geometry>
-        <xacro:insert_block name="material_light_grey"/>
-      </visual>
-      <collision>
-        <origin xyz=" 0 0 0 " rpy="0 0 0"/>
-        <geometry>
-          <cylinder length="0.008585" radius="0.001111"/>
-        </geometry>
-      </collision>
     </link>
   </xacro:macro>
@@ -141,5 +112,5 @@
 		    <origin xyz="0 0 0" rpy="${M_PI/2} 0 ${M_PI/2}"/>
 		    <geometry>
-		      <mesh filename="package://kobuki_description/meshes/turtlebot2_stack/high_res/stack_1st.stl" scale="${M_SCALE} ${M_SCALE} ${M_SCALE}"/>
+		      <mesh filename="package://turtlebot_description/meshes/turtlebot2_stack/plate_bottom.stl" scale="${M_SCALE} ${M_SCALE} ${M_SCALE}"/>
 		    </geometry>
         <xacro:insert_block name="material_light_grey"/>
@@ -173,5 +144,5 @@
 		    <origin xyz="0 0 0" rpy="${M_PI/2} 0 ${M_PI/2}"/>
 		    <geometry>
-		      <mesh filename="package://kobuki_description/meshes/turtlebot2_stack/high_res/stack_2nd.stl" scale="${M_SCALE} ${M_SCALE} ${M_SCALE}"/>
+		      <mesh filename="package://turtlebot_description/meshes/turtlebot2_stack/plate_middle.stl" scale="${M_SCALE} ${M_SCALE} ${M_SCALE}"/>
 		    </geometry>
         <xacro:insert_block name="material_light_grey"/>
@@ -204,5 +175,5 @@
         <origin xyz="0 0 0" rpy="${M_PI/2} 0 ${M_PI/2}"/>
 		    <geometry>
-		      <mesh filename="package://kobuki_description/meshes/turtlebot2_stack/high_res/stack_3rd.stl" scale="${M_SCALE} ${M_SCALE} ${M_SCALE}"/>
+		      <mesh filename="package://turtlebot_description/meshes/turtlebot2_stack/plate_top.stl" scale="${M_SCALE} ${M_SCALE} ${M_SCALE}"/>
 		    </geometry>
         <xacro:insert_block name="material_light_grey"/>

File: turtlebot_description/urdf/xtion_turtlebot2.urdf.xacro (robot description, xacro)
@@ -7,6 +7,5 @@
 												       xmlns:interface="http://playerstage.sourceforge.net/gazebo/xmlschema/#interface"
 												       xmlns:sensor="http://playerstage.sourceforge.net/gazebo/xmlschema/#sensor">
-  <include filename="$(find kobuki_description)/urdf/common_properties.urdf.xacro"/>
-  <include filename="$(find kobuki_description)/urdf/kobuki_gazebo.urdf.xacro"/>
+  <include filename="$(find turtlebot_description)/urdf/common_properties.urdf.xacro"/>
   <!-- Xacro properties -->
   <xacro:property name="M_SCALE" value="0.001"/>
@@ -28,5 +27,5 @@
         <origin xyz="0 0 0" rpy="${-M_PI/2} 0 0"/>
         <geometry>
-          <mesh filename="package://kobuki_description/meshes/turtlebot2_stack/high_res/poll_kinect.stl" scale="${M_SCALE} ${M_SCALE} ${M_SCALE}"/>
+          <mesh filename="package://turtlebot_description/meshes/turtlebot2_stack/pole_kinect.stl" scale="${M_SCALE} ${M_SCALE} ${M_SCALE}"/>
         </geometry>
         <xacro:insert_block name="material_light_grey"/>
@@ -61,5 +60,5 @@
         <geometry>
           <!-- Thanks to IHeartRobotics for the Collada model! -->
-          <mesh filename="package://kobuki_description/meshes/asus_xtion_pro_live.dae" scale="${M_SCALE} ${M_SCALE} ${M_SCALE}"/>
+          <mesh filename="package://turtlebot_description/meshes/asus_xtion_pro_live.dae" scale="${M_SCALE} ${M_SCALE} ${M_SCALE}"/>
         </geometry>
         <xacro:insert_block name="material_light_grey"/>

Commit message: changes remaining kinect/xtion mentioning in the link/joint names

File: turtlebot_description/urdf/kinect_turtlebot2.urdf.xacro (robot description, xacro)
@@ -49,5 +49,5 @@
 	  <stack_kinect_pole parent="${parent}" number="0" x_loc="-0.1024" y_loc= "0.098" z_loc="0.259"/>
 	  <stack_kinect_pole parent="${parent}" number="1" x_loc="-0.1024" y_loc="-0.098" z_loc="0.259"/>
-	  <joint name="kinect_joint" type="fixed">
+	  <joint name="camera_joint" type="fixed">
 	    <origin xyz="${turtlebot2_kinect_calib_px} ${turtlebot2_kinect_calib_py} ${turtlebot2_kinect_calib_pz}"
 	            rpy="${turtlebot2_kinect_calib_or} ${turtlebot2_kinect_calib_op} ${turtlebot2_kinect_calib_oy}"/>
@@ -55,5 +55,5 @@
 	    <child link="kinect_link"/>
 	  </joint>
-	  <link name="kinect_link">
+	  <link name="camera_link">
 	    <visual>
 	      <origin xyz="0 0 0" rpy="0 0 0"/>

File: turtlebot_description/urdf/xtion_turtlebot2.urdf.xacro (robot description, xacro)
@@ -49,5 +49,5 @@
     <stack_xtion_pole parent="${parent}" number="0" x_loc="-0.1024" y_loc= "0.098" z_loc="0.259"/>
     <stack_xtion_pole parent="${parent}" number="1" x_loc="-0.1024" y_loc="-0.098" z_loc="0.259"/>
-    <joint name="xtion_joint" type="fixed">
+    <joint name="camera_joint" type="fixed">
       <origin xyz="${turtlebot2_xtion_calib_px} ${turtlebot2_xtion_calib_py} ${turtlebot2_xtion_calib_pz}"
               rpy="${turtlebot2_xtion_calib_or} ${turtlebot2_xtion_calib_op} ${turtlebot2_xtion_calib_oy}"/>
@@ -55,5 +55,5 @@
       <child link="xtion_link"/>
     </joint>
-    <link name="xtion_link">
+    <link name="camera_link">
       <visual>
         <origin xyz="0 0 0" rpy="${M_PI/2} 0 ${M_PI/2}"/>

Commit message: changes remaining kinect/xtion mentioning in the link/joint names

File: turtlebot_description/urdf/kinect_turtlebot2.urdf.xacro (robot description, xacro)
@@ -8,4 +8,5 @@
                                 xmlns:sensor="http://playerstage.sourceforge.net/gazebo/xmlschema/#sensor">
   <include filename="$(find turtlebot_description)/urdf/common_properties.urdf.xacro"/>
+  <include filename="$(find turtlebot_description)/urdf/gazebo.urdf.xacro"/>
   <!-- Xacro properties -->
   <xacro:property name="M_SCALE" value="0.001"/>
@@ -49,11 +50,11 @@
 	  <stack_kinect_pole parent="${parent}" number="0" x_loc="-0.1024" y_loc= "0.098" z_loc="0.259"/>
 	  <stack_kinect_pole parent="${parent}" number="1" x_loc="-0.1024" y_loc="-0.098" z_loc="0.259"/>
-	  <joint name="kinect_joint" type="fixed">
+	  <joint name="camera_joint" type="fixed">
 	    <origin xyz="${turtlebot2_kinect_calib_px} ${turtlebot2_kinect_calib_py} ${turtlebot2_kinect_calib_pz}"
 	            rpy="${turtlebot2_kinect_calib_or} ${turtlebot2_kinect_calib_op} ${turtlebot2_kinect_calib_oy}"/>
 	    <parent link="${parent}"/>
-	    <child link="kinect_link"/>
+	    <child link="camera_link"/>
 	  </joint>
-	  <link name="kinect_link">
+	  <link name="camera_link">
 	    <visual>
 	      <origin xyz="0 0 0" rpy="0 0 0"/>
@@ -82,5 +83,5 @@
 		<joint name="camera_depth_joint" type="fixed">
 	    <origin xyz="0 0.0125 0" rpy="0 0 0" />
-	    <parent link="kinect_link" />
+	    <parent link="camera_link" />
 	    <child link="camera_depth_frame" />
 	  </joint>
@@ -110,5 +111,5 @@
 	  <joint name="camera_rgb_joint" type="fixed">
 	    <origin xyz="0 -0.0125 0" rpy="0 0 0" />
-	    <parent link="kinect_link" />
+	    <parent link="camera_link" />
 	    <child link="camera_rgb_frame" />
 	  </joint>
@@ -137,28 +138,30 @@
 	  </link>
 	  <!-- Kinect sensor for simulation -->
-	  <gazebo reference="kinect_link">
-	    <sensor:camera name="kinect">
-	      <imageFormat>R8G8B8</imageFormat>
-	      <imageSize>640 480</imageSize>
-	      <hfov>60</hfov>
-	      <nearClip>0.05</nearClip>
-	      <farClip>3</farClip>
-	      <updateRate>20</updateRate>
-	      <baseline>0.1</baseline>
-	      <controller:gazebo_ros_openni_kinect name="kinect_controller" plugin="libgazebo_ros_openni_kinect.so">
-	        <alwaysOn>true</alwaysOn>
-	        <updateRate>20</updateRate>
-	        <imageTopicName>/camera/image_raw</imageTopicName>
-	        <pointCloudTopicName>/camera/depth/points</pointCloudTopicName>
-	        <cameraInfoTopicName>/camera/camera_info</cameraInfoTopicName>
-	        <frameName>camera_depth_optical_frame</frameName>
-	        <distortion_k1>0.0</distortion_k1>
-	        <distortion_k2>0.0</distortion_k2>
-	        <distortion_k3>0.0</distortion_k3>
-	        <distortion_t1>0.0</distortion_t1>
-	        <distortion_t2>0.0</distortion_t2>
-	      </controller:gazebo_ros_openni_kinect>
-	    </sensor:camera>
-	  </gazebo>
+	  turtlebot_sim_kinect
+	  <turtlebot_sim_kinect/>
+<!-- 	  <gazebo reference="kinect_link"> -->
+<!-- 	    <sensor:camera name="kinect"> -->
+<!-- 	      <imageFormat>R8G8B8</imageFormat> -->
+<!-- 	      <imageSize>640 480</imageSize> -->
+<!-- 	      <hfov>60</hfov> -->
+<!-- 	      <nearClip>0.05</nearClip> -->
+<!-- 	      <farClip>3</farClip> -->
+<!-- 	      <updateRate>20</updateRate> -->
+<!-- 	      <baseline>0.1</baseline> -->
+<!-- 	      <controller:gazebo_ros_openni_kinect name="kinect_controller" plugin="libgazebo_ros_openni_kinect.so"> -->
+<!-- 	        <alwaysOn>true</alwaysOn> -->
+<!-- 	        <updateRate>20</updateRate> -->
+<!-- 	        <imageTopicName>/camera/image_raw</imageTopicName> -->
+<!-- 	        <pointCloudTopicName>/camera/depth/points</pointCloudTopicName> -->
+<!-- 	        <cameraInfoTopicName>/camera/camera_info</cameraInfoTopicName> -->
+<!-- 	        <frameName>camera_depth_optical_frame</frameName> -->
+<!-- 	        <distortion_k1>0.0</distortion_k1> -->
+<!-- 	        <distortion_k2>0.0</distortion_k2> -->
+<!-- 	        <distortion_k3>0.0</distortion_k3> -->
+<!-- 	        <distortion_t1>0.0</distortion_t1> -->
+<!-- 	        <distortion_t2>0.0</distortion_t2> -->
+<!-- 	      </controller:gazebo_ros_openni_kinect> -->
+<!-- 	    </sensor:camera> -->
+<!-- 	  </gazebo> -->
 	</xacro:macro>
 </robot>

File: turtlebot_description/urdf/xtion_turtlebot2.urdf.xacro (robot description, xacro)
@@ -49,11 +49,11 @@
     <stack_xtion_pole parent="${parent}" number="0" x_loc="-0.1024" y_loc= "0.098" z_loc="0.259"/>
     <stack_xtion_pole parent="${parent}" number="1" x_loc="-0.1024" y_loc="-0.098" z_loc="0.259"/>
-    <joint name="xtion_joint" type="fixed">
+    <joint name="camera_joint" type="fixed">
       <origin xyz="${turtlebot2_xtion_calib_px} ${turtlebot2_xtion_calib_py} ${turtlebot2_xtion_calib_pz}"
               rpy="${turtlebot2_xtion_calib_or} ${turtlebot2_xtion_calib_op} ${turtlebot2_xtion_calib_oy}"/>
       <parent link="${parent}"/>
-      <child link="xtion_link"/>
+      <child link="camera_link"/>
     </joint>
-    <link name="xtion_link">
+    <link name="camera_link">
       <visual>
         <origin xyz="0 0 0" rpy="${M_PI/2} 0 ${M_PI/2}"/>
