Commit message: Fixing Turtlebot URDF to add IMU in simulation (#91), adding Hokuyo sensor to laser link
--HG--
branch : tbot_improve
rename : turtlebot_description/urdf/turtlebot.urdf.xacro => turtlebot_description/robots/turtlebot.urdf.xacro

File: turtlebot_description/robots/turtlebot.urdf.xacro (robot description, xacro)
@@ -1,4 +1,3 @@
 <?xml version="1.0"?>
-<!-- Do not use this macro, use the one in turtlebot_description/robots instead -->
 <robot name="turtlebot"
     xmlns:sensor="http://playerstage.sourceforge.net/gazebo/xmlschema/#sensor"

File: turtlebot_description/urdf/gazebo.urdf.xacro (robot description, xacro)
@@ -1,4 +1,4 @@
 <?xml version="1.0"?>
-<robot xmlns:controller="http://playerstage.sourceforge.net/gazebo/xmlschema/#controller" xmlns:interface="http://playerstage.sourceforge.net/gazebo/xmlschema/#interface" xmlns:sensor="http://playerstage.sourceforge.net/gazebo/xmlschema/#sensor">
+<robot xmlns:controller="http://playerstage.sourceforge.net/gazebo/xmlschema/#controller" xmlns:interface="http://playerstage.sourceforge.net/gazebo/xmlschema/#interface" xmlns:sensor="http://playerstage.sourceforge.net/gazebo/xmlschema/#sensor" name="turtlebot_gazebo">
   <gazebo>
     <controller:gazebo_ros_create name="create_controller" plugin="libgazebo_ros_create.so">

File: turtlebot_description/urdf/turtlebot.xacro (robot description, xacro)
@@ -1,7 +1,12 @@
 <?xml version="1.0"?>
-<robot>
+<robot name="turtlebot"
+       xmlns:sensor="http://playerstage.sourceforge.net/gazebo/xmlschema/#sensor"
+       xmlns:controller="http://playerstage.sourceforge.net/gazebo/xmlschema/#controller"
+       xmlns:interface="http://playerstage.sourceforge.net/gazebo/xmlschema/#interface"
+       xmlns:xacro="http://ros.org/wiki/xacro">
   <include filename="$(find turtlebot_description)/urdf/turtlebot_hardware.xacro" />
   <include filename="$(find turtlebot_description)/urdf/gazebo.urdf.xacro"/>
   <include filename="$(find turtlebot_description)/urdf/turtlebot_calibration.xacro" />
+  <include filename="$(find turtlebot_description)/urdf/sensors/microstrain_3dmgx2_imu.urdf.xacro"/>
   <material name="Green">
     <color rgba="0.0 0.8 0.0 1.0"/>
@@ -235,24 +240,7 @@
   <turtlebot_spacer parent="base_link" number="2" x_loc="-0.07239" y_loc="-0.1114679" z_loc="0.062992"/>
   <turtlebot_spacer parent="base_link" number="3" x_loc="-0.07239" y_loc="0.1114679" z_loc="0.062992"/>
-  <joint name="gyro_joint" type="fixed">
-    <origin xyz="0 0 0.04" rpy="0 0 0" />
-    <parent link="base_link" />
-    <child link="gyro_link" />
-  </joint>
-  <link name="gyro_link">
-    <visual>
-      <geometry>
-        <box size="0.02 0.035 0.002" />
-      </geometry>
-      <material name="Green" />
-    </visual>
-    <inertial>
-      <mass value="0.001" />
-      <origin xyz="0 0 0" />
-      <inertia ixx="0.0001" ixy="0.0" ixz="0.0"
-        iyy="0.0001" iyz="0.0"
-        izz="0.0001" />
-    </inertial>
-  </link>
+ <xacro:microstrain_3dmgx2_imu_v0 name="gyro" parent="base" imu_topic="imu/data" update_rate="100.0" stdev="0.00017">
+   <origin xyz="0 0 0.04" rpy="0 0 0" />
+ </xacro:microstrain_3dmgx2_imu_v0>
   <joint name="laser_joint" type="fixed">
     <origin xyz="-0.065 0 0.075" rpy="0 0 0" />
@@ -476,4 +464,28 @@
     </collision>
   </link>
-  </macro>
+  <!-- Hokuyo laser -->
+  <gazebo reference="laser">
+    <sensor:ray name="laser">
+      <rayCount>180</rayCount>
+      <rangeCount>180</rangeCount>
+      <laserCount>1</laserCount>
+      <origin>0.0 0.0 0.0</origin>
+      <displayRays>false</displayRays>
+      <minAngle>-130</minAngle>
+      <maxAngle>130</maxAngle>
+      <minRange>0.08</minRange>
+      <maxRange>10.0</maxRange>
+      <resRange>0.01</resRange>
+      <updateRate>20</updateRate>
+      <controller:gazebo_ros_laser name="gazebo_ros_laser_controller" plugin="libgazebo_ros_laser.so">
+	<gaussianNoise>0.005</gaussianNoise>
+	<alwaysOn>true</alwaysOn>
+	<updateRate>20</updateRate>
+	<topicName>scan</topicName>
+	<frameName>laser</frameName>
+	<interface:laser name="gazebo_ros_laser_iface" />
+      </controller:gazebo_ros_laser>
+    </sensor:ray>
+  </gazebo>
+  </macro> <!--turtlebot -->
 </robot>

Commit message: Adding TurtleBot file for ASUS Xtion PRO camera instead of Kinect.
--HG--
branch : tbot_improve
rename : turtlebot_description/robots/turtlebot.urdf.xacro => turtlebot_description/robots/turtlebot_xtion_pro.urdf.xacro
rename : turtlebot_description/urdf/turtlebot_kinect.urdf.xacro => turtlebot_description/urdf/asus_xtion_pro.urdf.xacro

File: turtlebot_description/robots/turtlebot.urdf.xacro (robot description, xacro)
@@ -1,9 +1,17 @@
 <?xml version="1.0"?>
 <robot name="turtlebot"
-    xmlns:sensor="http://playerstage.sourceforge.net/gazebo/xmlschema/#sensor"
-    xmlns:controller="http://playerstage.sourceforge.net/gazebo/xmlschema/#controller"
-    xmlns:interface="http://playerstage.sourceforge.net/gazebo/xmlschema/#interface">
-    <!-- Included URDF Files -->
-    <include filename="$(find turtlebot_description)/urdf/turtlebot.xacro" />
-    <turtlebot />
+       xmlns:sensor="http://playerstage.sourceforge.net/gazebo/xmlschema/#sensor"
+       xmlns:controller="http://playerstage.sourceforge.net/gazebo/xmlschema/#controller"
+       xmlns:interface="http://playerstage.sourceforge.net/gazebo/xmlschema/#interface"
+       xmlns:xacro="http://ros.org/wiki/xacro">
+  <include filename="$(find turtlebot_description)/urdf/turtlebot_hardware.urdf.xacro" />
+  <include filename="$(find turtlebot_description)/urdf/turtlebot_body.urdf.xacro" />
+  <include filename="$(find turtlebot_description)/urdf/turtlebot_calibration.xacro" />
+  <include filename="$(find turtlebot_description)/urdf/turtlebot_kinect.urdf.xacro" />
+  <property name="M_PI" value="3.14159"/>
+  <property name="SCALE" value="0.0254"/>
+  <!-- Body of TurtleBot, with plates, standoffs and Create (including sim sensors) -->
+  <turtlebot_body/>
+  <!-- Kinect frames and mounting (includes simulation) -->
+  <turtlebot_kinect/>
 </robot>

File: turtlebot_description/urdf/gazebo.urdf.xacro (robot description, xacro)
@@ -1,4 +1,35 @@
 <?xml version="1.0"?>
 <robot xmlns:controller="http://playerstage.sourceforge.net/gazebo/xmlschema/#controller" xmlns:interface="http://playerstage.sourceforge.net/gazebo/xmlschema/#interface" xmlns:sensor="http://playerstage.sourceforge.net/gazebo/xmlschema/#sensor" xmlns:xacro="http://ros.org/wiki/xacro" name="turtlebot_gazebo">
+<!-- ASUS Xtion PRO camera for simulation -->
+<!-- gazebo_ros_wge100 plugin is in kt2_gazebo_plugins package -->
+<xacro:macro name="turtlebot_sim_asus_xtion">
+  <gazebo reference="kinect_link" >
+    <sensor:camera name="camera" >
+      <imageSize>640 480</imageSize>
+      <imageFormat>R8G8B8</imageFormat>
+      <hfov>62.8</hfov>
+      <nearClip>0.1</nearClip>
+      <farClip>10</farClip>
+      <updateRate>2.0</updateRate>
+      <controller:gazebo_ros_wge100 name="kinect_camera_controller" plugin="libgazebo_ros_wge100.so">
+	<alwaysOn>true</alwaysOn>
+	<updateRate>5000.0</updateRate>
+	<cameraName>camera/rgb</cameraName>
+	<frameName>kinect_rgb_optical_frame</frameName>
+	<hackBaseline>0.0</hackBaseline>
+	<CxPrime>320.5</CxPrime>
+	<Cx>320.5</Cx>
+	<Cy>240.5</Cy>
+	<baseline>0.09</baseline>
+	<!-- image_width / (2*tan(hfov_radian /2)) -->
+	<!-- 320 for wide and 772.55 for narrow stereo camera -->
+	<focal_length>525</focal_length>
+	<cameraNamespace>camera/rgb</cameraNamespace>
+	<depthData>true</depthData>
+	<interface:camera name="camera_iface" />
+      </controller:gazebo_ros_wge100>
+    </sensor:camera>
+  </gazebo>
+</xacro:macro>
 <xacro:macro name="turtlebot_sim_kinect">
   <gazebo reference="kinect_link">

File: turtlebot_description/urdf/turtlebot.urdf.xacro (robot description, xacro)
@@ -1,10 +1,17 @@
 <?xml version="1.0"?>
-<!-- Do not use this macro, use the one in turtlebot_description/robots instead -->
 <robot name="turtlebot"
-    xmlns:sensor="http://playerstage.sourceforge.net/gazebo/xmlschema/#sensor"
-    xmlns:controller="http://playerstage.sourceforge.net/gazebo/xmlschema/#controller"
-    xmlns:interface="http://playerstage.sourceforge.net/gazebo/xmlschema/#interface">
-    <!-- Included URDF Files -->
-    <include filename="$(find turtlebot_description)/urdf/turtlebot.xacro" />
-    <turtlebot />
+       xmlns:sensor="http://playerstage.sourceforge.net/gazebo/xmlschema/#sensor"
+       xmlns:controller="http://playerstage.sourceforge.net/gazebo/xmlschema/#controller"
+       xmlns:interface="http://playerstage.sourceforge.net/gazebo/xmlschema/#interface"
+       xmlns:xacro="http://ros.org/wiki/xacro">
+  <include filename="$(find turtlebot_description)/urdf/turtlebot_hardware.urdf.xacro" />
+  <include filename="$(find turtlebot_description)/urdf/turtlebot_body.urdf.xacro" />
+  <include filename="$(find turtlebot_description)/urdf/turtlebot_calibration.xacro" />
+  <include filename="$(find turtlebot_description)/urdf/turtlebot_kinect.urdf.xacro" />
+  <property name="M_PI" value="3.14159"/>
+  <property name="SCALE" value="0.0254"/>
+  <!-- Body of TurtleBot, with plates, standoffs and Create (including sim sensors) -->
+  <turtlebot_body/>
+  <!-- Kinect frames and mounting (includes simulation) -->
+  <turtlebot_kinect/>
 </robot>
