Commit message: turtlebot_description: adds updates to xacros and urdfs for Gazebo simulation

File: turtlebot_description/robots/create_circles_asus_xtion_pro.urdf.xacro (robot description, xacro)
@@ -5,10 +5,6 @@
     - 3d Sensor : kinect
 -->
-<robot name="turtlebot"
-       xmlns:sensor="http://playerstage.sourceforge.net/gazebo/xmlschema/#sensor"
-       xmlns:controller="http://playerstage.sourceforge.net/gazebo/xmlschema/#controller"
-       xmlns:interface="http://playerstage.sourceforge.net/gazebo/xmlschema/#interface"
-       xmlns:xacro="http://ros.org/wiki/xacro">
-  <include filename="$(find turtlebot_description)/urdf/turtlebot_library.urdf.xacro" />
+<robot name="turtlebot" xmlns:xacro="http://ros.org/wiki/xacro">
+  <xacro:include filename="$(find turtlebot_description)/urdf/turtlebot_library.urdf.xacro" />
   <create/>
   <stack_circles parent="base_link"/>

File: turtlebot_description/robots/create_circles_kinect.urdf.xacro (robot description, xacro)
@@ -5,10 +5,6 @@
     - 3d Sensor : kinect
 -->
-<robot name="turtlebot"
-       xmlns:sensor="http://playerstage.sourceforge.net/gazebo/xmlschema/#sensor"
-       xmlns:controller="http://playerstage.sourceforge.net/gazebo/xmlschema/#controller"
-       xmlns:interface="http://playerstage.sourceforge.net/gazebo/xmlschema/#interface"
-       xmlns:xacro="http://ros.org/wiki/xacro">
-  <include filename="$(find turtlebot_description)/urdf/turtlebot_library.urdf.xacro" />
+<robot name="turtlebot" xmlns:xacro="http://ros.org/wiki/xacro">
+  <xacro:include filename="$(find turtlebot_description)/urdf/turtlebot_library.urdf.xacro" />
   <create/>
   <stack_circles parent="base_link"/>

File: turtlebot_description/robots/kobuki_hexagons_asus_xtion_pro.urdf.xacro (robot description, xacro)
@@ -5,10 +5,6 @@
     - 3d Sensor : kinect
 -->
-<robot name="turtlebot"
-       xmlns:sensor="http://playerstage.sourceforge.net/gazebo/xmlschema/#sensor"
-       xmlns:controller="http://playerstage.sourceforge.net/gazebo/xmlschema/#controller"
-       xmlns:interface="http://playerstage.sourceforge.net/gazebo/xmlschema/#interface"
-       xmlns:xacro="http://ros.org/wiki/xacro">
-  <include filename="$(find turtlebot_description)/urdf/turtlebot_library.urdf.xacro" />
+<robot name="turtlebot" xmlns:xacro="http://ros.org/wiki/xacro">
+  <xacro:include filename="$(find turtlebot_description)/urdf/turtlebot_library.urdf.xacro" />
   <kobuki/>
   <stack_hexagons         parent="base_link"/>

File: turtlebot_description/robots/kobuki_hexagons_kinect.urdf.xacro (robot description, xacro)
@@ -5,10 +5,6 @@
     - 3d Sensor : kinect
 -->
-<robot name="turtlebot"
-       xmlns:sensor="http://playerstage.sourceforge.net/gazebo/xmlschema/#sensor"
-       xmlns:controller="http://playerstage.sourceforge.net/gazebo/xmlschema/#controller"
-       xmlns:interface="http://playerstage.sourceforge.net/gazebo/xmlschema/#interface"
-       xmlns:xacro="http://ros.org/wiki/xacro">
-  <include filename="$(find turtlebot_description)/urdf/turtlebot_library.urdf.xacro" />
+<robot name="turtlebot" xmlns:xacro="http://ros.org/wiki/xacro">
+  <xacro:include filename="$(find turtlebot_description)/urdf/turtlebot_library.urdf.xacro" />
   <kobuki/>
   <stack_hexagons parent="base_link"/>

File: turtlebot_description/urdf/sensors/asus_xtion_pro.urdf.xacro (robot description, xacro)
@@ -1,11 +1,6 @@
 <?xml version="1.0"?>
-<robot name="sensor_asus_xtion_pro" xmlns:xacro="http://ros.org/wiki/xacro"
-                                    xmlns:controller="http://playerstage.sourceforge.net/gazebo/xmlschema/#controller"
-                                    xmlns:interface="http://playerstage.sourceforge.net/gazebo/xmlschema/#interface"
-                                    xmlns:sensor="http://playerstage.sourceforge.net/gazebo/xmlschema/#sensor">
-  <include filename="$(find turtlebot_description)/urdf/common_properties.urdf.xacro"/>
-  <include filename="$(find turtlebot_description)/urdf/turtlebot_gazebo.urdf.xacro"/>
-  <include filename="$(find turtlebot_description)/urdf/common_properties.urdf.xacro" />
-  <include filename="$(find turtlebot_description)/urdf/turtlebot_properties.urdf.xacro" />
+<robot name="sensor_asus_xtion_pro" xmlns:xacro="http://ros.org/wiki/xacro">
+  <xacro:include filename="$(find turtlebot_description)/urdf/turtlebot_gazebo.urdf.xacro"/>
+  <xacro:include filename="$(find turtlebot_description)/urdf/turtlebot_properties.urdf.xacro"/>f.xacro"/>
   <!-- Xacro properties -->
   <xacro:property name="M_SCALE" value="0.001"/>
@@ -98,6 +93,6 @@
       </inertial>
     </link>
-    <!-- RGBD sensor for simulation -->
-<!--     <turtlebot_sim_xtion/> not working currently -->
+  <!-- RGBD sensor for simulation, same as Kinect -->
+  <turtlebot_sim_3dsensor/>
   </xacro:macro>
 </robot>

File: turtlebot_description/urdf/sensors/kinect.urdf.xacro (robot description, xacro)
@@ -1,11 +1,6 @@
 <?xml version="1.0"?>
-<robot name="sensor_kinect" xmlns:xacro="http://ros.org/wiki/xacro"
-                            xmlns:controller="http://playerstage.sourceforge.net/gazebo/xmlschema/#controller"
-                            xmlns:interface="http://playerstage.sourceforge.net/gazebo/xmlschema/#interface"
-                            xmlns:sensor="http://playerstage.sourceforge.net/gazebo/xmlschema/#sensor">
-  <include filename="$(find turtlebot_description)/urdf/common_properties.urdf.xacro"/>
-  <include filename="$(find turtlebot_description)/urdf/turtlebot_gazebo.urdf.xacro"/>
-  <include filename="$(find turtlebot_description)/urdf/common_properties.urdf.xacro" />
-  <include filename="$(find turtlebot_description)/urdf/turtlebot_properties.urdf.xacro" />
+<robot name="sensor_kinect" xmlns:xacro="http://ros.org/wiki/xacro">
+  <xacro:include filename="$(find turtlebot_description)/urdf/turtlebot_gazebo.urdf.xacro"/>
+  <xacro:include filename="$(find turtlebot_description)/urdf/turtlebot_properties.urdf.xacro"/>
   <!-- Parameterised in part by the values in turtlebot_properties.urdf.xacro -->
   <xacro:macro name="sensor_kinect" params="parent">
@@ -96,5 +91,5 @@
 	</link>
 	<!-- Kinect sensor for simulation -->
-<!-- 	<turtlebot_sim_kinect/> not working currently -->
+	<turtlebot_sim_3dsensor/>
   </xacro:macro>
 </robot>

File: turtlebot_description/urdf/turtlebot_gazebo.urdf.xacro (robot description, xacro)
@@ -1,93 +1,78 @@
 <?xml version="1.0"?>
-<robot name="turtlebot_gazebo"
-       xmlns:controller="http://playerstage.sourceforge.net/gazebo/xmlschema/#controller"
-       xmlns:interface="http://playerstage.sourceforge.net/gazebo/xmlschema/#interface"
-       xmlns:sensor="http://playerstage.sourceforge.net/gazebo/xmlschema/#sensor"
-       xmlns:xacro="http://ros.org/wiki/xacro">
-<!-- ASUS Xtion PRO camera for simulation -->
-<!-- gazebo_ros_wge100 plugin is in kt2_gazebo_plugins package -->
-	<xacro:macro name="turtlebot_sim_xtion">
-	  <gazebo reference="camera_link" >
-	    <sensor:camera name="camera" >
-	      <imageSize>640 480</imageSize>
-	      <imageFormat>R8G8B8</imageFormat>
-	      <hfov>62.8</hfov>
-	      <nearClip>0.1</nearClip>
-	      <farClip>10</farClip>
-	      <updateRate>2.0</updateRate>
-	      <controller:gazebo_ros_wge100 name="kinect_camera_controller" plugin="libgazebo_ros_wge100.so">
-		<alwaysOn>true</alwaysOn>
-		<updateRate>5000.0</updateRate>
-		<cameraName>camera/rgb</cameraName>
-		<frameName>camera_rgb_optical_frame</frameName>
-		<hackBaseline>0.0</hackBaseline>
-		<CxPrime>320.5</CxPrime>
-		<Cx>320.5</Cx>
-		<Cy>240.5</Cy>
-		<baseline>0.09</baseline>
-		<!-- image_width / (2*tan(hfov_radian /2)) -->
-		<!-- 320 for wide and 772.55 for narrow stereo camera -->
-		<focal_length>525</focal_length>
-		<cameraNamespace>camera/rgb</cameraNamespace>
-		<depthData>true</depthData>
-		<interface:camera name="camera_iface" />
-	      </controller:gazebo_ros_wge100>
-	    </sensor:camera>
-	  </gazebo>
-	</xacro:macro>
-	<xacro:macro name="turtlebot_sim_kinect">
-	  <gazebo reference="camera_link">
-	    <sensor:camera name="camera">
-<!-- 	      <always_on>1</always_on> -->
-<!-- 	      <update_rate>30</update_rate> -->
-<!-- 	      <visualize>true</visualize> -->
-<!-- 	      <pose>0 0 0 0 0 0</pose> -->
-<!-- 	      <topic>default</topic> -->
-<!-- 	      <plugin></plugin> -->
-<!--         <camera> -->
-<!-- 	        <horizontal_fov>60</horizontal_fov> -->
-<!-- 					<image> -->
-<!-- 					   <width>640</width> -->
-<!-- 					   <height>480</height> -->
-<!-- 					   <format>R8G8B8</format> -->
-<!-- 					</image> -->
-<!-- 					<clip> -->
-<!-- 					  <near>0.05</near> -->
-<!-- 					  <far>3.0</far> -->
-<!-- 					</clip> -->
-<!-- 				</camera> -->
-<!-- 				<save>false</save> -->
-<!--         <depth_camera> -->
-<!--           <output>default</output> -->
-<!--         </depth_camera> -->
-	      <always_on>true</always_on>
-	      <imageFormat>R8G8B8</imageFormat>
-	      <imageSize>640 480</imageSize>
-	      <hfov>60</hfov>
-	      <nearClip>0.05</nearClip>
-	      <farClip>3</farClip>
-	      <updateRate>20</updateRate>
-	      <baseline>0.1</baseline>
-<!-- 	      <controller:gazebo_ros_openni_kinect name="kinect_camera_controller" plugin="libgazebo_ros_openni_kinect.so"> -->
-<!-- 	        <cameraName>kinect</cameraName> -->
-<!-- 	        <alwaysOn>true</alwaysOn> -->
-<!-- 	        <updateRate>20</updateRate> -->
-<!-- 	        <imageTopicName>/camera/image_raw</imageTopicName> -->
-<!-- 	        <pointCloudTopicName>/camera/depth/points</pointCloudTopicName> -->
-<!-- 	        <cameraInfoTopicName>/camera/camera_info</cameraInfoTopicName> -->
-<!-- 	        <frameName>camera_depth_optical_frame</frameName> -->
-<!-- 	        <CxPrime>0.0</CxPrime> -->
-<!-- 	        <Cx>0.0</Cx> -->
-<!-- 	        <Cy>0.0</Cy> -->
-<!-- 	        <focalLength>0.0</focalLength> -->
-<!-- 	        <hackBaseline>0.0</hackBaseline> -->
-<!-- 	        <distortionK1>0.0</distortionK1> -->
-<!-- 	        <distortionK2>0.0</distortionK2> -->
-<!-- 	        <distortionK3>0.0</distortionK3> -->
-<!-- 	        <distortionT1>0.0</distortionT1> -->
-<!-- 	        <distortionT2>0.0</distortionT2> -->
-<!-- 	      </controller:gazebo_ros_openni_kinect> -->
-	    </sensor:camera>
-	  </gazebo>
-	</xacro:macro>
+<robot name="turtlebot_gazebo" xmlns:xacro="http://ros.org/wiki/xacro">
+  <!-- ASUS Xtion PRO Live for simulation -->
+<!--   <xacro:macro name="turtlebot_sim_xtion"> -->
+<!--     <gazebo reference="camera_link" > -->
+<!--     <sensor type="depth" name="camera"> -->
+<!--       <always_on>true</always_on> -->
+<!--       <update_rate>2.0</update_rate> -->
+<!--       <camera> -->
+<!--         <horizontal_fov>${62.8*M_PI/180.0}</horizontal_fov> -->
+<!--           <image> -->
+<!--             <format>R8G8B8</format> -->
+<!--             <width>640</width> -->
+<!--             <height>480</height> -->
+<!--           </image> -->
+<!--           <clip> -->
+<!--             <near>0.1</near> -->
+<!--             <far>10</far> -->
+<!--           </clip> -->
+<!--         </camera> -->
+<!--         <plugin name="kinect_camera_controller" filename="libgazebo_ros_wge100.so"> -->
+<!--           <alwaysOn>true</alwaysOn> -->
+<!--           <updateRate>5000.0</updateRate> -->
+<!--           <cameraName>camera/rgb</cameraName> -->
+<!--           <frameName>camera_rgb_optical_frame</frameName> -->
+<!--           <hackBaseline>0.0</hackBaseline> -->
+<!--           <CxPrime>320.5</CxPrime> -->
+<!--           <Cx>320.5</Cx> -->
+<!--           <Cy>240.5</Cy> -->
+<!--           <baseline>0.09</baseline> -->
+<!--           image_width / (2*tan(hfov_radian /2)) -->
+<!--           320 for wide and 772.55 for narrow stereo camera -->
+<!--           <focal_length>525</focal_length> -->
+<!--           <cameraNamespace>camera/rgb</cameraNamespace> -->
+<!--           <depthData>true</depthData> -->
+<!--         </plugin> -->
+<!--       </sensor> -->
+<!--     </gazebo> -->
+<!--   </xacro:macro> -->
+  <!-- Microsoft Kinect for simulation -->
+  <xacro:macro name="turtlebot_sim_3dsensor">
+    <gazebo reference="camera_link">
+      <sensor type="depth" name="camera">
+        <always_on>true</always_on>
+        <update_rate>20.0</update_rate>
+        <camera>
+          <horizontal_fov>${60.0*M_PI/180.0}</horizontal_fov>
+          <image>
+            <format>R8G8B8</format>
+            <width>640</width>
+            <height>480</height>
+          </image>
+          <clip>
+            <near>0.05</near>
+            <far>3.0</far>
+          </clip>
+        </camera>
+        <plugin name="kinect_camera_controller" filename="libgazebo_ros_openni_kinect.so">
+          <alwaysOn>true</alwaysOn>
+          <updateRate>20</updateRate>
+          <imageTopicName>/camera/rgb/image_raw</imageTopicName>
+          <depthImageTopicName>/camera/depth/image_raw</depthImageTopicName>
+          <pointCloudTopicName>/camera/depth/points</pointCloudTopicName>
+          <cameraInfoTopicName>/camera/rgb/camera_info</cameraInfoTopicName>
+          <depthImageCameraInfoTopicName>/camera/depth/camera_info</depthImageCameraInfoTopicName>
+          <frameName>camera_depth_optical_frame</frameName>
+          <baseline>0.1</baseline>
+          <distortion_k1>0.0</distortion_k1>
+          <distortion_k2>0.0</distortion_k2>
+          <distortion_k3>0.0</distortion_k3>
+          <distortion_t1>0.0</distortion_t1>
+          <distortion_t2>0.0</distortion_t2>
+          <pointCloudCutoff>0.4</pointCloudCutoff>
+        </plugin>
+      </sensor>
+    </gazebo>
+  </xacro:macro>
 </robot>

File: turtlebot_description/urdf/turtlebot_library.urdf.xacro (robot description, xacro)
@@ -3,18 +3,16 @@
   The complete turtlebot library of xacros for easy reference
  -->
-<robot>
+<robot xmlns:xacro="http://ros.org/wiki/xacro">
   <!-- General -->
-  <include filename="$(find turtlebot_description)/urdf/common_properties.urdf.xacro"/>
-  <include filename="$(find turtlebot_description)/urdf/turtlebot_properties.urdf.xacro"/>
+  <xacro:include filename="$(find turtlebot_description)/urdf/common_properties.urdf.xacro"/>
+  <xacro:include filename="$(find turtlebot_description)/urdf/turtlebot_properties.urdf.xacro"/>
   <!-- Bases -->
-  <include filename="$(find create_description)/urdf/create.urdf.xacro"/>
-  <include filename="$(find kobuki_description)/urdf/kobuki.urdf.xacro" />
+  <xacro:include filename="$(find create_description)/urdf/create.urdf.xacro"/>
+  <xacro:include filename="$(find kobuki_description)/urdf/kobuki.urdf.xacro" />
   <!-- Stacks -->
-  <include filename="$(find turtlebot_description)/urdf/stacks/circles.urdf.xacro"/>
-  <include filename="$(find turtlebot_description)/urdf/stacks/hexagons.urdf.xacro"/>
+  <xacro:include filename="$(find turtlebot_description)/urdf/stacks/circles.urdf.xacro"/>
+  <xacro:include filename="$(find turtlebot_description)/urdf/stacks/hexagons.urdf.xacro"/>
   <!-- 3D Sensors -->
-  <include filename="$(find turtlebot_description)/urdf/sensors/kinect.urdf.xacro"/>
-  <include filename="$(find turtlebot_description)/urdf/sensors/asus_xtion_pro.urdf.xacro"/>
-  <!-- Gazebo -->
-  <include filename="$(find turtlebot_description)/urdf/turtlebot_gazebo.urdf.xacro"/>
+  <xacro:include filename="$(find turtlebot_description)/urdf/sensors/kinect.urdf.xacro"/>
+  <xacro:include filename="$(find turtlebot_description)/urdf/sensors/asus_xtion_pro.urdf.xacro"/>
 </robot>
