Commit message: moving base link back in sync with create convention, closes #44

File: turtlebot_description/robots/kobuki_hexagons_asus_xtion_pro.urdf.xacro (robot description, xacro)
@@ -13,4 +13,4 @@
   <kobuki/>
   <stack_hexagons         parent="base_link"/>
-  <sensor_asus_xtion_pro  parent="base_bottom_link"/>
+  <sensor_asus_xtion_pro  parent="base_link"/>
 </robot>

File: turtlebot_description/robots/kobuki_hexagons_kinect.urdf.xacro (robot description, xacro)
@@ -13,4 +13,4 @@
   <kobuki/>
   <stack_hexagons parent="base_link"/>
-  <sensor_kinect  parent="base_bottom_link"/>
+  <sensor_kinect  parent="base_link"/>
 </robot>

File: turtlebot_description/urdf/stacks/hexagons.urdf.xacro (robot description, xacro)
@@ -125,31 +125,35 @@
     </link>
   </xacro:macro>
-  <!-- Stack macro -->
+  <!--
+    Stack macro - all the components relative transforms are made with respect
+    to the parent link (usually base_link). They could be made relative to each
+    other, but there is no necessary reason to do so.
+  -->
   <xacro:macro name="stack_hexagons" params="parent">
-	  <stack_bottom_pole    parent="${parent}" number="0" x_loc= "0.120" y_loc= "0.082" z_loc="0.073"/>
-	  <stack_bottom_pole    parent="${parent}" number="1" x_loc= "0.055" y_loc= "0.120" z_loc="0.073"/>
-	  <stack_bottom_pole    parent="${parent}" number="2" x_loc="-0.055" y_loc= "0.120" z_loc="0.073"/>
-    <stack_bottom_pole    parent="${parent}" number="3" x_loc= "0.120" y_loc="-0.082" z_loc="0.073"/>
-    <stack_bottom_pole    parent="${parent}" number="4" x_loc= "0.055" y_loc="-0.120" z_loc="0.073"/>
-    <stack_bottom_pole    parent="${parent}" number="5" x_loc="-0.055" y_loc="-0.120" z_loc="0.073"/>
-		<joint name="plate_bottom_joint" type="fixed">
-		  <origin xyz="0.02364 0.0 0.1006" rpy="0 0 0"/>
-		  <parent link="${parent}"/>
-		  <child link="plate_bottom_link"/>
-		</joint>
-		<link name="plate_bottom_link">
-		  <visual>
-		    <origin xyz="0 0 0" rpy="${M_PI/2} 0 ${M_PI/2}"/>
-		    <geometry>
-		      <mesh filename="package://turtlebot_description/meshes/stacks/hexagons/plate_bottom.dae" scale="${M_SCALE} ${M_SCALE} ${M_SCALE}"/>
-		    </geometry>
+    <stack_bottom_pole parent="${parent}" number="0" x_loc= "0.120" y_loc= "0.082" z_loc="0.0980"/>
+    <stack_bottom_pole parent="${parent}" number="1" x_loc= "0.055" y_loc= "0.120" z_loc="0.0980"/>
+    <stack_bottom_pole parent="${parent}" number="2" x_loc="-0.055" y_loc= "0.120" z_loc="0.0980"/>
+    <stack_bottom_pole parent="${parent}" number="3" x_loc= "0.120" y_loc="-0.082" z_loc="0.0980"/>
+    <stack_bottom_pole parent="${parent}" number="4" x_loc= "0.055" y_loc="-0.120" z_loc="0.0980"/>
+    <stack_bottom_pole parent="${parent}" number="5" x_loc="-0.055" y_loc="-0.120" z_loc="0.0980"/>
+    <joint name="plate_bottom_joint" type="fixed">
+      <origin xyz="0.02364 0.0 0.1256" rpy="0 0 0"/>
+      <parent link="${parent}"/>
+      <child link="plate_bottom_link"/>
+    </joint>
+    <link name="plate_bottom_link">
+      <visual>
+        <origin xyz="0 0 0" rpy="${M_PI/2} 0 ${M_PI/2}"/>
+        <geometry>
+          <mesh filename="package://turtlebot_description/meshes/stacks/hexagons/plate_bottom.dae" scale="${M_SCALE} ${M_SCALE} ${M_SCALE}"/>
+        </geometry>
         <xacro:insert_block name="material_black"/>
-		  </visual>
-		  <collision>
-		    <origin xyz="0 0 0" rpy="0 0 0"/>
-		    <geometry>
-		      <box size="0.26727 0.345 0.006"/>
-		    </geometry>
-		  </collision>
+      </visual>
+      <collision>
+        <origin xyz="0 0 0" rpy="0 0 0"/>
+        <geometry>
+          <box size="0.26727 0.345 0.006"/>
+        </geometry>
+      </collision>
       <inertial>
         <mass value="0.01" />
@@ -159,28 +163,28 @@
                  izz="0.01" />
       </inertial>
-		</link>
-		<stack_middle_pole parent="${parent}" number="0" x_loc= "0.0381" y_loc= "0.1505" z_loc="0.134"/>
-		<stack_middle_pole parent="${parent}" number="1" x_loc= "0.0381" y_loc="-0.1505" z_loc="0.134"/>
-		<stack_middle_pole parent="${parent}" number="2" x_loc="-0.0381" y_loc= "0.1505" z_loc="0.134"/>
-		<stack_middle_pole parent="${parent}" number="3" x_loc="-0.0381" y_loc="-0.1505" z_loc="0.134"/>
-		<joint name="plate_middle_joint" type="fixed">
-		  <origin xyz="-0.01364 0.0 0.1574" rpy="0 0 0"/>
-		  <parent link="${parent}"/>
-		  <child link="plate_middle_link"/>
-		</joint>
-		<link name="plate_middle_link">
-		  <visual>
-		    <origin xyz="0 0 0" rpy="${M_PI/2} 0 -${M_PI/2}"/>
-		    <geometry>
+    </link>
+    <stack_middle_pole parent="${parent}" number="0" x_loc= "0.0381" y_loc= "0.1505" z_loc="0.1590"/>
+    <stack_middle_pole parent="${parent}" number="1" x_loc= "0.0381" y_loc="-0.1505" z_loc="0.1590"/>
+    <stack_middle_pole parent="${parent}" number="2" x_loc="-0.0381" y_loc= "0.1505" z_loc="0.1590"/>
+    <stack_middle_pole parent="${parent}" number="3" x_loc="-0.0381" y_loc="-0.1505" z_loc="0.1590"/>
+    <joint name="plate_middle_joint" type="fixed">
+      <origin xyz="-0.01364 0.0 0.1824" rpy="0 0 0"/>
+      <parent link="${parent}"/>
+      <child link="plate_middle_link"/>
+    </joint>
+    <link name="plate_middle_link">
+      <visual>
+        <origin xyz="0 0 0" rpy="${M_PI/2} 0 -${M_PI/2}"/>
+        <geometry>
           <mesh filename="package://turtlebot_description/meshes/stacks/hexagons/plate_middle.dae" scale="${M_SCALE} ${M_SCALE} ${M_SCALE}"/>
-		    </geometry>
+        </geometry>
         <xacro:insert_block name="material_black"/>
-		  </visual>
-		  <collision>
-		    <origin xyz="0.0 0.0 0.0" rpy="0 0 0"/>
-		    <geometry>
-		      <box size="0.28727 0.340 0.006"/>
-		    </geometry>
-		  </collision>
+      </visual>
+      <collision>
+        <origin xyz="0.0 0.0 0.0" rpy="0 0 0"/>
+        <geometry>
+          <box size="0.28727 0.340 0.006"/>
+        </geometry>
+      </collision>
       <inertial>
         <mass value="0.01" />
@@ -190,30 +194,30 @@
                  izz="0.01" />
       </inertial>
-		</link>
-		<stack_top_pole parent="${parent}" number="0" x_loc= "0.0381" y_loc= "0.1505" z_loc="0.262"/>
-		<stack_top_pole parent="${parent}" number="1" x_loc= "0.0381" y_loc="-0.1505" z_loc="0.262"/>
-		<stack_top_pole parent="${parent}" number="2" x_loc="-0.0381" y_loc= "0.1505" z_loc="0.262"/>
-		<stack_top_pole parent="${parent}" number="3" x_loc="-0.0381" y_loc="-0.1505" z_loc="0.262"/>
-    <stack_3d_sensor_pole parent="${parent}" number="0" x_loc="-0.1024" y_loc= "0.098" z_loc="0.2072"/>
-    <stack_3d_sensor_pole parent="${parent}" number="1" x_loc="-0.1024" y_loc="-0.098" z_loc="0.2072"/>
-		<joint name="plate_top_joint" type="fixed">
-		  <origin xyz="-0.01364 0.0  0.3666" rpy="0 0 0"/>
-		  <parent link="${parent}"/>
-		  <child link="plate_top_link"/>
-		</joint>
-		<link name="plate_top_link">
-		  <visual>
+	</link>
+    <stack_top_pole parent="${parent}" number="0" x_loc= "0.0381" y_loc= "0.1505" z_loc="0.2870"/>
+    <stack_top_pole parent="${parent}" number="1" x_loc= "0.0381" y_loc="-0.1505" z_loc="0.2870"/>
+    <stack_top_pole parent="${parent}" number="2" x_loc="-0.0381" y_loc= "0.1505" z_loc="0.2870"/>
+    <stack_top_pole parent="${parent}" number="3" x_loc="-0.0381" y_loc="-0.1505" z_loc="0.2870"/>
+    <stack_3d_sensor_pole parent="${parent}" number="0" x_loc="-0.1024" y_loc= "0.098" z_loc="0.2322"/>
+    <stack_3d_sensor_pole parent="${parent}" number="1" x_loc="-0.1024" y_loc="-0.098" z_loc="0.2322"/>
+    <joint name="plate_top_joint" type="fixed">
+      <origin xyz="-0.01364 0.0  0.3916" rpy="0 0 0"/>
+      <parent link="${parent}"/>
+      <child link="plate_top_link"/>
+    </joint>
+    <link name="plate_top_link">
+      <visual>
         <origin xyz="0 0 0" rpy="${M_PI/2} 0 -${M_PI/2}"/>
-		    <geometry>
+        <geometry>
           <mesh filename="package://turtlebot_description/meshes/stacks/hexagons/plate_top.dae" scale="${M_SCALE} ${M_SCALE} ${M_SCALE}"/>
-		    </geometry>
+        </geometry>
         <xacro:insert_block name="material_black"/>
-		  </visual>
-		  <collision>
-        <origin xyz="0 0 0" rpy="0 0 0"/>
-		    <geometry>
+      </visual>
+      <collision>
+        <origin xyz="0 0 0" rpy="0 0 0"/>
+        <geometry>
           <box size="0.28727 0.340 0.006"/>
-		    </geometry>
-		  </collision>
+        </geometry>
+      </collision>
       <inertial>
         <mass value="0.01"/>

Commit message: update urdf. now new position uses asus_xtion_pro. Old position is asus_xtion_pro_offset

File: turtlebot_description/robots/kobuki_hexagons_asus_xtion_pro.urdf.xacro (robot description, xacro)
@@ -8,5 +8,5 @@
   <xacro:include filename="$(find turtlebot_description)/urdf/turtlebot_library.urdf.xacro" />
   <kobuki/>
-  <stack_hexagons         parent="base_link"/>
-  <sensor_asus_xtion_pro  parent="base_link"/>
+  <stack_hexagons                 parent="base_link"/>
+  <sensor_asus_xtion_pro          parent="base_link"/>
 </robot>

File: turtlebot_description/robots/kobuki_hexagons_asus_xtion_pro_offset.urdf.xacro (robot description, xacro)
@@ -9,4 +9,4 @@
   <kobuki/>
   <stack_hexagons                 parent="base_link"/>
-  <sensor_asus_xtion_pro_center   parent="base_link"/>
+  <sensor_asus_xtion_pro_offset   parent="base_link"/>
 </robot>

File: turtlebot_description/urdf/sensors/asus_xtion_pro.urdf.xacro (robot description, xacro)
@@ -2,8 +2,8 @@
 <robot name="sensor_asus_xtion_pro" xmlns:xacro="http://ros.org/wiki/xacro">
   <xacro:include filename="$(find turtlebot_description)/urdf/turtlebot_gazebo.urdf.xacro"/>
-  <xacro:include filename="$(find turtlebot_description)/urdf/turtlebot_properties.urdf.xacro"/>f.xacro"/>
+  <xacro:include filename="$(find turtlebot_description)/urdf/turtlebot_properties.urdf.xacro"/>
   <!-- Xacro properties -->
   <xacro:property name="M_SCALE" value="0.001"/>
-  <xacro:property name="asus_xtion_pro_cam_py" value="-0.0125"/>
+  <xacro:property name="asus_xtion_pro_cam_py" value="0.0205"/>
   <xacro:property name="asus_xtion_pro_depth_rel_rgb_py" value="0.0270" />
   <xacro:property name="asus_xtion_pro_cam_rel_rgb_py"   value="-0.0220" />
@@ -31,7 +31,7 @@
     <link name="camera_link">
       <visual>
-        <origin xyz="-0.01 0 0" rpy="${-M_PI/2} -${M_PI} ${-M_PI/2}"/>
+        <origin xyz="-0.015 0.0035 0.004" rpy="0 0 0"/>
         <geometry>
-          <mesh filename="package://turtlebot_description/meshes/sensors/asus_xtion_pro_live.dae" scale="${M_SCALE} ${M_SCALE} ${M_SCALE}"/>
+          <mesh filename="package://turtlebot_description/meshes/sensors/xtion_pro_camera.dae"/>
         </geometry>
       </visual>
@@ -64,4 +64,31 @@
     <!-- RGBD sensor for simulation, same as Kinect -->
     <turtlebot_sim_3dsensor/>
+    <!-- Asus mount -->
+    <joint name="mount_asus_xtion_pro_joint" type="fixed">
+      <origin xyz="-0.1024 0.0 0.272" rpy="0 0 0"/>
+      <parent link="${parent}"/>
+      <child link="mount_asus_xtion_pro_link"/>
+    </joint>
+    <link name="mount_asus_xtion_pro_link">
+      <visual>
+        <origin xyz="0 0 0" rpy="0 0 ${-M_PI/2}"/>
+        <geometry>
+          <mesh filename="package://turtlebot_description/meshes/sensors/xtion_pro_stack.dae"/>
+        </geometry>
+      </visual>
+      <collision>
+        <origin xyz="0.0 0.0 0.0" rpy="0 0 0" />
+        <geometry>
+        <box size="0.0330 0.2760 0.0120"/>
+      </geometry>
+      </collision>
+      <inertial>
+        <mass value="0.170" />
+        <origin xyz="0 0 0" />
+        <inertia ixx="0.001152600" ixy="0.0" ixz="0.0"
+                 iyy="0.000148934" iyz="0.0"
+                 izz="0.001154654" />
+      </inertial>
+    </link>
   </xacro:macro>
 </robot>

File: turtlebot_description/urdf/sensors/asus_xtion_pro_offset.urdf.xacro (robot description, xacro)
@@ -1,15 +1,15 @@
 <?xml version="1.0"?>
-<robot name="sensor_asus_xtion_pro_center" xmlns:xacro="http://ros.org/wiki/xacro">
+<robot name="sensor_asus_xtion_pro_offset" xmlns:xacro="http://ros.org/wiki/xacro">
   <xacro:include filename="$(find turtlebot_description)/urdf/turtlebot_gazebo.urdf.xacro"/>
   <xacro:include filename="$(find turtlebot_description)/urdf/turtlebot_properties.urdf.xacro"/>
   <!-- Xacro properties -->
   <xacro:property name="M_SCALE" value="0.001"/>
-  <xacro:property name="asus_xtion_pro_center_cam_py" value="0.0205"/>
-  <xacro:property name="asus_xtion_pro_center_depth_rel_rgb_py" value="0.0270" />
-  <xacro:property name="asus_xtion_pro_center_cam_rel_rgb_py"   value="-0.0220" />
+  <xacro:property name="asus_xtion_pro_offset_cam_py" value="-0.0125"/>
+  <xacro:property name="asus_xtion_pro_offset_depth_rel_rgb_py" value="0.0270" />
+  <xacro:property name="asus_xtion_pro_offset_cam_rel_rgb_py"   value="-0.0220" />
   <!-- Parameterised in part by the values in turtlebot_properties.urdf.xacro -->
-  <xacro:macro name="sensor_asus_xtion_pro_center" params="parent">
+  <xacro:macro name="sensor_asus_xtion_pro_offset" params="parent">
     <joint name="camera_rgb_joint" type="fixed">
-      <origin xyz="${cam_px} ${asus_xtion_pro_center_cam_py} ${cam_pz}"
+      <origin xyz="${cam_px} ${asus_xtion_pro_offset_cam_py} ${cam_pz}"
               rpy="${cam_or} ${cam_op} ${cam_oy}"/>
       <parent link="${parent}"/>
@@ -24,5 +24,5 @@
     <link name="camera_rgb_optical_frame"/>
     <joint name="camera_joint" type="fixed">
-      <origin xyz="0 ${asus_xtion_pro_center_cam_rel_rgb_py} 0"
+      <origin xyz="0 ${asus_xtion_pro_offset_cam_rel_rgb_py} 0"
               rpy="0 0 0"/>
       <parent link="camera_rgb_frame"/>
@@ -31,7 +31,7 @@
     <link name="camera_link">
       <visual>
-        <origin xyz="-0.015 0 -0.006" rpy="${-M_PI/2} -${M_PI} ${-M_PI/2}"/>
+        <origin xyz="-0.01 0 0" rpy="${-M_PI/2} -${M_PI} ${-M_PI/2}"/>
         <geometry>
-          <mesh filename="package://turtlebot_description/meshes/sensors/xtion_pro_camera.dae"/>
+          <mesh filename="package://turtlebot_description/meshes/sensors/asus_xtion_pro_live.dae" scale="${M_SCALE} ${M_SCALE} ${M_SCALE}"/>
         </geometry>
       </visual>
@@ -51,5 +51,5 @@
     </link>
     <joint name="camera_depth_joint" type="fixed">
-      <origin xyz="0 ${asus_xtion_pro_center_depth_rel_rgb_py} 0" rpy="0 0 0" />
+      <origin xyz="0 ${asus_xtion_pro_offset_depth_rel_rgb_py} 0" rpy="0 0 0" />
       <parent link="camera_rgb_frame" />
       <child link="camera_depth_frame" />
@@ -64,31 +64,4 @@
     <!-- RGBD sensor for simulation, same as Kinect -->
     <turtlebot_sim_3dsensor/>
-    <!-- Asus mount -->
-    <joint name="mount_asus_xtion_pro_center_joint" type="fixed">
-      <origin xyz="-0.1024 0.0 0.272" rpy="0 0 0"/>
-      <parent link="${parent}"/>
-      <child link="mount_asus_xtion_pro_center_link"/>
-    </joint>
-    <link name="mount_asus_xtion_pro_center_link">
-      <visual>
-        <origin xyz="0 0 0" rpy="0 0 ${-M_PI/2}"/>
-        <geometry>
-          <mesh filename="package://turtlebot_description/meshes/sensors/xtion_pro_stack.dae"/>
-        </geometry>
-      </visual>
-      <collision>
-        <origin xyz="0.0 0.0 0.0" rpy="0 0 0" />
-        <geometry>
-        <box size="0.0330 0.2760 0.0120"/>
-      </geometry>
-      </collision>
-      <inertial>
-        <mass value="0.170" />
-        <origin xyz="0 0 0" />
-        <inertia ixx="0.001152600" ixy="0.0" ixz="0.0"
-                 iyy="0.000148934" iyz="0.0"
-                 izz="0.001154654" />
-      </inertial>
-    </link>
   </xacro:macro>
 </robot>

File: turtlebot_description/urdf/turtlebot_library.urdf.xacro (robot description, xacro)
@@ -16,4 +16,4 @@
   <xacro:include filename="$(find turtlebot_description)/urdf/sensors/kinect.urdf.xacro"/>
   <xacro:include filename="$(find turtlebot_description)/urdf/sensors/asus_xtion_pro.urdf.xacro"/>
-  <xacro:include filename="$(find turtlebot_description)/urdf/sensors/asus_xtion_pro_center.urdf.xacro"/>
+  <xacro:include filename="$(find turtlebot_description)/urdf/sensors/asus_xtion_pro_offset.urdf.xacro"/>
 </robot>
