Commit message: add turtlebot_description

File: turtlebot_description/robots/create_circles_kinect.urdf.xacro (robot description, xacro)
@@ -1,8 +1,3 @@
 <?xml version="1.0"?>
-<!--
-    - Base      : create
-    - Stacks    : circles
-    - 3d Sensor : kinect
--->
 <robot name="turtlebot" xmlns:xacro="http://ros.org/wiki/xacro">
   <xacro:include filename="$(find turtlebot_description)/urdf/turtlebot_common_library.urdf.xacro" />

File: turtlebot_description/robots/kobuki_hexagons_kinect.urdf.xacro (robot description, xacro)
@@ -1,8 +1,3 @@
 <?xml version="1.0"?>
-<!--
-    - Base      : kobuki
-    - Stacks    : hexagons
-    - 3d Sensor : kinect
--->
 <robot name="turtlebot" xmlns:xacro="http://ros.org/wiki/xacro">
   <xacro:include filename="$(find turtlebot_description)/urdf/turtlebot_common_library.urdf.xacro" />

File: turtlebot_description/urdf/stacks/hexagons.urdf.xacro (robot description, xacro)
@@ -178,5 +178,5 @@
         <origin xyz="0.01364 0.0 0.0" rpy="0 0 0"/>
         <geometry>
-          <mesh filename="package://turtlebot_description/meshes/stacks/hexagons/plate_simple.stl"
+          <mesh filename="package://turtlebot_description/meshes/stacks/hexagons/plate_simple-binary.stl"
                 scale="${M_SCALE} ${M_SCALE} ${M_SCALE}"/>
         </geometry>
@@ -211,5 +211,5 @@
         <origin xyz="0.01364 0 0" rpy="0 0 0"/>
         <geometry>
-          <mesh filename="package://turtlebot_description/meshes/stacks/hexagons/plate_simple.stl"
+          <mesh filename="package://turtlebot_description/meshes/stacks/hexagons/plate_simple-binary.stl"
                 scale="${M_SCALE} ${M_SCALE} ${M_SCALE}"/>
         </geometry>
