Commit message: turtlebot2 descriptions rejiggled.

File: turtlebot_description/robots/graveyard/turtlebot.urdf.xacro (robot description, xacro)
@@ -5,8 +5,8 @@
        xmlns:interface="http://playerstage.sourceforge.net/gazebo/xmlschema/#interface"
        xmlns:xacro="http://ros.org/wiki/xacro">
-  <include filename="$(find turtlebot_description)/urdf/turtlebot_hardware.urdf.xacro" />
-  <include filename="$(find turtlebot_description)/urdf/turtlebot_body.urdf.xacro" />
-  <include filename="$(find turtlebot_description)/urdf/turtlebot_calibration.xacro" />
-  <include filename="$(find turtlebot_description)/urdf/turtlebot_kinect.urdf.xacro" />
+  <include filename="$(find turtlebot_description)/urdf/graveyard/turtlebot_hardware.urdf.xacro" />
+  <include filename="$(find turtlebot_description)/urdf/graveyard/turtlebot_body.urdf.xacro" />
+  <include filename="$(find turtlebot_description)/urdf/graveyard/turtlebot_calibration.xacro" />
+  <include filename="$(find turtlebot_description)/urdf/graveyard/turtlebot_kinect.urdf.xacro" />
   <property name="M_PI" value="3.14159"/>
   <property name="SCALE" value="0.0254"/>

File: turtlebot_description/urdf/graveyard/turtlebot_kinect.urdf.xacro (robot description, xacro)
@@ -3,5 +3,5 @@
   <property name="M_PI" value="3.14159"/>
   <include filename="$(find turtlebot_description)/urdf/gazebo.urdf.xacro"/>
-  <include filename="$(find turtlebot_description)/urdf/turtlebot_calibration.xacro" />
+  <include filename="$(find turtlebot_description)/urdf/graveyard/turtlebot_calibration.xacro" />
 <xacro:macro name="turtlebot_kinect">
   <joint name="base_camera_joint" type="fixed">
@@ -22,5 +22,5 @@
       <origin xyz=" 0 0 0 " rpy="0 0 0" />
       <geometry>
-        <mesh filename="package://turtlebot_description/meshes/kinect.dae"/>
+        <mesh filename="package://turtlebot_description/meshes/sensors/kinect.dae"/>
       </geometry>
     </visual>

File: turtlebot_description/urdf/stack_hexagons.urdf.xacro (robot description, xacro)
@@ -1,7 +1,7 @@
 <?xml version="1.0"?>
 <!--
-  Turtlebot 2 stack (plates + poles)
+  Hexagon stacks
  -->
-<robot name="turtlebot2_stack" xmlns:xacro="http://ros.org/wiki/xacro">
+<robot name="stack_hexagons" xmlns:xacro="http://ros.org/wiki/xacro">
   <include filename="$(find turtlebot_description)/urdf/common_properties.urdf.xacro"/>
   <!-- Xacro properties -->
@@ -18,5 +18,5 @@
         <origin xyz="0 0 0" rpy="${M_PI/2} 0 ${M_PI/2}"/>
         <geometry>
-          <mesh filename="package://turtlebot_description/meshes/turtlebot2_stack/pole_bottom.stl" scale="${M_SCALE} ${M_SCALE} ${M_SCALE}"/>
+          <mesh filename="package://turtlebot_description/meshes/stacks/hexagons/pole_bottom.stl" scale="${M_SCALE} ${M_SCALE} ${M_SCALE}"/>
         </geometry>
         <xacro:insert_block name="material_light_grey"/>
@@ -47,5 +47,5 @@
         <origin xyz="0 0 0" rpy="${-M_PI/2} 0 0"/>
         <geometry>
-          <mesh filename="package://turtlebot_description/meshes/turtlebot2_stack/pole_middle.stl" scale="${M_SCALE} ${M_SCALE} ${M_SCALE}"/>
+          <mesh filename="package://turtlebot_description/meshes/stacks/hexagons/pole_middle.stl" scale="${M_SCALE} ${M_SCALE} ${M_SCALE}"/>
         </geometry>
         <xacro:insert_block name="material_light_grey"/>
@@ -76,5 +76,5 @@
         <origin xyz=" 0 0 0" rpy="${M_PI/2} 0 ${M_PI/2}"/>
         <geometry>
-          <mesh filename="package://turtlebot_description/meshes/turtlebot2_stack/pole_top.stl" scale="${M_SCALE} ${M_SCALE} ${M_SCALE}"/>
+          <mesh filename="package://turtlebot_description/meshes/stacks/hexagons/pole_top.stl" scale="${M_SCALE} ${M_SCALE} ${M_SCALE}"/>
         </geometry>
         <xacro:insert_block name="material_light_grey"/>
@@ -95,12 +95,42 @@
     </link>
   </xacro:macro>
-  <!-- Turtlebot 2 stack -->
-  <xacro:macro name="turtlebot2_stack" params="parent">
-		<stack_bottom_pole parent="${parent}" number="0" x_loc= "0.120" y_loc= "0.082" z_loc="0.0534"/>
-		<stack_bottom_pole parent="${parent}" number="1" x_loc= "0.055" y_loc= "0.120" z_loc="0.0534"/>
-		<stack_bottom_pole parent="${parent}" number="2" x_loc="-0.055" y_loc= "0.120" z_loc="0.0534"/>
-    <stack_bottom_pole parent="${parent}" number="3" x_loc= "0.120" y_loc="-0.082" z_loc="0.0534"/>
-    <stack_bottom_pole parent="${parent}" number="4" x_loc= "0.055" y_loc="-0.120" z_loc="0.0534"/>
-    <stack_bottom_pole parent="${parent}" number="5" x_loc="-0.055" y_loc="-0.120" z_loc="0.0534"/>
+  <xacro:macro name="stack_3d_sensor_pole" params="parent number x_loc y_loc z_loc">
+    <joint name="pole_kinect_${number}_joint" type="fixed">
+      <origin xyz="${x_loc} ${y_loc} ${z_loc}" rpy="0 0 0"/>
+      <parent link="${parent}"/>
+      <child link="pole_kinect_${number}_link"/>
+    </joint>
+    <link name="pole_kinect_${number}_link">
+      <visual>
+        <origin xyz="0 0 0" rpy="${-M_PI/2} 0 0"/>
+        <geometry>
+          <mesh filename="package://turtlebot_description/meshes/stacks/hexagons/pole_kinect.stl" scale="${M_SCALE} ${M_SCALE} ${M_SCALE}"/>
+        </geometry>
+        <xacro:insert_block name="material_light_grey"/>
+      </visual>
+      <collision>
+        <origin xyz="0 0 0" rpy="0 0 0"/>
+        <geometry>
+          <cylinder length="0.0936" radius="0.006"/>
+        </geometry>
+      </collision>
+      <inertial>
+        <mass value="0.001"/>
+        <origin xyz="0 0 0"/>
+        <inertia ixx="0.0001" ixy="0.0" ixz="0.0"
+                 iyy="0.0001" iyz="0.0"
+                 izz="0.0001"/>
+      </inertial>
+    </link>
+  </xacro:macro>
+  <xacro:macro name="stack_hexagons" params="parent">
+	<stack_bottom_pole    parent="${parent}" number="0" x_loc= "0.120" y_loc= "0.082" z_loc="0.0534"/>
+	<stack_bottom_pole    parent="${parent}" number="1" x_loc= "0.055" y_loc= "0.120" z_loc="0.0534"/>
+	<stack_bottom_pole    parent="${parent}" number="2" x_loc="-0.055" y_loc= "0.120" z_loc="0.0534"/>
+    <stack_bottom_pole    parent="${parent}" number="3" x_loc= "0.120" y_loc="-0.082" z_loc="0.0534"/>
+    <stack_bottom_pole    parent="${parent}" number="4" x_loc= "0.055" y_loc="-0.120" z_loc="0.0534"/>
+    <stack_bottom_pole    parent="${parent}" number="5" x_loc="-0.055" y_loc="-0.120" z_loc="0.0534"/>
+    <stack_3d_sensor_pole parent="${parent}" number="0" x_loc="-0.1024" y_loc= "0.098" z_loc="0.259"/>
+    <stack_3d_sensor_pole parent="${parent}" number="1" x_loc="-0.1024" y_loc="-0.098" z_loc="0.259"/>
 		<joint name="plate_bottom_joint" type="fixed">
 		  <origin xyz="0.0 0.0  0.1026" rpy="0 0 0"/>
@@ -112,5 +142,5 @@
 		    <origin xyz="0 0 0" rpy="${M_PI/2} 0 ${M_PI/2}"/>
 		    <geometry>
-		      <mesh filename="package://turtlebot_description/meshes/turtlebot2_stack/plate_bottom.stl" scale="${M_SCALE} ${M_SCALE} ${M_SCALE}"/>
+		      <mesh filename="package://turtlebot_description/meshes/stacks/hexagons/plate_bottom.stl" scale="${M_SCALE} ${M_SCALE} ${M_SCALE}"/>
 		    </geometry>
         <xacro:insert_block name="material_light_grey"/>
@@ -144,5 +174,5 @@
 		    <origin xyz="0 0 0" rpy="${M_PI/2} 0 ${M_PI/2}"/>
 		    <geometry>
-		      <mesh filename="package://turtlebot_description/meshes/turtlebot2_stack/plate_middle.stl" scale="${M_SCALE} ${M_SCALE} ${M_SCALE}"/>
+		      <mesh filename="package://turtlebot_description/meshes/stacks/hexagons/plate_middle.stl" scale="${M_SCALE} ${M_SCALE} ${M_SCALE}"/>
 		    </geometry>
         <xacro:insert_block name="material_light_grey"/>
@@ -175,5 +205,5 @@
         <origin xyz="0 0 0" rpy="${M_PI/2} 0 ${M_PI/2}"/>
 		    <geometry>
-		      <mesh filename="package://turtlebot_description/meshes/turtlebot2_stack/plate_top.stl" scale="${M_SCALE} ${M_SCALE} ${M_SCALE}"/>
+		      <mesh filename="package://turtlebot_description/meshes/stacks/hexagons/plate_top.stl" scale="${M_SCALE} ${M_SCALE} ${M_SCALE}"/>
 		    </geometry>
         <xacro:insert_block name="material_light_grey"/>
