Commit message: turtlebot_description: fixes kinect's collision model misplacement

File: turtlebot_description/urdf/sensors/kinect.urdf.xacro (robot description, xacro)
@@ -46,5 +46,5 @@
     </visual>
 	  <collision>
-	    <origin xyz="-0.0315 0.0 -0.017" rpy="0 0 0"/>
+      <origin xyz="0.0 0.0 0.0" rpy="0 0 0"/>
 	    <geometry>
 	      <box size="0.07271 0.27794 0.073"/>
