Commit message: add urdf for asus center located version

File: turtlebot_description/urdf/sensors/asus_xtion_pro_center.urdf.xacro (robot description, xacro)
@@ -1,15 +1,15 @@
 <?xml version="1.0"?>
-<robot name="sensor_asus_xtion_pro" xmlns:xacro="http://ros.org/wiki/xacro">
+<robot name="sensor_asus_xtion_pro_center" xmlns:xacro="http://ros.org/wiki/xacro">
   <xacro:include filename="$(find turtlebot_description)/urdf/turtlebot_gazebo.urdf.xacro"/>
-  <xacro:include filename="$(find turtlebot_description)/urdf/turtlebot_properties.urdf.xacro"/>f.xacro"/>
+  <xacro:include filename="$(find turtlebot_description)/urdf/turtlebot_properties.urdf.xacro"/>
   <!-- Xacro properties -->
   <xacro:property name="M_SCALE" value="0.001"/>
-  <xacro:property name="asus_xtion_pro_cam_py" value="-0.0125"/>
-  <xacro:property name="asus_xtion_pro_depth_rel_rgb_py" value="0.0270" />
-  <xacro:property name="asus_xtion_pro_cam_rel_rgb_py"   value="-0.0220" />
+  <xacro:property name="asus_xtion_pro_center_cam_py" value="0.0205"/>
+  <xacro:property name="asus_xtion_pro_center_depth_rel_rgb_py" value="0.0270" />
+  <xacro:property name="asus_xtion_pro_center_cam_rel_rgb_py"   value="-0.0220" />
   <!-- Parameterised in part by the values in turtlebot_properties.urdf.xacro -->
-  <xacro:macro name="sensor_asus_xtion_pro" params="parent">
+  <xacro:macro name="sensor_asus_xtion_pro_center" params="parent">
     <joint name="camera_rgb_joint" type="fixed">
-      <origin xyz="${cam_px} ${asus_xtion_pro_cam_py} ${cam_pz}"
+      <origin xyz="${cam_px} ${asus_xtion_pro_center_cam_py} ${cam_pz}"
               rpy="${cam_or} ${cam_op} ${cam_oy}"/>
       <parent link="${parent}"/>
@@ -24,5 +24,5 @@
     <link name="camera_rgb_optical_frame"/>
     <joint name="camera_joint" type="fixed">
-      <origin xyz="0 ${asus_xtion_pro_cam_rel_rgb_py} 0"
+      <origin xyz="0 ${asus_xtion_pro_center_cam_rel_rgb_py} 0"
               rpy="0 0 0"/>
       <parent link="camera_rgb_frame"/>
@@ -51,5 +51,5 @@
     </link>
     <joint name="camera_depth_joint" type="fixed">
-      <origin xyz="0 ${asus_xtion_pro_depth_rel_rgb_py} 0" rpy="0 0 0" />
+      <origin xyz="0 ${asus_xtion_pro_center_depth_rel_rgb_py} 0" rpy="0 0 0" />
       <parent link="camera_rgb_frame" />
       <child link="camera_depth_frame" />

File: turtlebot_description/urdf/turtlebot_library.urdf.xacro (robot description, xacro)
@@ -16,3 +16,4 @@
   <xacro:include filename="$(find turtlebot_description)/urdf/sensors/kinect.urdf.xacro"/>
   <xacro:include filename="$(find turtlebot_description)/urdf/sensors/asus_xtion_pro.urdf.xacro"/>
+  <xacro:include filename="$(find turtlebot_description)/urdf/sensors/asus_xtion_pro_center.urdf.xacro"/>
 </robot>

File: turtlebot_description/urdf/turtlebot_properties.urdf.xacro (robot description, xacro)
@@ -20,5 +20,5 @@
    -->
 	<property name="cam_px" value="-0.087" />
-	<property name="cam_py" value="-0.0125" />
+<!--	<property name="cam_py" value="-0.0125" />-->
 	<property name="cam_pz" value="0.2870" />
 	<property name="cam_or" value="0" />

Commit message: add asus, mount, and new pole

File: turtlebot_description/urdf/sensors/asus_xtion_pro_center.urdf.xacro (robot description, xacro)
@@ -31,7 +31,7 @@
     <link name="camera_link">
       <visual>
-        <origin xyz="-0.01 0 0" rpy="${-M_PI/2} -${M_PI} ${-M_PI/2}"/>
+        <origin xyz="-0.015 0 -0.006" rpy="${-M_PI/2} -${M_PI} ${-M_PI/2}"/>
         <geometry>
-          <mesh filename="package://turtlebot_description/meshes/sensors/asus_xtion_pro_live.dae" scale="${M_SCALE} ${M_SCALE} ${M_SCALE}"/>
+          <mesh filename="package://turtlebot_description/meshes/sensors/xtion_pro_camera.dae"/>
         </geometry>
       </visual>
@@ -64,4 +64,31 @@
     <!-- RGBD sensor for simulation, same as Kinect -->
     <turtlebot_sim_3dsensor/>
+    <!-- Asus mount -->
+    <joint name="mount_asus_xtion_pro_center_joint" type="fixed">
+      <origin xyz="-0.1024 0.0 0.272" rpy="0 0 0"/>
+      <parent link="${parent}"/>
+      <child link="mount_asus_xtion_pro_center_link"/>
+    </joint>
+    <link name="mount_asus_xtion_pro_center_link">
+      <visual>
+        <origin xyz="0 0 0" rpy="0 0 ${-M_PI/2}"/>
+        <geometry>
+          <mesh filename="package://turtlebot_description/meshes/sensors/xtion_pro_stack.dae"/>
+        </geometry>
+      </visual>
+      <collision>
+        <origin xyz="0.0 0.0 0.0" rpy="0 0 0" />
+        <geometry>
+        <box size="0.0330 0.2760 0.0120"/>
+      </geometry>
+      </collision>
+      <inertial>
+        <mass value="0.170" />
+        <origin xyz="0 0 0" />
+        <inertia ixx="0.001152600" ixy="0.0" ixz="0.0"
+                 iyy="0.000148934" iyz="0.0"
+                 izz="0.001154654" />
+      </inertial>
+    </link>
   </xacro:macro>
 </robot>
