Commit message: Update R200 URDF
The name of the camera link has been changed to
conform to the common standard.

File: turtlebot_description/urdf/sensors/r200.urdf.xacro (robot description, xacro)
@@ -74,7 +74,7 @@
       <origin xyz="${r200_cam_offset_px} ${r200_cam_offset_py} ${r200_cam_offset_pz}" rpy="0 0 0"/>
       <parent link="bracket"/>
-      <child link="camera" />
+      <child link="camera_link" />
     </joint>
-    <link name="camera">
+    <link name="camera_link">
       <visual>
        <origin xyz="0 0 0" rpy="${M_PI/2} 0 ${M_PI/2}"/>
@@ -103,5 +103,5 @@
     <joint name="camera_rgb_joint" type="fixed">
       <origin xyz="${r200_cam_rgb_px} ${r200_cam_rgb_py} ${r200_cam_rgb_pz}" rpy="0 0 0"/>
-      <parent link="camera"/>
+      <parent link="camera_link"/>
       <child link="camera_rgb_frame" />
     </joint>
