Commit message: update astra urdf by Turtlebot REP

File: turtlebot_description/urdf/sensors/astra.urdf.xacro (robot description, xacro)
@@ -4,7 +4,5 @@
   <xacro:include filename="$(find turtlebot_description)/urdf/turtlebot_properties.urdf.xacro"/>
   <!-- Xacro properties -->
-  <xacro:property name="astra_cam_px" value="-0.129"/>
-  <xacro:property name="astra_cam_py" value="0.008"/>
-  <xacro:property name="astra_cam_pz" value="0.281"/>
+  <xacro:property name="astra_cam_py" value="-0.0125"/>
   <xacro:property name="astra_depth_rel_rgb_py" value="0.0250" />
   <xacro:property name="astra_cam_rel_rgb_py"   value="-0.0125" />
@@ -33,5 +31,5 @@
     <link name="camera_link">
       <visual>
-        <origin xyz="0 0 0" rpy="${M_PI/2} 0 ${M_PI/2}"/>
+        <origin xyz="-0.04 0.02 -0.01" rpy="${M_PI/2} 0 ${M_PI/2}"/>
         <geometry>
           <mesh filename="package://turtlebot_description/meshes/sensors/astra.dae" scale="${astra_dae_display_scale} ${astra_dae_display_scale} ${astra_dae_display_scale}"/>

Commit message: update astra urdf

File: turtlebot_description/urdf/sensors/astra.urdf.xacro (robot description, xacro)
@@ -11,5 +11,5 @@
   <xacro:macro name="sensor_astra" params="parent">
     <joint name="camera_rgb_joint" type="fixed">
-      <origin xyz="${astra_cam_px} ${astra_cam_py} ${astra_cam_pz}"
+      <origin xyz="${cam_px} ${astra_cam_py} ${cam_pz}"
               rpy="0 0 0"/>
       <parent link="${parent}"/>
