Commit message: finally making progress on a good asus/kinect xacro formalisation.

File: turtlebot_description/urdf/sensors/asus_xtion_pro.urdf.xacro (robot description, xacro)
@@ -1,95 +1,103 @@
 <?xml version="1.0"?>
-<robot name="turtlebot_hardware" xmlns:xacro="http://ros.org/wiki/xacro">
+<robot name="sensor_asus_xtion_pro" xmlns:xacro="http://ros.org/wiki/xacro"
+                                xmlns:controller="http://playerstage.sourceforge.net/gazebo/xmlschema/#controller"
+                                xmlns:interface="http://playerstage.sourceforge.net/gazebo/xmlschema/#interface"
+                                xmlns:sensor="http://playerstage.sourceforge.net/gazebo/xmlschema/#sensor">
+  <include filename="$(find turtlebot_description)/urdf/common_properties.urdf.xacro"/>
   <include filename="$(find turtlebot_description)/urdf/gazebo.urdf.xacro"/>
-  <include filename="$(find turtlebot_description)/urdf/common_properties.xacro" />
-  <include filename="$(find turtlebot_description)/urdf/turtlebot_properties.xacro" />
-<!-- Macro for ASUS Xtion PRO on Turtlebot. Uses Kinect frame names, but they have moved -->
-<!-- Parameterised in part by the values in turtlebot_properties.urdf.xacro -->
-<xacro:macro name="sensors_asus_xtion_pro" params="parent">
-  <joint name="base_camera_joint" type="fixed">
-    <origin xyz="${cam_px} ${cam_py} ${cam_pz}"
-            rpy="${cam_or} ${cam_op} ${cam_oy}"/>
-    <parent link="${turtlebot_camera_parent_name}" />
-    <child link="camera_link" />
-  </joint>
-  <link name="camera_link">
-    <inertial>
-      <mass value="0.01" />
-      <origin xyz="0 0 0" />
-      <inertia ixx="0.001" ixy="0.0" ixz="0.0"
-        iyy="0.001" iyz="0.0"
-        izz="0.001" />
-    </inertial>
-    <visual>
-      <origin xyz=" 0 0 0 " rpy="0 0 0" />
-      <geometry>
-        <mesh filename="package://turtlebot_description/meshes/sensors/asus_xtion_pro_live.dae"/>
-      </geometry>
-    </visual>
-    <collision>
-      <origin xyz="0.0 0.0 0.0" rpy="0 0 0" />
-      <geometry>
+  <include filename="$(find turtlebot_description)/urdf/common_properties.urdf.xacro" />
+  <include filename="$(find turtlebot_description)/urdf/turtlebot_properties.urdf.xacro" />
+  <!-- Xacro properties -->
+  <xacro:property name="M_SCALE" value="0.001"/>
+  <xacro:property name="depth_rel_rgb_py" value="0.0270" />
+  <xacro:property name="cam_rel_rgb_py"   value="-0.0220" />
+  <!-- Parameterised in part by the values in turtlebot_properties.urdf.xacro -->
+  <xacro:macro name="sensor_asus_xtion_pro" params="parent">
+    <joint name="camera_rgb_joint" type="fixed">
+      <origin xyz="${cam_px} ${cam_py} ${cam_pz}"
+              rpy="${cam_or} ${cam_op} ${cam_oy}"/>
+      <parent link="${parent}"/>
+      <child link="camera_rgb_frame" />
+    </joint>
+    <link name="camera_rgb_frame">
+      <inertial>
+        <mass value="0.001" />
+        <origin xyz="0 0 0" />
+        <inertia ixx="0.0001" ixy="0.0" ixz="0.0"
+          iyy="0.0001" iyz="0.0"
+          izz="0.0001" />
+      </inertial>
+    </link>
+    <joint name="camera_rgb_optical_joint" type="fixed">
+      <origin xyz="0 0 0" rpy="${-M_PI/2} 0 ${-M_PI/2}" />
+      <parent link="camera_rgb_frame" />
+      <child link="camera_rgb_optical_frame" />
+    </joint>
+    <link name="camera_rgb_optical_frame">
+      <inertial>
+        <mass value="0.001" />
+        <origin xyz="0 0 0" />
+        <inertia ixx="0.0001" ixy="0.0" ixz="0.0"
+          iyy="0.0001" iyz="0.0"
+          izz="0.0001" />
+      </inertial>
+    </link>
+    <joint name="camera_joint" type="fixed">
+      <origin xyz="0 ${cam_rel_rgb_py} 0"
+              rpy="0 0 0"/>
+      <parent link="camera_rgb_frame"/>
+      <child link="camera_link"/>
+    </joint>
+    <link name="camera_link">
+      <visual>
+        <origin xyz="-0.01 0 0" rpy="${-M_PI/2} -${M_PI} ${-M_PI/2}"/>
+        <geometry>
+          <mesh filename="package://turtlebot_description/meshes/sensors/asus_xtion_pro_live.dae" scale="${M_SCALE} ${M_SCALE} ${M_SCALE}"/>
+        </geometry>
+      </visual>
+      <collision>
+        <origin xyz="0.0 0.0 0.0" rpy="0 0 0" />
+        <geometry>
         <box size="0.0730 .2760 0.0720"/>
       </geometry>
-    </collision>
-  </link>
-  <joint name="camera_depth_joint" type="fixed">
-    <origin xyz="0 0.049 0" rpy="0 0 0" />
-    <parent link="camera_link" />
-    <child link="camera_depth_frame" />
-  </joint>
-  <link name="camera_depth_frame">
-    <inertial>
-      <mass value="0.01" />
-      <origin xyz="0 0 0" />
-      <inertia ixx="0.001" ixy="0.0" ixz="0.0"
-        iyy="0.001" iyz="0.0"
-        izz="0.001" />
-    </inertial>
-  </link>
-  <joint name="camera_depth_optical_joint" type="fixed">
-    <origin xyz="0 0 0" rpy="${-M_PI/2} 0 ${-M_PI/2}" />
-    <parent link="camera_depth_frame" />
-    <child link="camera_depth_optical_frame" />
-  </joint>
-  <link name="camera_depth_optical_frame">
-    <inertial>
-      <mass value="0.001" />
-      <origin xyz="0 0 0" />
-      <inertia ixx="0.0001" ixy="0.0" ixz="0.0"
-        iyy="0.0001" iyz="0.0"
-        izz="0.0001" />
-    </inertial>
-  </link>
-  <joint name="camera_rgb_joint" type="fixed">
-    <origin xyz="0 0.022 0" rpy="0 0 0" />
-    <parent link="camera_link" />
-    <child link="camera_rgb_frame" />
-  </joint>
-  <link name="camera_rgb_frame">
-    <inertial>
-      <mass value="0.001" />
-      <origin xyz="0 0 0" />
-      <inertia ixx="0.0001" ixy="0.0" ixz="0.0"
-        iyy="0.0001" iyz="0.0"
-        izz="0.0001" />
-    </inertial>
-  </link>
-  <joint name="camera_rgb_optical_joint" type="fixed">
-    <origin xyz="0 0 0" rpy="${-M_PI/2} 0 ${-M_PI/2}" />
-    <parent link="camera_rgb_frame" />
-    <child link="camera_rgb_optical_frame" />
-  </joint>
-  <link name="camera_rgb_optical_frame">
-    <inertial>
-      <mass value="0.001" />
-      <origin xyz="0 0 0" />
-      <inertia ixx="0.0001" ixy="0.0" ixz="0.0"
-        iyy="0.0001" iyz="0.0"
-        izz="0.0001" />
-    </inertial>
-  </link>
-  <!-- RGBD sensor for simulation -->
-  <turtlebot_sim_asus_xtion/>
-</xacro:macro>
+      </collision>
+      <inertial>
+        <mass value="0.01" />
+        <origin xyz="0 0 0" />
+        <inertia ixx="0.001" ixy="0.0" ixz="0.0"
+          iyy="0.001" iyz="0.0"
+          izz="0.001" />
+      </inertial>
+    </link>
+    <joint name="camera_depth_joint" type="fixed">
+      <origin xyz="0 ${depth_rel_rgb_py} 0" rpy="0 0 0" />
+      <parent link="camera_rgb_frame" />
+      <child link="camera_depth_frame" />
+    </joint>
+    <link name="camera_depth_frame">
+      <inertial>
+        <mass value="0.01" />
+        <origin xyz="0 0 0" />
+        <inertia ixx="0.001" ixy="0.0" ixz="0.0"
+          iyy="0.001" iyz="0.0"
+          izz="0.001" />
+      </inertial>
+    </link>
+    <joint name="camera_depth_optical_joint" type="fixed">
+      <origin xyz="0 0 0" rpy="${-M_PI/2} 0 ${-M_PI/2}" />
+      <parent link="camera_depth_frame" />
+      <child link="camera_depth_optical_frame" />
+    </joint>
+    <link name="camera_depth_optical_frame">
+      <inertial>
+        <mass value="0.001" />
+        <origin xyz="0 0 0" />
+        <inertia ixx="0.0001" ixy="0.0" ixz="0.0"
+          iyy="0.0001" iyz="0.0"
+          izz="0.0001" />
+      </inertial>
+    </link>
+    <!-- RGBD sensor for simulation -->
+    <turtlebot_sim_asus_xtion/>
+  </xacro:macro>
 </robot>

File: turtlebot_description/urdf/sensors/kinect.urdf.xacro (robot description, xacro)
@@ -1,6 +1,3 @@
 <?xml version="1.0"?>
-<!--
-  Poles + Kinect for the Turtlebot 2 stack
- -->
 <robot name="sensor_kinect" xmlns:xacro="http://ros.org/wiki/xacro"
                                 xmlns:controller="http://playerstage.sourceforge.net/gazebo/xmlschema/#controller"
@@ -13,26 +10,57 @@
   <!-- Xacro properties -->
   <xacro:property name="M_SCALE" value="0.001"/>
+  <xacro:property name="depth_rel_rgb_py" value="0.0270" />
+  <xacro:property name="cam_rel_rgb_py"   value="0.0135" />
   <!-- Parameterised in part by the values in turtlebot_properties.urdf.xacro -->
   <xacro:macro name="sensor_kinect" params="parent">
-	  <joint name="camera_joint" type="fixed">
-	    <origin xyz="${cam_px} ${cam_py} ${cam_pz}"
-	            rpy="${cam_or} ${cam_op} ${cam_oy}"/>
-	    <parent link="${parent}"/>
-	    <child link="camera_link"/>
-	  </joint>
-	  <link name="camera_link">
-	    <visual>
-	      <origin xyz="0 0 0" rpy="0 0 0"/>
-	      <geometry>
-	        <mesh filename="package://turtlebot_description/meshes/sensors/kinect.dae"/>
-	      </geometry>
+    <joint name="camera_rgb_joint" type="fixed">
+      <origin xyz="${cam_px} ${cam_py} ${cam_pz}"
+              rpy="${cam_or} ${cam_op} ${cam_oy}"/>
+      <parent link="${parent}"/>
+      <child link="camera_rgb_frame" />
+    </joint>
+    <link name="camera_rgb_frame">
+      <inertial>
+        <mass value="0.001" />
+        <origin xyz="0 0 0" />
+        <inertia ixx="0.0001" ixy="0.0" ixz="0.0"
+          iyy="0.0001" iyz="0.0"
+          izz="0.0001" />
+      </inertial>
+    </link>
+    <joint name="camera_rgb_optical_joint" type="fixed">
+      <origin xyz="0 0 0" rpy="${-M_PI/2} 0 ${-M_PI/2}" />
+      <parent link="camera_rgb_frame" />
+      <child link="camera_rgb_optical_frame" />
+    </joint>
+    <link name="camera_rgb_optical_frame">
+      <inertial>
+        <mass value="0.001" />
+        <origin xyz="0 0 0" />
+        <inertia ixx="0.0001" ixy="0.0" ixz="0.0"
+          iyy="0.0001" iyz="0.0"
+          izz="0.0001" />
+      </inertial>
+    </link>
+	<joint name="camera_joint" type="fixed">
+	  <origin xyz="0 ${cam_rel_rgb_py} 0"
+	          rpy="0 0 0"/>
+	  <parent link="camera_rgb_frame"/>
+	  <child link="camera_link"/>
+	</joint>
+    <link name="camera_link">
+	  <visual>
+	    <origin xyz="0 0 0" rpy="0 0 0"/>
+	    <geometry>
+	      <mesh filename="package://turtlebot_description/meshes/sensors/kinect.dae"/>
+	    </geometry>
         <xacro:insert_block name="material_light_grey"/>
-	    </visual>
-	    <collision>
-	      <origin xyz="-0.0315 0.0 -0.017" rpy="0 0 0"/>
-	      <geometry>
-	        <box size="0.07271 0.27794 0.073"/>
-	      </geometry>
-	    </collision>
+	  </visual>
+	  <collision>
+	    <origin xyz="-0.0315 0.0 -0.017" rpy="0 0 0"/>
+	    <geometry>
+	      <box size="0.07271 0.27794 0.073"/>
+	    </geometry>
+	  </collision>
       <inertial>
         <mass value="0.01"/>
@@ -42,66 +70,38 @@
                  izz="0.01" />
       </inertial>
-	  </link>
+	</link>
     <!-- The fixed joints & links below are usually published by static_transformers launched by the OpenNi launch
          files. However, for Gazebo simulation we need them, so we add them here.
          (Hence, don't publish them additionally!) -->
-	  <joint name="camera_depth_joint" type="fixed">
-	    <origin xyz="0 ${depth_rel_cam_py} 0" rpy="0 0 0" />
-	    <parent link="camera_link" />
-	    <child link="camera_depth_frame" />
-	  </joint>
-	  <link name="camera_depth_frame">
-	    <inertial>
-	      <mass value="0.01" />
-	      <origin xyz="0 0 0" />
-	      <inertia ixx="0.001" ixy="0.0" ixz="0.0"
-	        iyy="0.001" iyz="0.0"
-	        izz="0.001" />
-	    </inertial>
-	  </link>
-	  <joint name="camera_depth_optical_joint" type="fixed">
-	    <origin xyz="0 0 0" rpy="${-M_PI/2} 0 ${-M_PI/2}" />
-	    <parent link="camera_depth_frame" />
-	    <child link="camera_depth_optical_frame" />
-	  </joint>
-	  <link name="camera_depth_optical_frame">
-	    <inertial>
-	      <mass value="0.001" />
-	      <origin xyz="0 0 0" />
-	      <inertia ixx="0.0001" ixy="0.0" ixz="0.0"
-	        iyy="0.0001" iyz="0.0"
-	        izz="0.0001" />
-	    </inertial>
-	  </link>
-	  <joint name="camera_rgb_joint" type="fixed">
-        <origin xyz="0 ${rgb_rel_cam_py} 0" rpy="0 0 0"/>
-	    <parent link="camera_link" />
-	    <child link="camera_rgb_frame" />
-	  </joint>
-	  <link name="camera_rgb_frame">
-	    <inertial>
-	      <mass value="0.001" />
-	      <origin xyz="0 0 0" />
-	      <inertia ixx="0.0001" ixy="0.0" ixz="0.0"
-	        iyy="0.0001" iyz="0.0"
-	        izz="0.0001" />
-	    </inertial>
-	  </link>
-	  <joint name="camera_rgb_optical_joint" type="fixed">
-	    <origin xyz="0 0 0" rpy="${-M_PI/2} 0 ${-M_PI/2}" />
-	    <parent link="camera_rgb_frame" />
-	    <child link="camera_rgb_optical_frame" />
-	  </joint>
-	  <link name="camera_rgb_optical_frame">
-	    <inertial>
-	      <mass value="0.001" />
-	      <origin xyz="0 0 0" />
-	      <inertia ixx="0.0001" ixy="0.0" ixz="0.0"
-	        iyy="0.0001" iyz="0.0"
-	        izz="0.0001" />
-	    </inertial>
-	  </link>
-	  <!-- Kinect sensor for simulation -->
-	  <turtlebot_sim_kinect/>
-	</xacro:macro>
+	<joint name="camera_depth_joint" type="fixed">
+	  <origin xyz="0 ${depth_rel_rgb_py} 0" rpy="0 0 0" />
+	  <parent link="camera_rgb_frame" />
+	  <child link="camera_depth_frame" />
+	</joint>
+	<link name="camera_depth_frame">
+	  <inertial>
+	    <mass value="0.01" />
+	    <origin xyz="0 0 0" />
+	    <inertia ixx="0.001" ixy="0.0" ixz="0.0"
+	      iyy="0.001" iyz="0.0"
+	      izz="0.001" />
+	  </inertial>
+	</link>
+	<joint name="camera_depth_optical_joint" type="fixed">
+	  <origin xyz="0 0 0" rpy="${-M_PI/2} 0 ${-M_PI/2}" />
+	  <parent link="camera_depth_frame" />
+	  <child link="camera_depth_optical_frame" />
+	</joint>
+	<link name="camera_depth_optical_frame">
+	  <inertial>
+	    <mass value="0.001" />
+	    <origin xyz="0 0 0" />
+	    <inertia ixx="0.0001" ixy="0.0" ixz="0.0"
+	      iyy="0.0001" iyz="0.0"
+	      izz="0.0001" />
+	  </inertial>
+	</link>
+	<!-- Kinect sensor for simulation -->
+	<turtlebot_sim_kinect/>
+  </xacro:macro>
 </robot>

File: turtlebot_description/urdf/turtlebot_library.urdf.xacro (robot description, xacro)
@@ -9,4 +9,5 @@
   <include filename="$(find turtlebot_description)/urdf/stacks/hexagons.urdf.xacro"/>
   <include filename="$(find turtlebot_description)/urdf/sensors/kinect.urdf.xacro"/>
+  <include filename="$(find turtlebot_description)/urdf/sensors/asus_xtion_pro.urdf.xacro"/>
   <include filename="$(find kobuki_description)/urdf/kobuki.urdf.xacro" />
 </robot>

File: turtlebot_description/urdf/turtlebot_properties.urdf.xacro (robot description, xacro)
@@ -12,5 +12,10 @@
      ======================================================================
      -->
-	<!-- Actual REP specifications from Turtlebot 1
+    <!--
+      Actual REP specifications from base_link to rgb frame
+        [x:-0.087m, y:-0.005m, z:0.287m]
+      Is this actually correct?
+    -->
+	<!-- From Turtlebot 1, this is base_link to camera_link with offsets for cam frames
 	<property name="cam_px" value="-0.087" />
 	<property name="cam_py" value="0" />
@@ -23,12 +28,9 @@
 	 -->
 	 <!-- Yujin specifications - need to double check on these -->
-	<property name="cam_px" value="-0.060" />
-	<property name="cam_py" value="0" />
+	<property name="cam_px" value="-0.087" />
+	<property name="cam_py" value="-0.0135" />
 	<property name="cam_pz" value="0.2680" />
 	<property name="cam_or" value="0" />
 	<property name="cam_op" value="0" />
 	<property name="cam_oy" value="0" />
-     <!-- Yujin specifications - need to double check on these -->
-    <property name="depth_rel_cam_py" value="0.0125" />
-	<property name="rgb_rel_cam_py"   value="-0.0125" />
 </robot>

Commit message: found a bug, xacro globals get confused when pulling asus and kinect into turtlebot_library.xacro. fixed.

File: turtlebot_description/urdf/sensors/asus_xtion_pro.urdf.xacro (robot description, xacro)
@@ -10,6 +10,6 @@
   <!-- Xacro properties -->
   <xacro:property name="M_SCALE" value="0.001"/>
-  <xacro:property name="depth_rel_rgb_py" value="0.0270" />
-  <xacro:property name="cam_rel_rgb_py"   value="-0.0220" />
+  <xacro:property name="asus_xtion_pro_depth_rel_rgb_py" value="0.0270" />
+  <xacro:property name="asus_xtion_pro_cam_rel_rgb_py"   value="-0.0220" />
   <!-- Parameterised in part by the values in turtlebot_properties.urdf.xacro -->
   <xacro:macro name="sensor_asus_xtion_pro" params="parent">
@@ -44,5 +44,5 @@
     </link>
     <joint name="camera_joint" type="fixed">
-      <origin xyz="0 ${cam_rel_rgb_py} 0"
+      <origin xyz="0 ${asus_xtion_pro_cam_rel_rgb_py} 0"
               rpy="0 0 0"/>
       <parent link="camera_rgb_frame"/>
@@ -71,5 +71,5 @@
     </link>
     <joint name="camera_depth_joint" type="fixed">
-      <origin xyz="0 ${depth_rel_rgb_py} 0" rpy="0 0 0" />
+      <origin xyz="0 ${asus_xtion_pro_depth_rel_rgb_py} 0" rpy="0 0 0" />
       <parent link="camera_rgb_frame" />
       <child link="camera_depth_frame" />

File: turtlebot_description/urdf/sensors/kinect.urdf.xacro (robot description, xacro)
@@ -10,6 +10,6 @@
   <!-- Xacro properties -->
   <xacro:property name="M_SCALE" value="0.001"/>
-  <xacro:property name="depth_rel_rgb_py" value="0.0270" />
-  <xacro:property name="cam_rel_rgb_py"   value="0.0135" />
+  <xacro:property name="kinect_depth_rel_rgb_py" value="0.0270" />
+  <xacro:property name="kinect_cam_rel_rgb_py"   value="0.0135" />
   <!-- Parameterised in part by the values in turtlebot_properties.urdf.xacro -->
   <xacro:macro name="sensor_kinect" params="parent">
@@ -44,5 +44,5 @@
     </link>
 	<joint name="camera_joint" type="fixed">
-	  <origin xyz="0 ${cam_rel_rgb_py} 0"
+	  <origin xyz="0 ${kinect_cam_rel_rgb_py} 0"
 	          rpy="0 0 0"/>
 	  <parent link="camera_rgb_frame"/>
@@ -75,5 +75,5 @@
          (Hence, don't publish them additionally!) -->
 	<joint name="camera_depth_joint" type="fixed">
-	  <origin xyz="0 ${depth_rel_rgb_py} 0" rpy="0 0 0" />
+	  <origin xyz="0 ${kinect_depth_rel_rgb_py} 0" rpy="0 0 0" />
 	  <parent link="camera_rgb_frame" />
 	  <child link="camera_depth_frame" />
