Commit message: * updates collada meshes with correct units to be properly visualised in both rviz and gazebo * fixes related with a positioning bug in the kobuki base * fixes camera_rgb_frame position (refs #60) * introduces new kinect mesh with nice surface * moves create-specific parts (mostly gazebo related) out to create package

File: turtlebot_description/urdf/sensors/asus_xtion_pro.urdf.xacro (robot description, xacro)
@@ -1,9 +1,9 @@
 <?xml version="1.0"?>
 <robot name="sensor_asus_xtion_pro" xmlns:xacro="http://ros.org/wiki/xacro"
-                                xmlns:controller="http://playerstage.sourceforge.net/gazebo/xmlschema/#controller"
-                                xmlns:interface="http://playerstage.sourceforge.net/gazebo/xmlschema/#interface"
-                                xmlns:sensor="http://playerstage.sourceforge.net/gazebo/xmlschema/#sensor">
+                                    xmlns:controller="http://playerstage.sourceforge.net/gazebo/xmlschema/#controller"
+                                    xmlns:interface="http://playerstage.sourceforge.net/gazebo/xmlschema/#interface"
+                                    xmlns:sensor="http://playerstage.sourceforge.net/gazebo/xmlschema/#sensor">
   <include filename="$(find turtlebot_description)/urdf/common_properties.urdf.xacro"/>
-  <include filename="$(find turtlebot_description)/urdf/gazebo.urdf.xacro"/>
+  <include filename="$(find turtlebot_description)/urdf/turtlebot_gazebo.urdf.xacro"/>
   <include filename="$(find turtlebot_description)/urdf/common_properties.urdf.xacro" />
   <include filename="$(find turtlebot_description)/urdf/turtlebot_properties.urdf.xacro" />
@@ -99,5 +99,5 @@
     </link>
     <!-- RGBD sensor for simulation -->
-    <turtlebot_sim_asus_xtion/>
+<!--     <turtlebot_sim_xtion/> not working currently -->
   </xacro:macro>
 </robot>

File: turtlebot_description/urdf/sensors/kinect.urdf.xacro (robot description, xacro)
@@ -1,20 +1,15 @@
 <?xml version="1.0"?>
 <robot name="sensor_kinect" xmlns:xacro="http://ros.org/wiki/xacro"
-                                xmlns:controller="http://playerstage.sourceforge.net/gazebo/xmlschema/#controller"
-                                xmlns:interface="http://playerstage.sourceforge.net/gazebo/xmlschema/#interface"
-                                xmlns:sensor="http://playerstage.sourceforge.net/gazebo/xmlschema/#sensor">
+                            xmlns:controller="http://playerstage.sourceforge.net/gazebo/xmlschema/#controller"
+                            xmlns:interface="http://playerstage.sourceforge.net/gazebo/xmlschema/#interface"
+                            xmlns:sensor="http://playerstage.sourceforge.net/gazebo/xmlschema/#sensor">
   <include filename="$(find turtlebot_description)/urdf/common_properties.urdf.xacro"/>
-  <include filename="$(find turtlebot_description)/urdf/gazebo.urdf.xacro"/>
+  <include filename="$(find turtlebot_description)/urdf/turtlebot_gazebo.urdf.xacro"/>
   <include filename="$(find turtlebot_description)/urdf/common_properties.urdf.xacro" />
   <include filename="$(find turtlebot_description)/urdf/turtlebot_properties.urdf.xacro" />
-  <!-- Xacro properties -->
-  <xacro:property name="M_SCALE" value="0.001"/>
-  <xacro:property name="kinect_depth_rel_rgb_py" value="0.0270" />
-  <xacro:property name="kinect_cam_rel_rgb_py"   value="0.0135" />
   <!-- Parameterised in part by the values in turtlebot_properties.urdf.xacro -->
   <xacro:macro name="sensor_kinect" params="parent">
     <joint name="camera_rgb_joint" type="fixed">
-      <origin xyz="${cam_px} ${cam_py} ${cam_pz}"
-              rpy="${cam_or} ${cam_op} ${cam_oy}"/>
+      <origin xyz="${cam_px} ${cam_py} ${cam_pz}" rpy="${cam_or} ${cam_op} ${cam_oy}"/>
       <parent link="${parent}"/>
       <child link="camera_rgb_frame" />
@@ -25,6 +20,6 @@
         <origin xyz="0 0 0" />
         <inertia ixx="0.0001" ixy="0.0" ixz="0.0"
-          iyy="0.0001" iyz="0.0"
-          izz="0.0001" />
+                 iyy="0.0001" iyz="0.0"
+                 izz="0.0001" />
       </inertial>
     </link>
@@ -39,22 +34,20 @@
         <origin xyz="0 0 0" />
         <inertia ixx="0.0001" ixy="0.0" ixz="0.0"
-          iyy="0.0001" iyz="0.0"
-          izz="0.0001" />
+                 iyy="0.0001" iyz="0.0"
+                 izz="0.0001" />
       </inertial>
     </link>
-	<joint name="camera_joint" type="fixed">
-	  <origin xyz="0 ${kinect_cam_rel_rgb_py} 0"
-	          rpy="0 0 0"/>
-	  <parent link="camera_rgb_frame"/>
-	  <child link="camera_link"/>
-	</joint>
+  <joint name="camera_joint" type="fixed">
+    <origin xyz="-0.031 ${-cam_py} -0.016" rpy="0 0 0"/>
+    <parent link="camera_rgb_frame"/>
+    <child link="camera_link"/>
+  </joint>
     <link name="camera_link">
-	  <visual>
-	    <origin xyz="0 0 0" rpy="0 0 0"/>
-	    <geometry>
-	      <mesh filename="package://turtlebot_description/meshes/sensors/kinect.dae"/>
-	    </geometry>
-        <xacro:insert_block name="material_light_grey"/>
-	  </visual>
+    <visual>
+     <origin xyz="0 0 0" rpy="0 0 ${M_PI/2}"/>
+      <geometry>
+       <mesh filename="package://turtlebot_description/meshes/sensors/kinect.dae"/>
+      </geometry>
+    </visual>
 	  <collision>
 	    <origin xyz="-0.0315 0.0 -0.017" rpy="0 0 0"/>
@@ -63,28 +56,28 @@
 	    </geometry>
 	  </collision>
-      <inertial>
-        <mass value="0.01"/>
-        <origin xyz="0 0 0"/>
-        <inertia ixx="0.01" ixy="0.0" ixz="0.0"
-                 iyy="0.01" iyz="0.0"
-                 izz="0.01" />
-      </inertial>
-	</link>
-    <!-- The fixed joints & links below are usually published by static_transformers launched by the OpenNi launch
-         files. However, for Gazebo simulation we need them, so we add them here.
-         (Hence, don't publish them additionally!) -->
+    <inertial>
+      <mass value="0.001" />
+      <origin xyz="0 0 0" />
+      <inertia ixx="0.0001" ixy="0.0" ixz="0.0"
+               iyy="0.0001" iyz="0.0"
+               izz="0.0001" />
+    </inertial>
+  </link>
+  <!-- The fixed joints & links below are usually published by static_transformers launched by the OpenNi launch
+       files. However, for Gazebo simulation we need them, so we add them here.
+       (Hence, don't publish them additionally!) -->
 	<joint name="camera_depth_joint" type="fixed">
-	  <origin xyz="0 ${kinect_depth_rel_rgb_py} 0" rpy="0 0 0" />
+	  <origin xyz="0 ${2 * -cam_py} 0" rpy="0 0 0" />
 	  <parent link="camera_rgb_frame" />
 	  <child link="camera_depth_frame" />
 	</joint>
 	<link name="camera_depth_frame">
-	  <inertial>
-	    <mass value="0.01" />
-	    <origin xyz="0 0 0" />
-	    <inertia ixx="0.001" ixy="0.0" ixz="0.0"
-	      iyy="0.001" iyz="0.0"
-	      izz="0.001" />
-	  </inertial>
+    <inertial>
+      <mass value="0.001" />
+      <origin xyz="0 0 0" />
+      <inertia ixx="0.0001" ixy="0.0" ixz="0.0"
+               iyy="0.0001" iyz="0.0"
+               izz="0.0001" />
+    </inertial>
 	</link>
 	<joint name="camera_depth_optical_joint" type="fixed">
@@ -94,14 +87,14 @@
 	</joint>
 	<link name="camera_depth_optical_frame">
-	  <inertial>
-	    <mass value="0.001" />
-	    <origin xyz="0 0 0" />
-	    <inertia ixx="0.0001" ixy="0.0" ixz="0.0"
-	      iyy="0.0001" iyz="0.0"
-	      izz="0.0001" />
-	  </inertial>
+    <inertial>
+      <mass value="0.001" />
+      <origin xyz="0 0 0" />
+      <inertia ixx="0.0001" ixy="0.0" ixz="0.0"
+               iyy="0.0001" iyz="0.0"
+               izz="0.0001" />
+    </inertial>
 	</link>
 	<!-- Kinect sensor for simulation -->
-	<turtlebot_sim_kinect/>
+<!-- 	<turtlebot_sim_kinect/> not working currently -->
   </xacro:macro>
 </robot>

File: turtlebot_description/urdf/stacks/hexagons.urdf.xacro (robot description, xacro)
@@ -17,9 +17,8 @@
     <link name="pole_bottom_${number}_link">
       <visual>
-        <origin xyz="0 0 0" rpy="${M_PI/2} 0 ${M_PI/2}"/>
-        <geometry>
-          <mesh filename="package://turtlebot_description/meshes/stacks/hexagons/pole_bottom.dae" scale="${M_SCALE} ${M_SCALE} ${M_SCALE}"/>
-        </geometry>
-        <xacro:insert_block name="material_light_grey"/>
+        <origin xyz="0 0 0" rpy="0 0 0"/>
+        <geometry>
+          <mesh filename="package://turtlebot_description/meshes/stacks/hexagons/pole_bottom.dae"/>
+        </geometry>
       </visual>
       <collision>
@@ -46,9 +45,8 @@
     <link name="pole_middle_${number}_link">
       <visual>
-        <origin xyz="0 0 0" rpy="${-M_PI/2} ${M_PI} 0"/>
-        <geometry>
-          <mesh filename="package://turtlebot_description/meshes/stacks/hexagons/pole_middle.dae" scale="${M_SCALE} ${M_SCALE} ${M_SCALE}"/>
-        </geometry>
-        <xacro:insert_block name="material_light_grey"/>
+        <origin xyz="0 0 0" rpy="0 ${M_PI} 0"/>
+        <geometry>
+          <mesh filename="package://turtlebot_description/meshes/stacks/hexagons/pole_middle.dae"/>
+        </geometry>
       </visual>
       <collision>
@@ -75,9 +73,8 @@
     <link name="pole_top_${number}_link">
       <visual>
-        <origin xyz=" 0 0 0" rpy="${M_PI/2} 0 ${M_PI/2}"/>
-        <geometry>
-          <mesh filename="package://turtlebot_description/meshes/stacks/hexagons/pole_top.dae" scale="${M_SCALE} ${M_SCALE} ${M_SCALE}"/>
-        </geometry>
-        <xacro:insert_block name="material_light_grey"/>
+        <origin xyz=" 0 0 0" rpy="0 0 0"/>
+        <geometry>
+          <mesh filename="package://turtlebot_description/meshes/stacks/hexagons/pole_top.dae"/>
+        </geometry>
       </visual>
       <collision>
@@ -104,9 +101,9 @@
     <link name="pole_kinect_${number}_link">
       <visual>
-        <origin xyz="0 0 0" rpy="${-M_PI/2} ${M_PI} 0"/>
-        <geometry>
-          <mesh filename="package://turtlebot_description/meshes/stacks/hexagons/pole_kinect.dae" scale="${M_SCALE} ${M_SCALE} ${M_SCALE}"/>
-        </geometry>
-        <xacro:insert_block name="material_light_grey"/>
+        <origin xyz="0 0 0" rpy="0 0 0"/>
+<!--         <origin xyz="0 0 0" rpy="${-M_PI/2} ${M_PI} 0"/> -->
+        <geometry>
+          <mesh filename="package://turtlebot_description/meshes/stacks/hexagons/pole_kinect.dae"/>
+        </geometry>
       </visual>
       <collision>
@@ -131,12 +128,12 @@
   -->
   <xacro:macro name="stack_hexagons" params="parent">
-    <stack_bottom_pole parent="${parent}" number="0" x_loc= "0.120" y_loc= "0.082" z_loc="0.0980"/>
-    <stack_bottom_pole parent="${parent}" number="1" x_loc= "0.055" y_loc= "0.120" z_loc="0.0980"/>
-    <stack_bottom_pole parent="${parent}" number="2" x_loc="-0.055" y_loc= "0.120" z_loc="0.0980"/>
-    <stack_bottom_pole parent="${parent}" number="3" x_loc= "0.120" y_loc="-0.082" z_loc="0.0980"/>
-    <stack_bottom_pole parent="${parent}" number="4" x_loc= "0.055" y_loc="-0.120" z_loc="0.0980"/>
-    <stack_bottom_pole parent="${parent}" number="5" x_loc="-0.055" y_loc="-0.120" z_loc="0.0980"/>
+    <stack_bottom_pole parent="${parent}" number="0" x_loc= "0.120" y_loc= "0.082" z_loc="0.1028"/>
+    <stack_bottom_pole parent="${parent}" number="1" x_loc= "0.055" y_loc= "0.120" z_loc="0.1028"/>
+    <stack_bottom_pole parent="${parent}" number="2" x_loc="-0.055" y_loc= "0.120" z_loc="0.1028"/>
+    <stack_bottom_pole parent="${parent}" number="3" x_loc= "0.120" y_loc="-0.082" z_loc="0.1028"/>
+    <stack_bottom_pole parent="${parent}" number="4" x_loc= "0.055" y_loc="-0.120" z_loc="0.1028"/>
+    <stack_bottom_pole parent="${parent}" number="5" x_loc="-0.055" y_loc="-0.120" z_loc="0.1028"/>
     <joint name="plate_bottom_joint" type="fixed">
-      <origin xyz="0.02364 0.0 0.1256" rpy="0 0 0"/>
+      <origin xyz="0.02364 0.0 0.1306" rpy="0 0 0"/>
       <parent link="${parent}"/>
       <child link="plate_bottom_link"/>
@@ -144,14 +141,13 @@
     <link name="plate_bottom_link">
       <visual>
-        <origin xyz="0 0 0" rpy="${M_PI/2} 0 ${M_PI/2}"/>
-        <geometry>
-          <mesh filename="package://turtlebot_description/meshes/stacks/hexagons/plate_bottom.dae" scale="${M_SCALE} ${M_SCALE} ${M_SCALE}"/>
-        </geometry>
-        <xacro:insert_block name="material_black"/>
-      </visual>
-      <collision>
-        <origin xyz="0 0 0" rpy="0 0 0"/>
-        <geometry>
-          <box size="0.26727 0.345 0.006"/>
+        <origin xyz="0 0 0" rpy="0 0 0"/>
+        <geometry>
+          <mesh filename="package://turtlebot_description/meshes/stacks/hexagons/plate_bottom.dae"/>
+        </geometry>
+      </visual>
+      <collision>
+        <origin xyz="0 0 0" rpy="0 0 0"/>
+        <geometry>
+          <box size="0.26727 0.340 0.006"/>
         </geometry>
       </collision>
@@ -164,10 +160,10 @@
       </inertial>
     </link>
-    <stack_middle_pole parent="${parent}" number="0" x_loc= "0.0381" y_loc= "0.1505" z_loc="0.1590"/>
-    <stack_middle_pole parent="${parent}" number="1" x_loc= "0.0381" y_loc="-0.1505" z_loc="0.1590"/>
-    <stack_middle_pole parent="${parent}" number="2" x_loc="-0.0381" y_loc= "0.1505" z_loc="0.1590"/>
-    <stack_middle_pole parent="${parent}" number="3" x_loc="-0.0381" y_loc="-0.1505" z_loc="0.1590"/>
+    <stack_middle_pole parent="${parent}" number="0" x_loc= "0.0381" y_loc= "0.1505" z_loc="0.1640"/>
+    <stack_middle_pole parent="${parent}" number="1" x_loc= "0.0381" y_loc="-0.1505" z_loc="0.1640"/>
+    <stack_middle_pole parent="${parent}" number="2" x_loc="-0.0381" y_loc= "0.1505" z_loc="0.1640"/>
+    <stack_middle_pole parent="${parent}" number="3" x_loc="-0.0381" y_loc="-0.1505" z_loc="0.1640"/>
     <joint name="plate_middle_joint" type="fixed">
-      <origin xyz="-0.01364 0.0 0.1824" rpy="0 0 0"/>
+      <origin xyz="-0.01364 0.0 0.1874" rpy="0 0 0"/>
       <parent link="${parent}"/>
       <child link="plate_middle_link"/>
@@ -175,9 +171,8 @@
     <link name="plate_middle_link">
       <visual>
-        <origin xyz="0 0 0" rpy="${M_PI/2} 0 -${M_PI/2}"/>
-        <geometry>
-          <mesh filename="package://turtlebot_description/meshes/stacks/hexagons/plate_middle.dae" scale="${M_SCALE} ${M_SCALE} ${M_SCALE}"/>
-        </geometry>
-        <xacro:insert_block name="material_black"/>
+        <origin xyz="0 0 0" rpy="0 0 0"/>
+        <geometry>
+          <mesh filename="package://turtlebot_description/meshes/stacks/hexagons/plate_middle.dae"/>
+        </geometry>
       </visual>
       <collision>
@@ -194,13 +189,13 @@
                  izz="0.01" />
       </inertial>
-	</link>
-    <stack_top_pole parent="${parent}" number="0" x_loc= "0.0381" y_loc= "0.1505" z_loc="0.2870"/>
-    <stack_top_pole parent="${parent}" number="1" x_loc= "0.0381" y_loc="-0.1505" z_loc="0.2870"/>
-    <stack_top_pole parent="${parent}" number="2" x_loc="-0.0381" y_loc= "0.1505" z_loc="0.2870"/>
-    <stack_top_pole parent="${parent}" number="3" x_loc="-0.0381" y_loc="-0.1505" z_loc="0.2870"/>
-    <stack_3d_sensor_pole parent="${parent}" number="0" x_loc="-0.1024" y_loc= "0.098" z_loc="0.2322"/>
-    <stack_3d_sensor_pole parent="${parent}" number="1" x_loc="-0.1024" y_loc="-0.098" z_loc="0.2322"/>
+    </link>
+    <stack_top_pole parent="${parent}" number="0" x_loc= "0.0381" y_loc= "0.1505" z_loc="0.2920"/>
+    <stack_top_pole parent="${parent}" number="1" x_loc= "0.0381" y_loc="-0.1505" z_loc="0.2920"/>
+    <stack_top_pole parent="${parent}" number="2" x_loc="-0.0381" y_loc= "0.1505" z_loc="0.2920"/>
+    <stack_top_pole parent="${parent}" number="3" x_loc="-0.0381" y_loc="-0.1505" z_loc="0.2920"/>
+    <stack_3d_sensor_pole parent="${parent}" number="0" x_loc="-0.1024" y_loc= "0.098" z_loc="0.2372"/>
+    <stack_3d_sensor_pole parent="${parent}" number="1" x_loc="-0.1024" y_loc="-0.098" z_loc="0.2372"/>
     <joint name="plate_top_joint" type="fixed">
-      <origin xyz="-0.01364 0.0  0.3916" rpy="0 0 0"/>
+      <origin xyz="-0.01364 0.0  0.3966" rpy="0 0 0"/>
       <parent link="${parent}"/>
       <child link="plate_top_link"/>
@@ -208,9 +203,8 @@
     <link name="plate_top_link">
       <visual>
-        <origin xyz="0 0 0" rpy="${M_PI/2} 0 -${M_PI/2}"/>
-        <geometry>
-          <mesh filename="package://turtlebot_description/meshes/stacks/hexagons/plate_top.dae" scale="${M_SCALE} ${M_SCALE} ${M_SCALE}"/>
-        </geometry>
-        <xacro:insert_block name="material_black"/>
+        <origin xyz="0 0 0" rpy="0 0 0"/>
+        <geometry>
+          <mesh filename="package://turtlebot_description/meshes/stacks/hexagons/plate_top.dae"/>
+        </geometry>
       </visual>
       <collision>

File: turtlebot_description/urdf/turtlebot_library.urdf.xacro (robot description, xacro)
@@ -17,4 +17,4 @@
   <include filename="$(find turtlebot_description)/urdf/sensors/asus_xtion_pro.urdf.xacro"/>
   <!-- Gazebo -->
-  <include filename="$(find turtlebot_description)/urdf/gazebo.urdf.xacro"/>
+  <include filename="$(find turtlebot_description)/urdf/turtlebot_gazebo.urdf.xacro"/>
 </robot>

File: turtlebot_description/urdf/turtlebot_properties.urdf.xacro (robot description, xacro)
@@ -20,5 +20,5 @@
    -->
 	<property name="cam_px" value="-0.087" />
-	<property name="cam_py" value="-0.005" />
+	<property name="cam_py" value="-0.0125" />
 	<property name="cam_pz" value="0.2870" />
 	<property name="cam_or" value="0" />
