Commit message: move kobuki and hexagon references to updated base_link at the bottom of the base to match the create convention.

File: turtlebot_description/urdf/stacks/hexagons.urdf.xacro (robot description, xacro)
@@ -125,14 +125,14 @@
   </xacro:macro>
   <xacro:macro name="stack_hexagons" params="parent">
-	<stack_bottom_pole    parent="${parent}" number="0" x_loc= "0.120" y_loc= "0.082" z_loc="0.0534"/>
-	<stack_bottom_pole    parent="${parent}" number="1" x_loc= "0.055" y_loc= "0.120" z_loc="0.0534"/>
-	<stack_bottom_pole    parent="${parent}" number="2" x_loc="-0.055" y_loc= "0.120" z_loc="0.0534"/>
-    <stack_bottom_pole    parent="${parent}" number="3" x_loc= "0.120" y_loc="-0.082" z_loc="0.0534"/>
-    <stack_bottom_pole    parent="${parent}" number="4" x_loc= "0.055" y_loc="-0.120" z_loc="0.0534"/>
-    <stack_bottom_pole    parent="${parent}" number="5" x_loc="-0.055" y_loc="-0.120" z_loc="0.0534"/>
-    <stack_3d_sensor_pole parent="${parent}" number="0" x_loc="-0.1024" y_loc= "0.098" z_loc="0.259"/>
-    <stack_3d_sensor_pole parent="${parent}" number="1" x_loc="-0.1024" y_loc="-0.098" z_loc="0.259"/>
+	<stack_bottom_pole    parent="${parent}" number="0" x_loc= "0.120" y_loc= "0.082" z_loc="0.0714"/>
+	<stack_bottom_pole    parent="${parent}" number="1" x_loc= "0.055" y_loc= "0.120" z_loc="0.0714"/>
+	<stack_bottom_pole    parent="${parent}" number="2" x_loc="-0.055" y_loc= "0.120" z_loc="0.0714"/>
+    <stack_bottom_pole    parent="${parent}" number="3" x_loc= "0.120" y_loc="-0.082" z_loc="0.0714"/>
+    <stack_bottom_pole    parent="${parent}" number="4" x_loc= "0.055" y_loc="-0.120" z_loc="0.0714"/>
+    <stack_bottom_pole    parent="${parent}" number="5" x_loc="-0.055" y_loc="-0.120" z_loc="0.0714"/>
+    <stack_3d_sensor_pole parent="${parent}" number="0" x_loc="-0.1024" y_loc= "0.098" z_loc="0.277"/>
+    <stack_3d_sensor_pole parent="${parent}" number="1" x_loc="-0.1024" y_loc="-0.098" z_loc="0.277"/>
 		<joint name="plate_bottom_joint" type="fixed">
-		  <origin xyz="0.0 0.0  0.1026" rpy="0 0 0"/>
+		  <origin xyz="0.0 0.0  0.1206" rpy="0 0 0"/>
 		  <parent link="${parent}"/>
 		  <child link="plate_bottom_link"/>
@@ -161,10 +161,10 @@
       </inertial>
 		</link>
-		<stack_middle_pole parent="${parent}" number="0" x_loc= "0.0702" y_loc= "0.1314" z_loc="0.1694"/>
-		<stack_middle_pole parent="${parent}" number="1" x_loc="-0.0503" y_loc= "0.1314" z_loc="0.1694"/>
-		<stack_middle_pole parent="${parent}" number="2" x_loc= "0.0702" y_loc="-0.1314" z_loc="0.1694"/>
-		<stack_middle_pole parent="${parent}" number="3" x_loc="-0.0503" y_loc="-0.1314" z_loc="0.1694"/>
+		<stack_middle_pole parent="${parent}" number="0" x_loc= "0.0702" y_loc= "0.1314" z_loc="0.1874"/>
+		<stack_middle_pole parent="${parent}" number="1" x_loc="-0.0503" y_loc= "0.1314" z_loc="0.1874"/>
+		<stack_middle_pole parent="${parent}" number="2" x_loc= "0.0702" y_loc="-0.1314" z_loc="0.1874"/>
+		<stack_middle_pole parent="${parent}" number="3" x_loc="-0.0503" y_loc="-0.1314" z_loc="0.1874"/>
 		<joint name="plate_middle_joint" type="fixed">
-		  <origin xyz="0.0 0.0 0.1594" rpy="0 0 0"/>
+		  <origin xyz="0.0 0.0 0.1774" rpy="0 0 0"/>
 		  <parent link="${parent}"/>
 		  <child link="plate_middle_link"/>
@@ -192,10 +192,10 @@
       </inertial>
 		</link>
-		<stack_top_pole parent="${parent}" number="0" x_loc= "0.0702" y_loc= "0.1314" z_loc="0.1534"/>
-		<stack_top_pole parent="${parent}" number="1" x_loc="-0.0503" y_loc= "0.1314" z_loc="0.1534"/>
-		<stack_top_pole parent="${parent}" number="2" x_loc= "0.0702" y_loc="-0.1314" z_loc="0.1534"/>
-		<stack_top_pole parent="${parent}" number="3" x_loc="-0.0503" y_loc="-0.1314" z_loc="0.1534"/>
+		<stack_top_pole parent="${parent}" number="0" x_loc= "0.0702" y_loc= "0.1314" z_loc="0.1714"/>
+		<stack_top_pole parent="${parent}" number="1" x_loc="-0.0503" y_loc= "0.1314" z_loc="0.1714"/>
+		<stack_top_pole parent="${parent}" number="2" x_loc= "0.0702" y_loc="-0.1314" z_loc="0.1714"/>
+		<stack_top_pole parent="${parent}" number="3" x_loc="-0.0503" y_loc="-0.1314" z_loc="0.1714"/>
 		<joint name="plate_top_joint" type="fixed">
-		  <origin xyz="0.0 0.0  0.3686" rpy="0 0 0"/>
+		  <origin xyz="0.0 0.0  0.3866" rpy="0 0 0"/>
 		  <parent link="${parent}"/>
 		  <child link="plate_top_link"/>

File: turtlebot_description/urdf/turtlebot_properties.urdf.xacro (robot description, xacro)
@@ -12,23 +12,7 @@
      ======================================================================
      -->
-    <!--
-      Actual REP specifications from base_link to rgb frame
-        [x:-0.087m, y:-0.005m, z:0.287m]
-      Is this actually correct?
-    -->
-	<!-- From Turtlebot 1, this is base_link to camera_link with offsets for cam frames
-	<property name="cam_px" value="-0.087" />
-	<property name="cam_py" value="0" />
-	<property name="cam_pz" value="0.287" />
-	<property name="cam_or" value="0" />
-	<property name="cam_op" value="0" />
-	<property name="cam_oy" value="0" />
-    <property name="depth_rel_cam_py" value="0.018" />
-    <property name="rgb_rel_cam_py"   value="-0.005" />
-	 -->
-	 <!-- Yujin specifications - need to double check on these -->
 	<property name="cam_px" value="-0.087" />
 	<property name="cam_py" value="-0.0135" />
-	<property name="cam_pz" value="0.2680" />
+	<property name="cam_pz" value="0.2870" />
 	<property name="cam_or" value="0" />
 	<property name="cam_op" value="0" />

Commit message: original create urdf's for circle stacks, kinect and xtion pro.

File: turtlebot_description/urdf/stacks/hexagons.urdf.xacro (robot description, xacro)
@@ -222,5 +222,5 @@
                  izz="0.01" />
       </inertial>
-		</link>
+    </link>
   </xacro:macro>
 </robot>

File: turtlebot_description/urdf/turtlebot_library.urdf.xacro (robot description, xacro)
@@ -4,10 +4,17 @@
  -->
 <robot>
+  <!-- General -->
   <include filename="$(find turtlebot_description)/urdf/common_properties.urdf.xacro"/>
   <include filename="$(find turtlebot_description)/urdf/turtlebot_properties.urdf.xacro"/>
-  <include filename="$(find turtlebot_description)/urdf/gazebo.urdf.xacro"/>
+  <!-- Bases -->
+  <include filename="$(find turtlebot_description)/urdf/base/create.urdf.xacro"/>
+  <include filename="$(find kobuki_description)/urdf/kobuki.urdf.xacro" />
+  <!-- Stacks -->
+  <include filename="$(find turtlebot_description)/urdf/stacks/circles.urdf.xacro"/>
   <include filename="$(find turtlebot_description)/urdf/stacks/hexagons.urdf.xacro"/>
+  <!-- 3D Sensors -->
   <include filename="$(find turtlebot_description)/urdf/sensors/kinect.urdf.xacro"/>
   <include filename="$(find turtlebot_description)/urdf/sensors/asus_xtion_pro.urdf.xacro"/>
-  <include filename="$(find kobuki_description)/urdf/kobuki.urdf.xacro" />
+  <!-- Gazebo -->
+  <include filename="$(find turtlebot_description)/urdf/gazebo.urdf.xacro"/>
 </robot>

Commit message: removes stl and adds new collada meshes for the hexagon stack; also modifies the urdf accordingly

File: turtlebot_description/urdf/stacks/hexagons.urdf.xacro (robot description, xacro)
@@ -8,4 +8,5 @@
   <xacro:property name="M_SCALE" value="0.001"/>
   <!-- Xacro macros -->
+  <!-- Pole macros -->
   <xacro:macro name="stack_bottom_pole" params="parent number x_loc y_loc z_loc">
     <joint name="pole_bottom_${number}_joint" type="fixed">
@@ -18,10 +19,10 @@
         <origin xyz="0 0 0" rpy="${M_PI/2} 0 ${M_PI/2}"/>
         <geometry>
-          <mesh filename="package://turtlebot_description/meshes/stacks/hexagons/pole_bottom.stl" scale="${M_SCALE} ${M_SCALE} ${M_SCALE}"/>
-        </geometry>
-        <xacro:insert_block name="material_light_grey"/>
-      </visual>
-      <collision>
-        <origin xyz="0 0 0.0246" rpy="0 0 0"/>
+          <mesh filename="package://turtlebot_description/meshes/stacks/hexagons/pole_bottom.dae" scale="${M_SCALE} ${M_SCALE} ${M_SCALE}"/>
+        </geometry>
+        <xacro:insert_block name="material_light_grey"/>
+      </visual>
+      <collision>
+        <origin xyz="0 0 0" rpy="0 0 0"/>
         <geometry>
           <cylinder length="0.0492" radius=".006"/>
@@ -45,7 +46,7 @@
     <link name="pole_middle_${number}_link">
       <visual>
-        <origin xyz="0 0 0" rpy="${-M_PI/2} 0 0"/>
-        <geometry>
-          <mesh filename="package://turtlebot_description/meshes/stacks/hexagons/pole_middle.stl" scale="${M_SCALE} ${M_SCALE} ${M_SCALE}"/>
+        <origin xyz="0 0 0" rpy="${-M_PI/2} ${M_PI} 0"/>
+        <geometry>
+          <mesh filename="package://turtlebot_description/meshes/stacks/hexagons/pole_middle.dae" scale="${M_SCALE} ${M_SCALE} ${M_SCALE}"/>
         </geometry>
         <xacro:insert_block name="material_light_grey"/>
@@ -76,5 +77,5 @@
         <origin xyz=" 0 0 0" rpy="${M_PI/2} 0 ${M_PI/2}"/>
         <geometry>
-          <mesh filename="package://turtlebot_description/meshes/stacks/hexagons/pole_top.stl" scale="${M_SCALE} ${M_SCALE} ${M_SCALE}"/>
+          <mesh filename="package://turtlebot_description/meshes/stacks/hexagons/pole_top.dae" scale="${M_SCALE} ${M_SCALE} ${M_SCALE}"/>
         </geometry>
         <xacro:insert_block name="material_light_grey"/>
@@ -103,7 +104,7 @@
     <link name="pole_kinect_${number}_link">
       <visual>
-        <origin xyz="0 0 0" rpy="${-M_PI/2} 0 0"/>
-        <geometry>
-          <mesh filename="package://turtlebot_description/meshes/stacks/hexagons/pole_kinect.stl" scale="${M_SCALE} ${M_SCALE} ${M_SCALE}"/>
+        <origin xyz="0 0 0" rpy="${-M_PI/2} ${M_PI} 0"/>
+        <geometry>
+          <mesh filename="package://turtlebot_description/meshes/stacks/hexagons/pole_kinect.dae" scale="${M_SCALE} ${M_SCALE} ${M_SCALE}"/>
         </geometry>
         <xacro:insert_block name="material_light_grey"/>
@@ -124,15 +125,14 @@
     </link>
   </xacro:macro>
+  <!-- Stack macro -->
   <xacro:macro name="stack_hexagons" params="parent">
-	<stack_bottom_pole    parent="${parent}" number="0" x_loc= "0.120" y_loc= "0.082" z_loc="0.0714"/>
-	<stack_bottom_pole    parent="${parent}" number="1" x_loc= "0.055" y_loc= "0.120" z_loc="0.0714"/>
-	<stack_bottom_pole    parent="${parent}" number="2" x_loc="-0.055" y_loc= "0.120" z_loc="0.0714"/>
-    <stack_bottom_pole    parent="${parent}" number="3" x_loc= "0.120" y_loc="-0.082" z_loc="0.0714"/>
-    <stack_bottom_pole    parent="${parent}" number="4" x_loc= "0.055" y_loc="-0.120" z_loc="0.0714"/>
-    <stack_bottom_pole    parent="${parent}" number="5" x_loc="-0.055" y_loc="-0.120" z_loc="0.0714"/>
-    <stack_3d_sensor_pole parent="${parent}" number="0" x_loc="-0.1024" y_loc= "0.098" z_loc="0.277"/>
-    <stack_3d_sensor_pole parent="${parent}" number="1" x_loc="-0.1024" y_loc="-0.098" z_loc="0.277"/>
+	  <stack_bottom_pole    parent="${parent}" number="0" x_loc= "0.120" y_loc= "0.082" z_loc="0.073"/>
+	  <stack_bottom_pole    parent="${parent}" number="1" x_loc= "0.055" y_loc= "0.120" z_loc="0.073"/>
+	  <stack_bottom_pole    parent="${parent}" number="2" x_loc="-0.055" y_loc= "0.120" z_loc="0.073"/>
+    <stack_bottom_pole    parent="${parent}" number="3" x_loc= "0.120" y_loc="-0.082" z_loc="0.073"/>
+    <stack_bottom_pole    parent="${parent}" number="4" x_loc= "0.055" y_loc="-0.120" z_loc="0.073"/>
+    <stack_bottom_pole    parent="${parent}" number="5" x_loc="-0.055" y_loc="-0.120" z_loc="0.073"/>
 		<joint name="plate_bottom_joint" type="fixed">
-		  <origin xyz="0.0 0.0  0.1206" rpy="0 0 0"/>
+		  <origin xyz="0.02364 0.0 0.1006" rpy="0 0 0"/>
 		  <parent link="${parent}"/>
 		  <child link="plate_bottom_link"/>
@@ -142,14 +142,13 @@
 		    <origin xyz="0 0 0" rpy="${M_PI/2} 0 ${M_PI/2}"/>
 		    <geometry>
-		      <mesh filename="package://turtlebot_description/meshes/stacks/hexagons/plate_bottom.stl" scale="${M_SCALE} ${M_SCALE} ${M_SCALE}"/>
-		    </geometry>
-        <xacro:insert_block name="material_light_grey"/>
+		      <mesh filename="package://turtlebot_description/meshes/stacks/hexagons/plate_bottom.dae" scale="${M_SCALE} ${M_SCALE} ${M_SCALE}"/>
+		    </geometry>
+        <xacro:insert_block name="material_black"/>
 		  </visual>
 		  <collision>
-		    <origin xyz="0.02364 0.0 0.003" rpy="0 0 0"/>
+		    <origin xyz="0 0 0" rpy="0 0 0"/>
 		    <geometry>
 		      <box size="0.26727 0.345 0.006"/>
 		    </geometry>
-        <xacro:insert_block name="material_light_grey"/>
 		  </collision>
       <inertial>
@@ -161,10 +160,10 @@
       </inertial>
 		</link>
-		<stack_middle_pole parent="${parent}" number="0" x_loc= "0.0702" y_loc= "0.1314" z_loc="0.1874"/>
-		<stack_middle_pole parent="${parent}" number="1" x_loc="-0.0503" y_loc= "0.1314" z_loc="0.1874"/>
-		<stack_middle_pole parent="${parent}" number="2" x_loc= "0.0702" y_loc="-0.1314" z_loc="0.1874"/>
-		<stack_middle_pole parent="${parent}" number="3" x_loc="-0.0503" y_loc="-0.1314" z_loc="0.1874"/>
+		<stack_middle_pole parent="${parent}" number="0" x_loc= "0.0381" y_loc= "0.1505" z_loc="0.134"/>
+		<stack_middle_pole parent="${parent}" number="1" x_loc= "0.0381" y_loc="-0.1505" z_loc="0.134"/>
+		<stack_middle_pole parent="${parent}" number="2" x_loc="-0.0381" y_loc= "0.1505" z_loc="0.134"/>
+		<stack_middle_pole parent="${parent}" number="3" x_loc="-0.0381" y_loc="-0.1505" z_loc="0.134"/>
 		<joint name="plate_middle_joint" type="fixed">
-		  <origin xyz="0.0 0.0 0.1774" rpy="0 0 0"/>
+		  <origin xyz="-0.01364 0.0 0.1574" rpy="0 0 0"/>
 		  <parent link="${parent}"/>
 		  <child link="plate_middle_link"/>
@@ -172,14 +171,14 @@
 		<link name="plate_middle_link">
 		  <visual>
-		    <origin xyz="0 0 0" rpy="${M_PI/2} 0 ${M_PI/2}"/>
-		    <geometry>
-		      <mesh filename="package://turtlebot_description/meshes/stacks/hexagons/plate_middle.stl" scale="${M_SCALE} ${M_SCALE} ${M_SCALE}"/>
-		    </geometry>
-        <xacro:insert_block name="material_light_grey"/>
+		    <origin xyz="0 0 0" rpy="${M_PI/2} 0 -${M_PI/2}"/>
+		    <geometry>
+          <mesh filename="package://turtlebot_description/meshes/stacks/hexagons/plate_middle.dae" scale="${M_SCALE} ${M_SCALE} ${M_SCALE}"/>
+		    </geometry>
+        <xacro:insert_block name="material_black"/>
 		  </visual>
 		  <collision>
-		    <origin xyz="0.0 0.0 -0.015" rpy="0 0 0"/>
-		    <geometry>
-		      <box size="0.31454 0.345 0.006"/>
+		    <origin xyz="0.0 0.0 0.0" rpy="0 0 0"/>
+		    <geometry>
+		      <box size="0.28727 0.340 0.006"/>
 		    </geometry>
 		  </collision>
@@ -192,10 +191,12 @@
       </inertial>
 		</link>
-		<stack_top_pole parent="${parent}" number="0" x_loc= "0.0702" y_loc= "0.1314" z_loc="0.1714"/>
-		<stack_top_pole parent="${parent}" number="1" x_loc="-0.0503" y_loc= "0.1314" z_loc="0.1714"/>
-		<stack_top_pole parent="${parent}" number="2" x_loc= "0.0702" y_loc="-0.1314" z_loc="0.1714"/>
-		<stack_top_pole parent="${parent}" number="3" x_loc="-0.0503" y_loc="-0.1314" z_loc="0.1714"/>
+		<stack_top_pole parent="${parent}" number="0" x_loc= "0.0381" y_loc= "0.1505" z_loc="0.262"/>
+		<stack_top_pole parent="${parent}" number="1" x_loc= "0.0381" y_loc="-0.1505" z_loc="0.262"/>
+		<stack_top_pole parent="${parent}" number="2" x_loc="-0.0381" y_loc= "0.1505" z_loc="0.262"/>
+		<stack_top_pole parent="${parent}" number="3" x_loc="-0.0381" y_loc="-0.1505" z_loc="0.262"/>
+    <stack_3d_sensor_pole parent="${parent}" number="0" x_loc="-0.1024" y_loc= "0.098" z_loc="0.2072"/>
+    <stack_3d_sensor_pole parent="${parent}" number="1" x_loc="-0.1024" y_loc="-0.098" z_loc="0.2072"/>
 		<joint name="plate_top_joint" type="fixed">
-		  <origin xyz="0.0 0.0  0.3866" rpy="0 0 0"/>
+		  <origin xyz="-0.01364 0.0  0.3666" rpy="0 0 0"/>
 		  <parent link="${parent}"/>
 		  <child link="plate_top_link"/>
@@ -203,14 +204,14 @@
 		<link name="plate_top_link">
 		  <visual>
-        <origin xyz="0 0 0" rpy="${M_PI/2} 0 ${M_PI/2}"/>
-		    <geometry>
-		      <mesh filename="package://turtlebot_description/meshes/stacks/hexagons/plate_top.stl" scale="${M_SCALE} ${M_SCALE} ${M_SCALE}"/>
-		    </geometry>
-        <xacro:insert_block name="material_light_grey"/>
+        <origin xyz="0 0 0" rpy="${M_PI/2} 0 -${M_PI/2}"/>
+		    <geometry>
+          <mesh filename="package://turtlebot_description/meshes/stacks/hexagons/plate_top.dae" scale="${M_SCALE} ${M_SCALE} ${M_SCALE}"/>
+		    </geometry>
+        <xacro:insert_block name="material_black"/>
 		  </visual>
 		  <collision>
         <origin xyz="0 0 0" rpy="0 0 0"/>
 		    <geometry>
-		      <box size="0.233502 0.314845 0.006401"/>
+          <box size="0.28727 0.340 0.006"/>
 		    </geometry>
 		  </collision>

Commit message: turtlebot_description: changes hexagon stack plates collision models to cylinders

File: turtlebot_description/urdf/stacks/hexagons.urdf.xacro (robot description, xacro)
@@ -147,7 +147,7 @@
       </visual>
       <collision>
-        <origin xyz="0 0 0" rpy="0 0 0"/>
-        <geometry>
-          <box size="0.26727 0.340 0.006"/>
+        <origin xyz="-0.02364 0 0" rpy="0 0 0"/>
+        <geometry>
+          <cylinder length="0.006" radius="0.170"/>
         </geometry>
       </collision>
@@ -177,7 +177,7 @@
       </visual>
       <collision>
-        <origin xyz="0.0 0.0 0.0" rpy="0 0 0"/>
-        <geometry>
-          <box size="0.28727 0.340 0.006"/>
+        <origin xyz="0.01364 0.0 0.0" rpy="0 0 0"/>
+        <geometry>
+          <cylinder length="0.006" radius="0.170"/>
         </geometry>
       </collision>
@@ -209,7 +209,7 @@
       </visual>
       <collision>
-        <origin xyz="0 0 0" rpy="0 0 0"/>
-        <geometry>
-          <box size="0.28727 0.340 0.006"/>
+        <origin xyz="0.01364 0 0" rpy="0 0 0"/>
+        <geometry>
+          <cylinder length="0.006" radius="0.170"/>
         </geometry>
       </collision>

Commit message: Drop wrong sensor_pole.dae mesh and use instead hexagons/pole_kinect.dae

File: turtlebot_description/urdf/stacks/hexagons.urdf.xacro (robot description, xacro)
@@ -101,7 +101,7 @@
     <link name="pole_kinect_${number}_link">
       <visual>
-        <origin xyz="0 0 -0.01" rpy="0 0 0"/>
-        <geometry>
-          <mesh filename="package://turtlebot_description/meshes/sensors/sensor_pole.dae" />
+        <origin xyz="0 0 0" rpy="0 0 0"/>
+        <geometry>
+          <mesh filename="package://turtlebot_description/meshes/stacks/hexagons/pole_kinect.dae" />
         </geometry>
       </visual>
